File: Hardware/_Sub_Hardware_Project/vX_YYYYMMDD/Design Folder/_ProjectFiles_/_ProjectTemplate_/_ProjectTemplate_.kicad_sch (KiCad schematic)
At the start: 0 parts

Commit message: Working on file structures
Other:
- note added: "${COMMENT2}"
- note added: "1- Go to View -> Pge Preview Setting 2- Set Parameters based on the following Info COMMENT 1: Project Version COMMENT 2: Document Status COMMENT 3: Doc. Approval Eng. COMMENT 4: BOM Ref. DOC. COMMENT 5: PCB Ref. DOC. COMMENT 6: GBR Ref. DOC. COMMENT 7: ASM Ref. DOC. COMMENT 8: Variant Name COMMENT 9: Revision Description"
- note added: "21"
- note added: "22"
- note added: "23"
- note added: "24"
- note added: "25"
- note added: "26"
- note added: "27"
- note added: "28"
- note added: "29"
- note added: "30"
- note added: "3D Preview BOTTOM"
- note added: "3D Preview TOP"
- note added: "Board Statistics Stackup Info"
- note added: "SHOULD BE ADDED AFTER RELEASE"
- note removed: "1- Go to View -> Pge Preview Setting 2- Set Parameters based on the following Info COMMENT 1: Project Version COMMENT 2: Document Version COMMENT 3: Doc. Approval Eng. COMMENT 4: BOM Ref. DOC. COMMENT 5: PCB Ref. DOC. COMMENT 6: GBR Ref. DOC. COMMENT 7: ASM Ref. DOC. COMMENT 8: Variant Name COMMENT 9: Revision Description"
- note removed: "DRAFT"
