File: Hardware/_Sub_HW_Qcopter/v1_20240309/Design Folder/_Sub_HW_Qcopter/[0303] - Debug USART.kicad_sch (KiCad schematic)
At the start: 0 parts

Commit message: Schematic is done by 90%
Parts:
- added J701: HDR_1X3_THD-1.27MM, Connector_PinHeader_1.27mm:PinHeader_1x03_P1.27mm_Vertical, symbol _SCHLIB_Qcopter:CONN_HDR_1X3_VERT_THD-1.27MM
- added R701, R702: 100R_1/10W_1%, Resistor_SMD:R_0603_1608Metric, symbol _SCHLIB_Qcopter:RES_100R_1/10W_1%_R0603
Connections:
- new net: J701.2, R701.2
- new net: J701.3, R702.2
- new net GND: J701.1
- new net UART_RX: R701.1
- new net UART_TX: R702.1
