File: Hardware/_Sub_HW_Qcopter/v1_20240309/Design Folder/_Sub_HW_Qcopter/[0307] - OV2640 Driver.kicad_sch (KiCad schematic)
At the start: 0 parts

Commit message: Schematic is done by 90%
Parts:
- added C1101, C1107, C1108: 4u7F_16V_X7R, Capacitor_SMD:C_0603_1608Metric, symbol _SCHLIB_Qcopter:CAP_CER_4.7uF_16V_X7R_C0603
- added J1101: FPC_24_R/A-BOTT, footrpring, symbol _SCHLIB_Qcopter:CONN_FPC/FFC_24POS_R/A_SMD-0.5MM
Connections:
- new net OV2460_+1V3DC: C1101.1, J1101.10
- new net OV2460_+2V8DC: C1108.1, J1101.4
- new net OV2460_+3V3DC: C1107.1, J1101.11
- new net OV2460_AGND: C1108.2, J1101.2
- new net OV2460_DATA0: J1101.24
- new net OV2460_DATA1: J1101.23
- new net OV2460_DATA2: J1101.19
- new net OV2460_DATA3: J1101.21
- new net OV2460_DATA4: J1101.22
- new net OV2460_DATA5: J1101.20
- new net OV2460_DATA6: J1101.18
- new net OV2460_DATA7: J1101.16
- new net OV2460_DATA8: J1101.14
- new net OV2460_DATA9: J1101.12
- new net OV2460_DGND: C1101.2, C1107.2, J1101.15
- new net OV2460_HREF: J1101.9
- new net OV2460_PCLK: J1101.17
- new net OV2460_PWDN: J1101.8
- new net OV2460_RESETB: J1101.6
- new net OV2460_SIOC: J1101.5
- new net OV2460_SIOD: J1101.3
- new net OV2460_STROBE: J1101.1
- new net OV2460_VSYNC: J1101.7
- new net OV2460_XCLK: J1101.13
Other:
- note added: "DESIGN NOTE:"
- note added: "INFO:"
