File: Hardware/_Sub_HW_Qcopter/v1_20240309/Design Folder/_Sub_HW_Qcopter/[0308] - W25Q64 Driver.kicad_sch (KiCad schematic)
At the start: 0 parts

Commit message: Schematic is done by 90%
Parts:
- added C1201: 1uF_10V_X7R, Capacitor_SMD:C_0603_1608Metric, symbol _SCHLIB_Qcopter:CAP_CER_1uF_10V_X7R_C0603
- added R1201: 10kR_1/10W_1%, Resistor_SMD:R_0603_1608Metric, symbol _SCHLIB_Qcopter:RES_10kR_1/10W_1%_R0603
- added U1201: W25Q64JVSSIQ, Package_SO:SOIC-8_5.23x5.23mm_P1.27mm, symbol _SCHLIB_Qcopter:IC_MEM_W25Q64JVSSIQ_64MBIT_NOR_QSPI/SPI_8-SOIC
Connections:
- new net GND: C1201.2, U1201.4 (GND)
- new net PWR: C1201.1, R1201.1, U1201.8 (VCC)
- new net QSPI_CLK: U1201.6 (CLK)
- new net QSPI_IO0: U1201.5 (IO0)
- new net QSPI_IO1: U1201.2 (IO1)
- new net QSPI_IO2: U1201.3 (IO2)
- new net QSPI_IO3: U1201.7 (IO3)
- new net QSPI_~{CS}: R1201.2, U1201.1 (~{CS})
Other:
- note added: "INFO:"
