File: Hardware/_Sub_HW_Qcopter/v1_20240309/Design Folder/_Sub_HW_Qcopter/[0311] - Battery Voltage Sampler.kicad_sch (KiCad schematic)
At the start: 0 parts

Commit message: Schematic is done by 90%
Parts:
- added C2101: 100nF_16V_X7R, Capacitor_SMD:C_0603_1608Metric, symbol _SCHLIB_Qcopter:CAP_CER_100nF_16V_X7R_C0603
- added R2101: 10kR_1/10W_1%, Resistor_SMD:R_0603_1608Metric, symbol _SCHLIB_Qcopter:RES_10kR_1/10W_1%_R0603
- added R2102, R2103, R2104: 100kR_1/10W_1%, Resistor_SMD:R_0603_1608Metric, symbol _SCHLIB_Qcopter:RES_100kR_1/10W_1%_R0603
- added U2101: MCP6006T-E/OT, Package_TO_SOT_SMD:SOT-23-5, symbol _SCHLIB_Qcopter:IC_OPAMP_MCP6006T-E/OT_GP_1C_SOT-23-5
Connections:
- new net GND: C2101.2, R2103.2, R2104.2, U2101.2 (VSS)
- new net MCP_VIN+: R2102.2, R2103.1, U2101.3 (VIN+)
- new net MCP_VIN-: R2101.1, U2101.4 (VIN-)
- new net PWR: C2101.1, U2101.5 (VDD)
- new net V_IN: R2102.1
- new net V_OUT: R2101.2, R2104.1, U2101.1 (VOUT)
