File: Hardware/_Sub_HW_Qcopter/v1_20240309/Design Folder/_Sub_HW_Qcopter/[0402] - RESET Circuit.kicad_sch (KiCad schematic)
At the start: 0 parts

Commit message: Schematic is done by 90%
Parts:
- added C1601: 100nF_16V_X7R, Capacitor_SMD:C_0603_1608Metric, symbol _SCHLIB_Qcopter:CAP_CER_100nF_16V_X7R_C0603
- added JP1601: JP_2POS, Jumper:SolderJumper-2_P1.3mm_Open_TrianglePad1.0x1.5mm, symbol _SCHLIB_Qcopter:MECH_JUMPER_2POS_J1015
- added R1601: 10kR_1/10W_1%, Resistor_SMD:R_0603_1608Metric, symbol _SCHLIB_Qcopter:RES_10kR_1/10W_1%_R0603
- added R1602: 100kR_1/10W_1%, Resistor_SMD:R_0603_1608Metric, symbol _SCHLIB_Qcopter:RES_100kR_1/10W_1%_R0603
- added U1601: SN74LVC1G17DCKR, Package_TO_SOT_SMD:SOT-353_SC-70-5, symbol _SCHLIB_Qcopter:IC_BUFF_SN74LVC1G17DCKR_NON-INV_1BIT_SC-70-5
Connections:
- new net BUFF_IN: JP1601.1, R1601.2, U1601.2 (A)
- new net BUFF_OUT: R1602.1, U1601.4 (Y)
- new net GND: C1601.2, JP1601.2, R1602.2, U1601.3 (GND)
- new net PWR: C1601.1, R1601.1, U1601.5 (VCC)
- no-connect marks 0 -> 1
Other:
- note added: "DESIGN NOTE:"
- note added: "INFO:"
- note added: "To reset the target IC just short circuit the jumper and the output will set to zero"
