File: Hardware/_Sub_HW_Qcopter/v1_20240309/Design Folder/_Sub_HW_Qcopter/[020106] - GPIO Expander.kicad_sch (KiCad schematic)
At the start: 0 parts

Commit message: 97% drawing schematic is done
Changed lines of the file:
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@@
+	(wire
+		(pts
+			(xy 363.22 185.42) (xy 372.11 185.42)
+		)
+		(stroke
+			(width 0)
+			(type default)
+		)
+	)
 	(wire
 		(pts
@@
 	(wire
 		(pts
+			(xy 363.22 187.96) (xy 372.11 187.96)
+		)
+		(stroke
+			(width 0)
+			(type default)
+		)
+	)
+	(wire
+		(pts
 			(xy 185.42 180.34) (xy 194.31 180.34)
 		)
@@
 		)
 	)
-	(text_box "INFO:\n\nMOTOR CTRL 1\nMOTOR CTRL 2\nMOTOR CTRL 3\nMOTOR CTRL 4\nMOTOR DIR 1\nMOTOR DIR 2\nMOTOR DIR 3\nMOTOR DIR 4\n\nIMU CS\nBME250 CS\nCAMERA PWRDN\nCAMERA RST\nRADIO CONTROLLER RST\nLDO1 RST\nLDO2 RST\nLDO3 RST\n\nCHASSIS LED 1\nCHASSIS LED 2\nCHASSIS LED 3\nCHASSIS LED 4\nDEBUG USART LED TX\nDEBUG USART LED RX"
+	(text_box "INFO:\n\nMOTOR CTRL 1\nMOTOR CTRL 2\nMOTOR CTRL 3\nMOTOR CTRL 4\nMOTOR DIR 1\nMOTOR DIR 2\nMOTOR DIR 3\nMOTOR DIR 4\n\nLDO1 RST\nLDO2 RST\nLDO3 RST\nLDO4 RST\nLDO5 RST\nCAMERA PWRDN\nCAMERA RST\nRADIO CONTROLLER RST\n\nCHASSIS LED 1\nCHASSIS LED 2\nCHASSIS LED 3\nCHASSIS LED 4\nDEBUG USART LED TX\nDEBUG USART LED RX\nIMU CS\nBME250 CS"
 		(exclude_from_sim no)
 		(at 54.864 244.856 0)
-		(size 64.77 109.22)
+		(size 64.77 118.364)
 		(stroke
 			(width 0)
@@
 	(text "GROUP 3"
 		(exclude_from_sim no)
-		(at 110.744 340.36 90)
+		(at 110.744 344.678 90)
 		(effects
 			(font
@@
 		)
 	)
-	(hierarchical_label "OV2640_PWRDN"
-		(shape output)
-		(at 285.75 175.26 0)
+	(hierarchical_label "EN_LDO_5"
+		(shape output)
+		(at 285.75 180.34 0)
 		(fields_autoplaced yes)
 		(effects
@@
 	(hierarchical_label "OV2640_RST"
 		(shape output)
-		(at 285.75 177.8 0)
+		(at 285.75 185.42 0)
+		(fields_autoplaced yes)
+		(effects
+			(font
+				(size 1.27 1.27)
+			)
+			(justify left)
+		)
+	)
+	(hierarchical_label "CHASSIS_LED_2"
+		(shape output)
+		(at 372.11 172.72 0)
+		(fields_autoplaced yes)
+		(effects
+			(font
+				(size 1.27 1.27)
+			)
+			(justify left)
+		)
+	)
+	(hierarchical_label "DEBUG_USART_LED_TX"
+		(shape output)
+		(at 372.11 180.34 0)
 		(fields_autoplaced yes)
 		(effects
@@
 	(hierarchical_label "ICM_AD0"
 		(shape output)
+		(at 372.11 185.42 0)
+		(fields_autoplaced yes)
+		(effects
+			(font
+				(size 1.27 1.27)
+			)
+			(justify left)
+		)
+	)
+	(hierarchical_label "EN_LDO_1"
+		(shape output)
 		(at 285.75 170.18 0)
-		(fields_autoplaced yes)
-		(effects
-			(font
-				(size 1.27 1.27)
-			)
-			(justify left)
-		)
-	)
-	(hierarchical_label "RADIO_CTRL_RST"
-		(shape output)
-		(at 285.75 180.34 0)
-		(fields_autoplaced yes)
-		(effects
-			(font
-				(size 1.27 1.27)
-			)
-			(justify left)
-		)
-	)
-	(hierarchical_label "CHASSIS_LED_2"
-		(shape output)
-		(at 372.11 172.72 0)
-		(fields_autoplaced yes)
-		(effects
-			(font
-				(size 1.27 1.27)
-			)
-			(justify left)
-		)
-	)
-	(hierarchical_label "DEBUG_USART_LED_TX"
-		(shape output)
-		(at 372.11 180.34 0)
-		(fields_autoplaced yes)
-		(effects
-			(font
-				(size 1.27 1.27)
-			)
-			(justify left)
-		)
-	)
-	(hierarchical_label "EN_LDO_1"
-		(shape output)
-		(at 285.75 182.88 0)
 		(fields_autoplaced yes)
 		(effects
@@
 		)
 	)
+	(hierarchical_label "BME280_AD0"
+		(shape output)
+		(at 372.11 187.96 0)
+		(fields_autoplaced yes)
+		(effects
+			(font
+				(size 1.27 1.27)
+			)
+			(justify left)
+		)
+	)
+	(hierarchical_label "MOTOR_DIR_1"
+		(shape output)
+		(at 194.31 180.34 0)
+		(fields_autoplaced yes)
+		(effects
+			(font
+				(size 1.27 1.27)
+			)
+			(justify left)
+		)
+	)
+	(hierarchical_label "CHASSIS_LED_1"
+		(shape output)
+		(at 372.11 170.18 0)
+		(fields_autoplaced yes)
+		(effects
+			(font
+				(size 1.27 1.27)
+			)
+			(justify left)
+		)
+	)
+	(hierarchical_label "MOTOR_DIR_4"
+		(shape output)
+		(at 194.31 187.96 0)
+		(fields_autoplaced yes)
+		(effects
+			(font
+				(size 1.27 1.27)
+			)
+			(justify left)
+		)
+	)
 	(hierarchical_label "EN_LDO_2"
 		(shape output)
-		(at 285.75 185.42 0)
-		(fields_autoplaced yes)
-		(effects
-			(font
-				(size 1.27 1.27)
-			)
-			(justify left)
-		)
-	)
-	(hierarchical_label "MOTOR_DIR_1"
-		(shape output)
-		(at 194.31 180.34 0)
-		(fields_autoplaced yes)
-		(effects
-			(font
-				(size 1.27 1.27)
-			)
-			(justify left)
-		)
-	)
-	(hierarchical_label "CHASSIS_LED_1"
-		(shape output)
-		(at 372.11 170.18 0)
-		(fields_autoplaced yes)
-		(effects
-			(font
-				(size 1.27 1.27)
-			)
-			(justify left)
-		)
-	)
-	(hierarchical_label "MOTOR_DIR_4"
-		(shape output)
-		(at 194.31 187.96 0)
+		(at 285.75 172.72 0)
 		(fields_autoplaced yes)
 		(effects
@@
 		)
 	)
-	(hierarchical_label "EN_LDO_3"
+	(hierarchical_label "EN_LDO_4"
+		(shape output)
+		(at 285.75 177.8 0)
+		(fields_autoplaced yes)
+		(effects
+			(font
+				(size 1.27 1.27)
+			)
+			(justify left)
+		)
+	)
+	(hierarchical_label "MOTOR_CTRL_4"
+		(shape output)
+		(at 194.31 177.8 0)
+		(fields_autoplaced yes)
+		(effects
+			(font
+				(size 1.27 1.27)
+			)
+			(justify left)
+		)
+	)
+	(hierarchical_label "CHASSIS_LED_4"
+		(shape output)
+		(at 372.11 177.8 0)
+		(fields_autoplaced yes)
+		(effects
+			(font
+				(size 1.27 1.27)
+			)
+			(justify left)
+		)
+	)
+	(hierarchical_label "OV2640_PWRDN"
+		(shape output)
+		(at 285.75 182.88 0)
+		(fields_autoplaced yes)
+		(effects
+			(font
+				(size 1.27 1.27)
+			)
+			(justify left)
+		)
+	)
+	(hierarchical_label "RADIO_CTRL_RST"
 		(shape output)
 		(at 285.75 187.96 0)
-		(fields_autoplaced yes)
-		(effects
-			(font
-				(size 1.27 1.27)
-			)
-			(justify left)
-		)
-	)
-	(hierarchical_label "MOTOR_CTRL_4"
-		(shape output)
-		(at 194.31 177.8 0)
-		(fields_autoplaced yes)
-		(effects
-			(font
-				(size 1.27 1.27)
-			)
-			(justify left)
-		)
-	)
-	(hierarchical_label "CHASSIS_LED_4"
-		(shape output)
-		(at 372.11 177.8 0)
-		(fields_autoplaced yes)
-		(effects
-			(font
-				(size 1.27 1.27)
-			)
-			(justify left)
-		)
-	)
-	(hierarchical_label "BME280_AD0"
-		(shape output)
-		(at 285.75 172.72 0)
 		(fields_autoplaced yes)
 		(effects
@@
 		)
 	)
+	(hierarchical_label "EN_LDO_3"
+		(shape output)
+		(at 285.75 175.26 0)
+		(fields_autoplaced yes)
+		(effects
+			(font
+				(size 1.27 1.27)
+			)
+			(justify left)
+		)
+	)
