File: Hardware/_Sub_HW_Qcopter/v1_20240309/Design Folder/_Sub_HW_Qcopter/[03] - FBD_FlightController.kicad_sch (KiCad schematic)
At the start: 0 parts

Commit message: Schematic is done by 90%
Other:
- sheet BMI160 Driver renamed ICM-20948 Driver
- sheet SN74HC595 Driver renamed GPIO Expander
- removed sheet LDO
- removed sheet Radio Controller Interface
- added sheet LEDs Driver ([020110] - LEDs Driver.kicad_sch)
- sheet BME280 Driver: file [0305] - BME Driver.kicad_sch -> [020105] - BME280 Driver.kicad_sch
- sheet BME280 Driver ports: added BME280_A0, BME280_SCL, BME280_SDA, GND, PWR; removed none
- sheet Battery Voltage Sampler ports: added GND, PWR, V_IN, V_OUT; removed none
- sheet Debug USART ports: added GND, UART_RX, UART_TX; removed none
- sheet GPIO Expander: file [0306] - SN74HC595 Driver.kicad_sch -> [020106] - GPIO Expander.kicad_sch
- sheet GPIO Expander ports: added +PWR, BME280_AD0, CHASSIS_LED_1, CHASSIS_LED_2, CHASSIS_LED_3, CHASSIS_LED_4, DEBUG_USART_LED_RX, DEBUG_USART_LED_TX, EN_LDO_1, EN_LDO_2, EN_LDO_3, GND, I2C_SCL, I2C_SDA, ICM_AD0, MOTOR_CTRL_1, MOTOR_CTRL_2, MOTOR_CTRL_3, MOTOR_CTRL_4, MOTOR_DIR_1, MOTOR_DIR_2, MOTOR_DIR_3, MOTOR_DIR_4, OV2640_PWRDN, OV2640_RST, RADIO_CTRL_RST; removed none
- sheet ICM-20948 Driver: file [0304] - BMI160 Driver.kicad_sch -> [020104] - ICM-20948 Driver.kicad_sch
- sheet ICM-20948 Driver ports: added GND, ICM_AD0, ICM_INT, ICM_SCL, ICM_SDA, PWR; removed none
- sheet MCU Driver ports: added ADC_A0, DCMI_D0, DCMI_D1, DCMI_D2, DCMI_D3, DCMI_D4, DCMI_D5, DCMI_D6, DCMI_D7, DCMI_D8, DCMI_D9, DCMI_HSYNC, DCMI_PIXCLK, DCMI_VSYNC, DCMI_XLCK, GND, I2C1_SCL, I2C1_SDA, I2C2_SCL, I2C2_SDA, ICM_INT, LPUART1_RX, LPUART1_TX, MCU_NRST, OTG_USB_DM, OTG_USB_DP, OTG_USB_ID, PWR, QSPI_CLK, QSPI_D0, QSPI_D1, QSPI_D2, QSPI_D3, QSPI_NSS, SPI_CLK, SPI_MISO, SPI_MOSI, SPI_NSS, TIM3_CH1, TIM3_CH2, TIM3_CH3, TIM3_CH4, USART2_RX, USART2_TX; removed none
- sheet Motor Driver ports: added MOTOR_CTR_+V, MOTOR_EN_1, MOTOR_EN_2, MOTOR_EN_3, MOTOR_EN_4, MOTOR_GND, MOTOR_VM, MOTO_DIR_1, MOTO_DIR_2, MOTO_DIR_3, MOTO_DIR_4, MOTO_PWM_1, MOTO_PWM_2, MOTO_PWM_3, MOTO_PWM_4; removed none
- sheet OV2640 Driver ports: added OV2460_+1V3DC, OV2460_+2V8DC, OV2460_+3V3DC, OV2460_AGND, OV2460_DATA0, OV2460_DATA1, OV2460_DATA2, OV2460_DATA3, OV2460_DATA4, OV2460_DATA5, OV2460_DATA6, OV2460_DATA7, OV2460_DATA8, OV2460_DATA9, OV2460_DGND, OV2460_HREF, OV2460_PCLK, OV2460_PWDN, OV2460_RESETB, OV2460_SIOC, OV2460_SIOD, OV2460_STROBE, OV2460_VSYNC, OV2460_XCLK; removed none
- sheet RESET Circuit ports: added BUFF_OUT, GND, PWR; removed none
- sheet W25Q64 Driver ports: added GND, PWR, QSPI_CLK, QSPI_IO0, QSPI_IO1, QSPI_IO2, QSPI_IO3, QSPI_~{CS}; removed none
- note removed: "10"
- note removed: "11"

Commit message: 97% drawing schematic is done
Other:
- sheet GPIO Expander ports: added EN_LDO_4, EN_LDO_5; removed none
Changed lines of the file:
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@@
 	(wire
 		(pts
-			(xy 408.94 227.33) (xy 408.94 142.24)
+			(xy 408.94 231.14) (xy 408.94 142.24)
 		)
 		(stroke
@@
 	(wire
 		(pts
-			(xy 410.21 80.01) (xy 431.8 80.01)
+			(xy 419.1 85.09) (xy 431.8 85.09)
 		)
 		(stroke
@@
 	(wire
 		(pts
-			(xy 421.64 85.09) (xy 431.8 85.09)
+			(xy 172.72 279.4) (xy 177.8 279.4)
 		)
 		(stroke
@@
 	(wire
 		(pts
-			(xy 172.72 279.4) (xy 177.8 279.4)
+			(xy 414.02 209.55) (xy 431.8 209.55)
 		)
 		(stroke
@@
 	(wire
 		(pts
-			(xy 414.02 209.55) (xy 431.8 209.55)
+			(xy 419.1 82.55) (xy 431.8 82.55)
 		)
 		(stroke
@@
 	(wire
 		(pts
-			(xy 421.64 82.55) (xy 431.8 82.55)
+			(xy 381 223.52) (xy 386.08 223.52)
 		)
 		(stroke
@@
 	(wire
 		(pts
-			(xy 381 218.44) (xy 386.08 218.44)
+			(xy 381 214.63) (xy 386.08 214.63)
 		)
 		(stroke
@@
 	(wire
 		(pts
-			(xy 406.4 224.79) (xy 406.4 139.7)
+			(xy 406.4 228.6) (xy 406.4 139.7)
 		)
 		(stroke
@@
 	(wire
 		(pts
-			(xy 381 224.79) (xy 406.4 224.79)
+			(xy 381 228.6) (xy 406.4 228.6)
 		)
 		(stroke
@@
 	(wire
 		(pts
-			(xy 381 227.33) (xy 408.94 227.33)
+			(xy 381 231.14) (xy 408.94 231.14)
 		)
 		(stroke
@@
 	(wire
 		(pts
+			(xy 381 217.17) (xy 386.08 217.17)
+		)
+		(stroke
+			(width 0)
+			(type default)
+		)
+	)
+	(wire
+		(pts
 			(xy 283.21 213.36) (xy 292.1 213.36)
 		)
@@
 	(wire
 		(pts
+			(xy 419.1 80.01) (xy 431.8 80.01)
+		)
+		(stroke
+			(width 0)
+			(type default)
+		)
+	)
+	(wire
+		(pts
 			(xy 364.49 177.8) (xy 364.49 111.76)
 		)
@@
 	(text_box "2 X SN74HC595\nDriver"
 		(exclude_from_sim no)
-		(at 315.468 247.65 0)
+		(at 342.138 328.93 0)
 		(size 25.4 25.4)
 		(stroke
@@
 	(text "7"
 		(exclude_from_sim no)
-		(at 328.93 267.97 0)
+		(at 355.6 349.25 0)
 		(effects
 			(font
@@
 		)
 	)
+	(label "+3V3_1"
+		(at 419.1 195.58 0)
+		(fields_autoplaced yes)
+		(effects
+			(font
+				(size 1.27 1.27)
+			)
+			(justify left bottom)
+		)
+	)
 	(label "GND"
 		(at 165.1 248.92 0)
@@
 		)
 	)
+	(label "+3V3_1"
+		(at 419.1 231.14 0)
+		(fields_autoplaced yes)
+		(effects
+			(font
+				(size 1.27 1.27)
+			)
+			(justify left bottom)
+		)
+	)
 	(label "I2C_SCL"
 		(at 292.1 243.84 0)
@@
 		)
 	)
-	(label "+3V3DC"
-		(at 330.2 207.01 0)
-		(fields_autoplaced yes)
-		(effects
-			(font
-				(size 1.27 1.27)
-			)
-			(justify left bottom)
-		)
-	)
 	(label "GND"
 		(at 165.1 173.99 0)
@@
 		)
 	)
-	(label "+3V3DC"
-		(at 243.84 154.94 0)
+	(label "+3V3_1"
+		(at 419.1 335.28 0)
 		(fields_autoplaced yes)
 		(effects
@@
 	)
 	(label "+3V3DC"
-		(at 165.1 232.41 0)
+		(at 243.84 154.94 0)
 		(fields_autoplaced yes)
 		(effects
@@
 		)
 	)
-	(label "I2C_SCL"
-		(at 419.1 204.47 0)
+	(label "+3V3DC"
+		(at 165.1 232.41 0)
 		(fields_autoplaced yes)
 		(effects
@@
 		)
 	)
-	(label "+3V3DC"
-		(at 419.1 335.28 0)
+	(label "I2C_SCL"
+		(at 419.1 204.47 0)
 		(fields_autoplaced yes)
 		(effects
@@
 		)
 	)
-	(label "+3V3DC"
-		(at 419.1 195.58 0)
+	(label "+3V3_1"
+		(at 330.2 207.01 0)
 		(fields_autoplaced yes)
 		(effects
@@
 		)
 	)
-	(label "+3V3DC"
-		(at 419.1 231.14 0)
-		(fields_autoplaced yes)
-		(effects
-			(font
-				(size 1.27 1.27)
-			)
-			(justify left bottom)
-		)
-	)
 	(label "GND"
 		(at 165.1 288.29 0)
@@
 		)
 	)
-	(label "+3V3DC"
-		(at 410.21 80.01 0)
+	(label "+3V3_1"
+		(at 420.37 80.01 0)
 		(fields_autoplaced yes)
 		(effects
@@
 		)
 	)
+	(hierarchical_label "EN_LDO_5"
+		(shape output)
+		(at 386.08 217.17 0)
+		(fields_autoplaced yes)
+		(effects
+			(font
+				(size 1.27 1.27)
+			)
+			(justify left)
+		)
+	)
 	(hierarchical_label "RADIO_CTR_UART_TX"
 		(shape input)
@@
 		)
 	)
+	(hierarchical_label "+3V3_1"
+		(shape input)
+		(at 419.1 80.01 180)
+		(fields_autoplaced yes)
+		(effects
+			(font
+				(size 1.27 1.27)
+			)
+			(justify right)
+		)
+	)
+	(hierarchical_label "VM"
+		(shape input)
+		(at 419.1 332.74 180)
+		(fields_autoplaced yes)
+		(effects
+			(font
+				(size 1.27 1.27)
+			)
+			(justify right)
+		)
+	)
 	(hierarchical_label "PWR_+1V3"
 		(shape input)
-		(at 421.64 85.09 180)
+		(at 419.1 85.09 180)
 		(fields_autoplaced yes)
 		(effects
@@
 	(hierarchical_label "RADIO_CTR_RST"
 		(shape output)
-		(at 386.08 218.44 0)
+		(at 386.08 223.52 0)
 		(fields_autoplaced yes)
 		(effects
@@
 		)
 	)
-	(hierarchical_label "PWR_+2V8"
-		(shape input)
-		(at 421.64 82.55 180)
+	(hierarchical_label "EN_LDO_4"
+		(shape output)
+		(at 386.08 214.63 0)
 		(fields_autoplaced yes)
 		(effects
@@
 				(size 1.27 1.27)
 			)
-			(justify right)
+			(justify left)
 		)
 	)
-	(hierarchical_label "+3V3_1"
+	(hierarchical_label "PWR_+2V8"
 		(shape input)
-		(at 419.1 332.74 180)
+		(at 419.1 82.55 180)
 		(fields_autoplaced yes)
 		(effects
@@
 		)
 		(pin "RADIO_CTRL_RST" output
-			(at 381 218.44 0)
+			(at 381 223.52 0)
 			(effects
 				(font
@@
 		)
 		(pin "OV2640_RST" output
-			(at 381 224.79 0)
+			(at 381 228.6 0)
 			(effects
 				(font
@@
 		)
 		(pin "OV2640_PWRDN" output
-			(at 381 227.33 0)
+			(at 381 231.14 0)
 			(effects
 				(font
@@
 			(effects
 				(font
+					(size 1.27 1.27)
+				)
+				(justify right)
+			)
+		)
+		(pin "EN_LDO_4" output
+			(at 381 214.63 0)
+			(effects
+				(font
+					(size 1.27 1.27)
+				)
+				(justify right)
+			)
+		)
+		(pin "EN_LDO_5" output
+			(at 381 217.17 0)
+			(effects
+				(font
