File: Hardware/_Sub_HW_Qcopter/v1_20240309/Design Folder/_Sub_HW_Qcopter/[0405] - ATWIL1000C Driver.kicad_sch (KiCad schematic)
At the start: 0 parts

Commit message: Schematic is done by 90%
Parts:
- added C1801, C1802, C1803: 1uF_10V_X7R, Capacitor_SMD:C_0603_1608Metric, symbol _SCHLIB_Qcopter:CAP_CER_1uF_10V_X7R_C0603
- added C1804, C1805, C1806, C1807, C1808, C1809, C1810, C1811, C1812, C1813, C1814, C1815: 4u7F_16V_X7R, Capacitor_SMD:C_0603_1608Metric, symbol _SCHLIB_Qcopter:CAP_CER_4.7uF_16V_X7R_C0603
- added C1816, C1817: 12pF_50V_C0G, Capacitor_SMD:C_0603_1608Metric, symbol _SCHLIB_Qcopter:CAP_CER_12pF_50V_C0G_C0603
- added R1801, R1802, R1803, R1804, R1805, R1806: 100kR_1/10W_1%, Resistor_SMD:R_0603_1608Metric, symbol _SCHLIB_Qcopter:RES_100kR_1/10W_1%_R0603
- added R1807, R1808, R1809, R1810: 1kR_1/10W_1%, Resistor_SMD:R_0603_1608Metric, symbol _SCHLIB_Qcopter:RES_1kR_1/10W_1%_R0603
- added U1801: ATWILC1000B-MU-Y, _PCBLIB_SparkleSplashy:QFN-40-1EP_5x5mm_P0.4mm_EP3.8x3.8mm_ThermalVias, symbol _SCHLIB_Qcopter:IC_RF TXRX_ATWILC1000B-MU-Y_Wifi_2.4GHz_40-QFN (5x5)
- added X1801: 26MHz_10ppm_12pF, Crystal:Crystal_SMD_2016-4Pin_2.0x1.6mm, symbol _SCHLIB_Qcopter:XTAL_ECS-260-12-37B2-CKM-TR_26MHz_10PPM_12pF_4-SMD, No Lead
Connections:
- new net: R1810.1, U1801.30 (GPIO5)
- new net: R1809.1, U1801.28 (GPIO3)
- new net +PWR: C1801.1, C1802.1, C1803.1, C1804.1, C1805.1, C1806.1, R1801.1, R1802.1, R1803.1, R1806.1, R1807.1, R1808.1, U1801.15 (VDDIO_3V3), U1801.20 (VBATT_BUCK_3V3), U1801.26 (VDDIO_3V3), U1801.39 (VDDIO_A_3V3), U1801.5 (VDD_BATT_PPA_3V3), U1801.6 (VDD_BATT_PA_3V3)
- new net ATWILC_+1.3V: C1807.1, C1808.1, C1809.1, C1810.1, C1811.1, C1812.1, C1813.1, C1814.1, C1815.1, U1801.14 (VDDC_1V3), U1801.2 (VDD_RF_RX_1V3), U1801.21 (VSW), U1801.22 (VREG_BUCK), U1801.27 (VDDC_1V3), U1801.3 (VDD_AMS_1V3), U1801.37 (VDD_SXDIG_1V3), U1801.38 (VDD_VCO_1V3), U1801.4 (VDD_RF_TX_1V3)
- new net ATWILC_CHIPN: R1804.1, U1801.23 (CHIP_EN)
- new net ATWILC_IRQN: R1803.2, U1801.11 (GPIO2/IRQN)
- new net ATWILC_RESETN: R1805.1, U1801.34 (RESETN)
- new net ATWILC_RXD: R1809.2
- new net ATWILC_TXD: R1810.2
- new net ATWILC_WAKEUP: R1802.2, U1801.10 (GPIO0/HOST_WAKEUP)
- new net ATWILC_XON: C1817.1, U1801.35 (XO_N), X1801.3
- new net ATWILC_XOP: C1816.1, U1801.36 (XO_P), X1801.1
- new net ATWILC_~{SDIO}_SPI: R1801.2, U1801.9 (~{SDIO}_SPI_CFG)
- new net GND: C1801.2, C1802.2, C1803.2, C1804.2, C1805.2, C1806.2, C1807.2, C1808.2, C1809.2, C1810.2, C1811.2, C1812.2, C1813.2, C1814.2, C1815.2, C1816.2, C1817.2, R1804.2, R1805.2, U1801.25 (TEST_MODE), U1801.41 (VSS), X1801.2, X1801.4
- new net I2C_SCL: R1808.2, U1801.32 (I2C_SCL)
- new net I2C_SDA: R1807.2, U1801.33 (I2C_SDA)
- new net SPI_CS: R1806.2, U1801.16 (SD_DAT1/SPI_SSN)
- new net SPI_MISO: U1801.17 (SD_DAT0/SPI_TXD)
- new net SPI_MOSI: U1801.13 (SD_DAT2/SPI_RXD)
- new net SPI_SCK: U1801.18 (SD_CMD/SPI_SCK)
- no-connect marks 0 -> 7
Other:
- note added: "INFO: (CHIP_EN PIN) • Device enable • High level enables device, low level places device in Power-Down mode • Connect to a host output that has default low at power-up; if the host output is tristated, add a 1 MΩ pull-down resistor to ensure a low level at power-up"
- note added: "INFO: (RESETN PIN) • Active-low hard Reset • Assert low to place the device in Reset state • Assert high to put the device in Normal state and move it out of Reset state • Connect to a host output that has default low at power-up; if the host output is tristated, add a 1 MΩ pull-down res"
- note added: "INFO: (SDIO_SPI_CFG) • Tie to VDDIO through a 1 MΩ resistor to enable the SPI interface • Tie to GND to enable the SDIO interface"
- note added: "INFO: (TEST MODE PIN) Test Mode – User must tie this pin to GND"
- note added: "INFO: Used only for development debug purposes; It is recommended to add test point for this pin"

Commit message: 97% drawing schematic is done
Parts:
- removed C1809: 4u7F_16V_X7R, Capacitor_SMD:C_0603_1608Metric, symbol _SCHLIB_Qcopter:CAP_CER_4.7uF_16V_X7R_C0603
- added ANT1801: 2.4GHz_2W_0.5dBi, RF_Antenna:Johanson_2450AT18x100, symbol _SCHLIB_Qcopter:ANT_2450AT18A100E_2.4GHz_2W_0.5dBi_SMD
- added C1809: 1uF_10V_X7R, Capacitor_SMD:C_0603_1608Metric, symbol _SCHLIB_Qcopter:CAP_CER_1uF_10V_X7R_C0603
- added C1818, C1819: 1p8F_50V_C0G, Capacitor_SMD:C_0201_0603Metric, symbol _SCHLIB_Qcopter:CAP_CER_1.8pF_50V_C0G_C0201
- added C1820, C1821, C1822: 1pF_50V_C0G, Capacitor_SMD:C_0201_0603Metric, symbol _SCHLIB_Qcopter:CAP_CER_1pF_50V_C0G_C0201
- added FB1801, FB1802, FB1803, FB1804: FB_550mA_0.19R, Inductor_SMD:L_0402_1005Metric, symbol _SCHLIB_Qcopter:IND_FB_BLM15AG121SN1D_550mA_0.19R_120R@100MHz_L0402
- added L1801: 2u2H_350mA_0.55R, Inductor_SMD:L_0402_1005Metric, symbol _SCHLIB_Qcopter:IND_2.2uH_350mA_0.55R_L0402
- added L1802: 15nH_560mA_0.172R, Inductor_SMD:L_0402_1005Metric, symbol _SCHLIB_Qcopter:IND_15nH_560mA_0.172R_3.28GHz_L0402
- added L1803, L1804: 3n3H_400mA_0.3R, Inductor_SMD:L_0201_0603Metric, symbol _SCHLIB_Qcopter:IND_3.3nH_400mA_0.3R_9.5GHz_L0201
- added L1805: 2n7H_300mA_0.17R, Inductor_SMD:L_0402_1005Metric, symbol _SCHLIB_Qcopter:IND_2.7nH_300mA_0.17R_9.5GHz_L0402
- added L1806: 3n9H_300mA_0.22R, Inductor_SMD:L_0402_1005Metric, symbol _SCHLIB_Qcopter:IND_3.9nH_300mA_0.22R_7GHz_L0402
Connections:
- net ATWILC_+1.3V: now also FB1801.1, FB1802.1, FB1803.1, L1801.1; no longer C1812.1, C1813.1, C1814.1, C1815.1, U1801.2 (VDD_RF_RX_1V3), U1801.21 (VSW), U1801.3 (VDD_AMS_1V3), U1801.37 (VDD_SXDIG_1V3), U1801.38 (VDD_VCO_1V3), U1801.4 (VDD_RF_TX_1V3)
- net GND: now also C1809.2, C1821.1, L1804.2, L1805.2
- net at U1801.7 (RFIOP): now also C1818.1
- net at U1801.8 (RFION): now also C1819.2
- net +PWR renamed +PWR_+3.3V
- net +PWR_+3.3V: no longer C1804.1, C1805.1, C1806.1, U1801.20 (VBATT_BUCK_3V3), U1801.5 (VDD_BATT_PPA_3V3), U1801.6 (VDD_BATT_PA_3V3)
- new net: C1809.1, C1814.1, C1815.1, FB1801.2, U1801.2 (VDD_RF_RX_1V3), U1801.38 (VDD_VCO_1V3), U1801.4 (VDD_RF_TX_1V3)
- new net: C1812.1, C1813.1, FB1802.2, U1801.3 (VDD_AMS_1V3), U1801.37 (VDD_SXDIG_1V3)
- new net: L1801.2, L1802.1
- new net: C1804.1, C1805.1, FB1804.2, U1801.5 (VDD_BATT_PPA_3V3), U1801.6 (VDD_BATT_PA_3V3)
- new net: C1806.1, FB1803.2, FB1804.1, U1801.20 (VBATT_BUCK_3V3)
- new net: C1820.2, C1822.1, L1803.1
- new net: C1819.1, C1821.2, L1803.2
- new net: C1818.2, C1820.1, L1804.1
- new net: C1822.2, L1805.1, L1806.2
- new net: ANT1801.1, L1806.1
- new net ATWILC_SW: L1802.2, U1801.21 (VSW)
Other:
- note added: "LAYOUT NOTE:"
- moved on the sheet: C1801, C1802, C1803, C1804, C1805, C1806, C1807, C1808, C1810, C1811, C1812, C1813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
