File: Hardware/_Sub_HW_Qcopter/v1_20240309/Design Folder/_Sub_HW_Qcopter/[05] - Power Supply .kicad_sch (KiCad schematic)
At the start: 0 parts

Commit message: Schematic is done by 90%
Parts:
- added C2201, C2202, C2203, C2204: 10uF_16V_X5R, Capacitor_SMD:C_0603_1608Metric, symbol _SCHLIB_Qcopter:CAP_CER_10uF_16V_X5R_C0603
- added LED2201, LED2202: ORANGE_2V_20mA, LED_SMD:LED_0603_1608Metric, symbol _SCHLIB_Qcopter:DIODE_LED_ORANGE_2V_20mA_611nm_LED0603
- added R2201, R2203: 100kR_1/10W_1%, Resistor_SMD:R_0603_1608Metric, symbol _SCHLIB_Qcopter:RES_100kR_1/10W_1%_R0603
- added R2202, R2204: 470R_1/10W_1%, Resistor_SMD:R_0603_1608Metric, symbol _SCHLIB_Qcopter:RES_470R_1/10W_1%_R0603
- added U2203: TLV70313DBVR, Package_TO_SOT_SMD:SOT-23-5, symbol _SCHLIB_Qcopter:IC_PMIC_TLV70313DBVR_LDO_1.3V_0.3A_SOT-23-5
- added U2204: TLV70328DBVR, Package_TO_SOT_SMD:SOT-23-5, symbol _SCHLIB_Qcopter:IC_PMIC_TLV70328DBVR_LDO_2.8V_0.3A_SOT-23-5
Connections:
- new net: LED2202.2, R2204.2
- new net: LED2201.2, R2202.2
- new net +1V3OUT: C2202.1, R2202.1, U2203.5 (VOUT)
- new net +2V8OUT: C2204.1, R2204.1, U2204.5 (VOUT)
- new net +5VDC: C2201.1, C2203.1, R2201.1, R2203.1, U2203.1 (VIN), U2203.3 (EN), U2204.1 (VIN), U2204.3 (EN)
- new net GND: C2201.2, C2202.2, C2203.2, C2204.2, LED2201.1, LED2202.1, R2201.2, R2203.2, U2203.2 (GND), U2204.2 (GND)
- no-connect marks 0 -> 2
Other:
- added sheet BATTERY CHARGER ([020301] - BATTERY CHARGER.kicad_sch)
- added sheet LDO +3V3 ([020303] - LDO +3V3.kicad_sch)
- added sheet SMPS DCDC-BOOST +5V ([020302] - SMPS DCDC-BOOST +5V.kicad_sch)
- note added: "LAYOUT NOTE:"

Commit message: 97% drawing schematic is done
Parts:
- added F2101: 4A_8V_2mR, Fuse:Fuse_0805_2012Metric, symbol _SCHLIB_Qcopter:FUSE_PTC_PTSLR08058V400_4A_8A_8V_F0805
- added J2101: HDR_1X2_5A_THD-RA, Connector_PinHeader_2.54mm:PinHeader_1x02_P2.54mm_Horizontal, symbol _SCHLIB_Qcopter:CONN_HDR_1X2_5A_RA_THD-2.54MM
- added JP2101: JP_2POS, Jumper:SolderJumper-2_P1.3mm_Open_TrianglePad1.0x1.5mm, symbol _SCHLIB_Qcopter:MECH_JUMPER_2POS_J1015
Connections:
- net +5VDC: no longer R2201.1, R2203.1, U2203.3 (EN), U2204.3 (EN)
- net +VBAT: now also JP2101.1
- net GND: now also J2101.1
- new net: F2101.1, J2101.2, JP2101.2
- new net EN_+1V3: R2201.1, U2203.3 (EN)
- new net EN_+2V8: R2203.1, U2204.3 (EN)
- new net VM: F2101.2
Other:
- note added: "DESIGN NOTE:"
