File: Hardware/_Sub_HW_Qcopter/v1_20240309/Design Folder/_Sub_HW_Qcopter/[0301] - MCU Driver.kicad_sch (KiCad schematic)
At the start: 0 parts

Commit message: Schematic is done by 90%
Parts:
- added C501, C503, C505, C509, C511, C512, C513, C519, C521, C523, C526: 1uF_10V_X7R, Capacitor_SMD:C_0603_1608Metric, symbol _SCHLIB_Qcopter:CAP_CER_1uF_10V_X7R_C0603
- added C502, C504, C506, C520, C522, C524, C527: 100nF_16V_X7R, Capacitor_SMD:C_0603_1608Metric, symbol _SCHLIB_Qcopter:CAP_CER_100nF_16V_X7R_C0603
- added C514, C515: 4u7F_16V_X7R, Capacitor_SMD:C_0603_1608Metric, symbol _SCHLIB_Qcopter:CAP_CER_4.7uF_16V_X7R_C0603
- added C517, C518: 12pF_50V_C0G, Capacitor_SMD:C_0603_1608Metric, symbol _SCHLIB_Qcopter:CAP_CER_12pF_50V_C0G_C0603
- added C525: 10nF_100V_X7R, Capacitor_SMD:C_0603_1608Metric, symbol _SCHLIB_Qcopter:CAP_CER_10nF_100V_X7R_C0603
- added J501: HDR_1X3_THD-1.27MM, Connector_PinHeader_1.27mm:PinHeader_1x03_P1.27mm_Vertical, symbol _SCHLIB_Qcopter:CONN_HDR_1X3_VERT_THD-1.27MM
- added JP501: JP_2POS, Jumper:SolderJumper-2_P1.3mm_Open_TrianglePad1.0x1.5mm, symbol _SCHLIB_Qcopter:MECH_JUMPER_2POS_J1015
- added L501: 2u2H_1.3A_156mOhm, Resistor_SMD:R_0805_2012Metric, symbol _SCHLIB_Qcopter:IND_2.2uH_1.3A_156mOhm_40MHz_L0805
- added LED501: RED_2V_20mA, LED_SMD:LED_0603_1608Metric, symbol _SCHLIB_Qcopter:DIODE_LED_RED_2V_20mA_624nm_LED0603
- added R501, R503, R505, R506, R507: 10kR_1/10W_1%, Resistor_SMD:R_0603_1608Metric, symbol _SCHLIB_Qcopter:RES_10kR_1/10W_1%_R0603
- added R502: 1kR_1/10W_1%, Resistor_SMD:R_0603_1608Metric, symbol _SCHLIB_Qcopter:RES_1kR_1/10W_1%_R0603
- added U501: STM32U575VIT6Q, Package_QFP:LQFP-100_14x14mm_P0.5mm, symbol _SCHLIB_Qcopter:IC_EMBD_STM32U575VIT6Q_MCU_ARM® Cortex®-M33_160MHz_2MB_100-LQFP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
- added X501: 16MHz_12pF_10ppm, Crystal:Crystal_SMD_2016-4Pin_2.0x1.6mm, symbol _SCHLIB_Qcopter:XTAL_ECS-160-12-37B-CTN-TR_16MHz_12pF_4SMD-1206
Connections:
- new net: LED501.2, R502.2
- new net ADC_A0: U501.15 (PC0)
- new net DCMI_D0: U501.63 (PC6)
- new net DCMI_D1: U501.64 (PC7)
- new net DCMI_D2: U501.65 (PC8)
- new net DCMI_D3: U501.66 (PC9)
- new net DCMI_D4: U501.3 (PE4)
- new net DCMI_D5: U501.84 (PD3)
- new net DCMI_D6: U501.4 (PE5)
- new net DCMI_D7: U501.5 (PE6)
- new net DCMI_D8: U501.78 (PC10)
- new net DCMI_D9: U501.80 (PC12)
- new net DCMI_HSYNC: U501.28 (PA4)
- new net DCMI_PIXCLK: U501.30 (PA6)
- new net DCMI_VSYNC: U501.93 (PB7)
- new net DCMI_XLCK: U501.22 (PA0)
- new net GND: C501.2, C502.2, C503.2, C504.2, C505.2, C506.2, C509.2, C511.2, C512.2, C513.2, C514.2, C515.2, C517.2, C518.2, C519.2, C520.2, C521.2, C522.2, C523.2, C524.2, C525.2, C526.2, C527.2, J501.1, LED501.1, R501.2, U501.10 (VSS), U501.19 (VSSA), U501.26 (VSS), U501.48 (VSSSMPS), U501.50 (VSS), U501.74 (VSS), U501.99 (VSS), X501.2, X501.4
- new net I2C1_SCL: R505.2, U501.92 (PB6)
- new net I2C1_SDA: R503.2, U501.89 (PB3)
- new net I2C2_SCL: R506.2, U501.44 (PB10)
- new net I2C2_SDA: R507.2, U501.45 (PB11)
- new net ICM_INT: U501.90 (PB4)
- new net LPUART1_RX: U501.25 (PA3)
- new net LPUART1_TX: U501.24 (PA2)
- new net MCU_NRST: U501.14 (NRST)
- new net OTG_USB_DM: U501.70 (PA11)
- new net OTG_USB_DP: U501.71 (PA12)
- new net OTG_USB_ID: U501.69 (PA10)
- new net PWR: C501.1, C502.1, C503.1, C504.1, C505.1, C506.1, C514.1, C515.1, C519.1, C520.1, C521.1, C522.1, C523.1, C524.1, C525.1, C526.1, C527.1, JP501.1, R503.1, R505.1, R506.1, R507.1, U501.100 (VDD), U501.11 (VDD), U501.20 (VREF+), U501.21 (VDDA), U501.27 (VDD), U501.46 (VLXSMPS), U501.51 (VDD), U501.6 (VBAT), U501.73 (VDDUSB), U501.75 (VDD)
- new net QSPI_CLK: U501.38 (PE10)
- new net QSPI_D0: U501.16 (PC1)
- new net QSPI_D1: U501.17 (PC2)
- new net QSPI_D2: U501.18 (PC3)
- new net QSPI_D3: U501.88 (PD7)
- new net QSPI_NSS: U501.39 (PE11)
- new net SPI_CLK: U501.23 (PA1)
- new net SPI_MISO: U501.42 (PE14)
- new net SPI_MOSI: U501.43 (PE15)
- new net SPI_NSS: U501.40 (PE12)
- new net STM32U5_BOOT0: JP501.2, R501.1, U501.94 (PH3-BOOT0)
- new net STM32U5_LED_IND: R502.1, U501.97 (PE0)
- new net STM32U5_OSC_I: C518.1, U501.12 (PH0-OSC_IN), X501.3
- new net STM32U5_OSC_O: C517.1, U501.13 (PH1-OSC_OUT), X501.1
- new net STM32U5_SWCLK: J501.2
- new net STM32U5_SWDIO: J501.3
- new net STM32U5_VDD11: C509.1, C511.1, C512.1, C513.1, L501.1, U501.49 (VDD11), U501.98 (VDD11)
- new net STM32U5_VDDSMPS: L501.2, U501.47 (VDDSMPS)
- new net TIM3_CH1: U501.2 (PE3)
- new net TIM3_CH2: U501.31 (PA7)
- new net TIM3_CH3: U501.32 (PB0)
- new net TIM3_CH4: U501.33 (PB1)
- new net USART2_RX: U501.77 (PA15)
- new net USART2_TX: U501.86 (PD5)
- no-connect marks 0 -> 34
Other:
- note added: "I2C Pull-up Resistors"
- note added: "PROG HDR"

Commit message: Schematic draft is done
Parts:
- removed LED501: RED_2V_20mA, LED_SMD:LED_0603_1608Metric, symbol _SCHLIB_Qcopter:DIODE_LED_RED_2V_20mA_624nm_LED0603
- added LED502: WHITE_3V2_420mcd, LED_SMD:LED_0603_1608Metric, symbol _SCHLIB_Qcopter:DIODE_LED_WHITE_3.2V_20mA_420mcd_LED0603
Connections:
- net GND: now also LED502.1
- net at R502.2: now also LED502.2
Changed lines of the file:
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@@
-	)
-	(symbol
-		(lib_id "_SCHLIB_Qcopter:DIODE_LED_RED_2V_20mA_624nm_LED0603")
-		(at 355.6 297.18 0)
-		(unit 1)
-		(exclude_from_sim no)
-		(in_bom yes)
-		(on_board yes)
-		(dnp no)
-		(property "Reference" "LED501"
-			(at 371.856 295.656 0)
-			(effects
-				(font
-					(size 1.27 1.27)
-				)
-			)
-		)
-		(property "Value" "RED_2V_20mA"
-			(at 348.742 295.91 0)
-			(effects
-				(font
-					(size 1.27 1.27)
-				)
-			)
-		)
-		(property "Footprint" "LED_SMD:LED_0603_1608Metric"
-			(at 359.41 279.4 0)
-			(effects
-				(font
-					(size 1.27 1.27)
-				)
-				(justify left)
-				(hide yes)
-			)
-		)
-		(property "Datasheet" "https://mm.digikey.com/Volume0/opasdata/d220001/medias/docus/3777/B1931USD-20D000814U1930.pdf"
-			(at 359.156 287.02 0)
-			(effects
-				(font
-					(size 1.27 1.27)
-				)
-				(justify left)
-				(hide yes)
-			)
-		)
-		(property "Description" "Red 624nm LED Indication - Discrete 2V 0603 (1608 Metric)"
-			(at 359.156 282.194 0)
-			(effects
-				(font
-					(size 1.27 1.27)
-				)
-				(justify left)
-				(hide yes)
-			)
-		)
-		(property "Package" "LED0603"
-			(at 351.536 298.704 0)
-			(effects
-				(font
-					(size 1.27 1.27)
-				)
-			)
-		)
-		(property "Part Number (Manufacturer)" "B1931USD-20D000814U1930"
-			(at 359.41 276.606 0)
-			(effects
-				(font
-					(size 1.27 1.27)
-				)
-				(justify left)
-				(hide yes)
-			)
-		)
-		(property "Manufacturer" "Harvatek Corporation"
-			(at 359.41 271.78 0)
-			(effects
-				(font
-					(size 1.27 1.27)
-				)
-				(justify left)
-				(hide yes)
-			)
-		)
-		(property "Part Number (Vendor)" "3147-B1931USD-20D000814U1930TR-ND"
-			(at 359.41 274.066 0)
-			(effects
-				(font
-					(size 1.27 1.27)
-				)
-				(justify left)
-				(hide yes)
-			)
-		)
-		(property "Vendor" "Digikey"
-			(at 359.41 269.24 0)
-			(effects
-				(font
-					(size 1.27 1.27)
-				)
-				(justify left)
-				(hide yes)
-			)
-		)
-		(property "Purchase Link" "https://www.digikey.ca/en/products/detail/harvatek-corporation/B1931USD-20D000814U1930/15861265"
-			(at 359.156 284.48 0)
-			(effects
-				(font
-					(size 1.27 1.27)
-				)
-				(justify left)
-				(hide yes)
-			)
-		)
-		(property "SCH CHECK" "SCH (N/A)"
-			(at 373.634 298.704 0)
-			(effects
-				(font
-					(size 1.27 1.27)
-				)
-			)
-		)
-		(property "PCB CHECK" "PCB (N/A)"
-			(at 373.634 301.244 0)
-			(effects
-				(font
-					(size 1.27 1.27)
-				)
-			)
-		)
-		(pin "2"
-		)
-		(pin "1"
-		)
-		(instances
-			(project "_Sub_HW_Qcopter"
-				(path "/b8703f06-b3da-4de2-b217-f104939b36e8/6184e84e-040e-4878-8152-76cf0b949e21/e826979f-4a88-401c-bba5-a1c30231907a/4eee3e1d-9a89-4293-ad66-a6ef408897f9"
-					(reference "LED501")
-					(unit 1)
-				)
-			)
-		)
 	)
 	(symbol
@@
 					(unit 1)
 				)
+			)
+		)
+	)
+	(symbol
+		(lib_id "_SCHLIB_Qcopter:DIODE_LED_WHITE_3.2V_20mA_420mcd_LED0603")
+		(at 355.6 297.18 0)
+		(unit 1)
+		(exclude_from_sim no)
+		(in_bom yes)
+		(on_board yes)
+		(dnp no)
+		(property "Reference" "LED502"
+			(at 371.856 295.91 0)
+			(effects
+				(font
+					(size 1.27 1.27)
+				)
+			)
+		)
+		(property "Value" "WHITE_3V2_420mcd"
+			(at 346.71 295.91 0)
+			(effects
+				(font
+					(size 1.27 1.27)
+				)
+			)
+		)
+		(property "Footprint" "LED_SMD:LED_0603_1608Metric"
+			(at 359.41 277.622 0)
+			(effects
+				(font
+					(size 1.27 1.27)
+				)
+				(justify left)
+				(hide yes)
+			)
+		)
+		(property "Datasheet" "https://mm.digikey.com/Volume0/opasdata/d220001/medias/docus/3694/B1931TW--20P000314U1930.pdf"
+			(at 359.156 285.242 0)
+			(effects
+				(font
+					(size 1.27 1.27)
+				)
+				(justify left)
+				(hide yes)
+			)
+		)
+		(property "Description" "White LED Indication - Discrete 3.2V 0603 (1608 Metric)"
+			(at 359.156 280.416 0)
+			(effects
+				(font
+					(size 1.27 1.27)
+				)
+				(justify left)
+				(hide yes)
+			)
+		)
+		(property "Package" "LED0603"
+			(at 351.79 298.704 0)
+			(effects
+				(font
+					(size 1.27 1.27)
+				)
+			)
+		)
+		(property "Part Number (Manufacturer)" "B1931TW--20P000314U1930"
+			(at 359.41 274.828 0)
+			(effects
+				(font
+					(size 1.27 1.27)
+				)
+				(justify left)
+				(hide yes)
+			)
+		)
+		(property "Manufacturer" "Harvatek Corporation"
+			(at 359.41 270.002 0)
+			(effects
+				(font
+					(size 1.27 1.27)
+				)
+				(justify left)
+				(hide yes)
+			)
+		)
+		(property "Part Number (Vendor)" "3147-B1931TW--20P000314U1930TR-ND"
+			(at 359.41 272.288 0)
+			(effects
+				(font
+					(size 1.27 1.27)
+				)
+				(justify left)
+				(hide yes)
+			)
+		)
+		(property "Vendor" "Digikey"
+			(at 359.41 267.462 0)
+			(effects
+				(font
+					(size 1.27 1.27)
+				)
+				(justify left)
+				(hide yes)
+			)
+		)
+		(property "Purchase Link" "https://www.digikey.ca/en/products/detail/harvatek-corporation/B1931TW-20P000314U1930/14302790"
+			(at 359.156 282.702 0)
+			(effects
+				(font
+					(size 1.27 1.27)
+				)
+				(justify left)
+				(hide yes)
+			)
+		)
+		(property "SCH CHECK" "SCH (N/A)"
+			(at 373.38 298.704 0)
+			(effects
+				(font
+					(size 1.27 1.27)
+				)
+			)
+		)
+		(property "PCB CHECK" "PCB (N/A)"
+			(at 373.38 301.244 0)
+			(effects
+				(font
+					(size 1.27 1.27)
+				)
+			)
+		)
+		(pin "2"
+		)
+		(pin "1"
+		)
+		(instances
+			(project "_Sub_HW_Qcopter"
+				(path "/b8703f06-b3da-4de2-b217-f104939b36e8/6184e84e-040e-4878-8152-76cf0b949e21/e826979f-4a88-401c-bba5-a1c30231907a/4eee3e1d-9a89-4293-ad66-a6ef408897f9"
+					(reference "LED502")
+					(unit 1)
+				)
