File: Hardware/_Sub_HW_Qcopter/v1_20240309/Design Folder/_Sub_HW_Qcopter/[0401] - STM32WLE5 Driver.kicad_sch (KiCad schematic)
At the start: 0 parts

Commit message: Schematic is done by 90%
Parts:
- added C1501, C1504, C1506: 100nF_16V_X7R, Capacitor_SMD:C_0603_1608Metric, symbol _SCHLIB_Qcopter:CAP_CER_100nF_16V_X7R_C0603
- added C1502, C1503, C1505: 1uF_10V_X7R, Capacitor_SMD:C_0603_1608Metric, symbol _SCHLIB_Qcopter:CAP_CER_1uF_10V_X7R_C0603
- added JP1501: JP_2POS, Jumper:SolderJumper-2_P1.3mm_Open_TrianglePad1.0x1.5mm, symbol _SCHLIB_Qcopter:MECH_JUMPER_2POS_J1015
- added R1501: 10kR_1/10W_1%, Resistor_SMD:R_0603_1608Metric, symbol _SCHLIB_Qcopter:RES_10kR_1/10W_1%_R0603
- added U1501: STM32WLE5CCU7, Package_DFN_QFN:QFN-48-1EP_7x7mm_P0.5mm_EP5.6x5.6mm_ThermalVias, symbol _SCHLIB_Qcopter:IC_EMBD_STM32WLE5CCU7_MCU_LoRa_LoRaWAN1.0_SigFox_48-UFQFPN (7x7)
Connections:
- new net: JP1501.2, R1501.1, U1501.19 (PH3-BOOT0)
- new net +PWR: C1501.1, C1502.1, C1503.1, C1504.1, C1505.1, C1506.1, JP1501.1, U1501.11 (VDD), U1501.37 (VBAT), U1501.41 (VDDA), U1501.44 (VDD)
- new net ATWILC_CHIPN: U1501.8 (PA1)
- new net ATWILC_IRQN: U1501.42 (PA14)
- new net ATWILC_RESETN: U1501.7 (PA0)
- new net ATWILC_WAKEUP: U1501.36 (PA13)
- new net GND: C1501.2, C1502.2, C1503.2, C1504.2, C1505.2, C1506.2, R1501.2, U1501.49 (EP)
- new net STM32WLE5_I2C2_SCL: U1501.35 (PA12)
- new net STM32WLE5_I2C2_SDA: U1501.43 (PA15)
- new net STM32WLE5_LPUART1_RX: U1501.10 (PA3)
- new net STM32WLE5_LPUART1_TX: U1501.9 (PA2)
- new net STM32WLE5_NRESET: U1501.18 (NRST)
- new net STM32WLE5_PWM_CH1: U1501.15 (PA7)
- new net STM32WLE5_PWM_CH2: U1501.17 (PA9)
- new net STM32WLE5_PWM_CH3: U1501.34 (PA11)
- new net STM32WLE5_SPI2_MISO: U1501.13 (PA5)
- new net STM32WLE5_SPI2_MOSI: U1501.33 (PA10)
- new net STM32WLE5_SPI2_NSS: U1501.32 (PB12)
- new net STM32WLE5_SPI2_SCK: U1501.16 (PA8)
- new net STM32WLE5_SPI_MISO: U1501.2 (PB4)
- new net STM32WLE5_SPI_MOSI: U1501.3 (PB5)
- new net STM32WLE5_SPI_NSS: U1501.12 (PA4)
- new net STM32WLE5_SPI_SCK: U1501.1 (PB3)
- new net STM32WLE5_UART1_RX: U1501.5 (PB7)
- new net STM32WLE5_UART1_TX: U1501.4 (PB6)
- no-connect marks 0 -> 5

Commit message: 97% drawing schematic is done
Parts:
- added C1507, C1508: 10pF_50V_C0G, Capacitor_SMD:C_0603_1608Metric, symbol _SCHLIB_Qcopter:CAP_CER_10pF_50V_C0G_C0603
- added J1501: HDR_1X3_THD-1.27MM, Connector_PinHeader_1.27mm:PinHeader_1x03_P1.27mm_Vertical, symbol _SCHLIB_Qcopter:CONN_HDR_1X3_VERT_THD-1.27MM
- added X1501: 32MHz_10pF_10ppm, footrpring, symbol _SCHLIB_Qcopter:XTAL_CS06465-32M_32MHz_10pF_4-SMD (2.0X1.6)
Connections:
- net +PWR: now also U1501.25 (VDDPA), U1501.46 (VDDSMPS)
- net GND: now also C1507.2, C1508.2, J1501.1, X1501.2, X1501.4
- net FE_CTRL1: now reaches U1501.14 (PA6)
- net STM32WLE5_RFIP: now reaches U1501.20 (RFI_P)
- net STM32WLE5_RFIN: now reaches U1501.21 (RFI_N)
- net STM32WLE5_RFOLP: now reaches U1501.22 (RFO_LP)
- net STM32WLE5_RFOHP: now reaches U1501.23 (RFO_HP)
- net STM32WLE5_VRPA: now reaches U1501.24 (VR_PA)
- net STM32WLE5_OSC-IN: now reaches U1501.26 (OSC_IN)
- net STM32WLE5_OSC-IN: now also C1507.1, X1501.1
- net STM32WLE5_OSC-OUT: now reaches U1501.27 (OSC_OUT)
- net STM32WLE5_OSC-OUT: now also C1508.1, X1501.3
- net STM32WLE5_+1.55V: now reaches U1501.29 (VDDRF1V55)
- net STM32WLE5_+1.55V: now also U1501.45 (VFBSMPS)
- net FE_CTRL2: now reaches U1501.31 (PB2)
- net FE_CTRL3: now reaches U1501.6 (PB8)
- new net STM32WLE5_SWCLK: J1501.2
- new net STM32WLE5_SWDIO: J1501.3
- no-connect marks 5 -> 2
Other:
- note added: "MAKE SURE ABOUT THE CORRECT MCU AS IT HAS A BT AND LOAR THING!!!"
- note added: "PROG HDR"

Commit message: Schematic draft is done
Parts:
- added C1509: 470nF_16V_X7R, Capacitor_SMD:C_0603_1608Metric, symbol _SCHLIB_Qcopter:CAP_CER_470nF_16V_X7R_C0603
- added C1510: 100nF_16V_X7R, Capacitor_SMD:C_0603_1608Metric, symbol _SCHLIB_Qcopter:CAP_CER_100nF_16V_X7R_C0603
- added C1511: 4u7F_16V_X7R, Capacitor_SMD:C_0603_1608Metric, symbol _SCHLIB_Qcopter:CAP_CER_4.7uF_16V_X7R_C0603
- added L1501: 15uH_250mA_0.95Ohm, Inductor_SMD:L_0805_2012Metric, symbol _SCHLIB_Qcopter:IND_15uH_250mA_0.95Ohm_40MHz_L0805
- added LED1501: WHITE_3V2_420mcd, LED_SMD:LED_0603_1608Metric, symbol _SCHLIB_Qcopter:DIODE_LED_WHITE_3.2V_20mA_420mcd_LED0603
- added R1502: 470R_1/10W_1%, Resistor_SMD:R_0603_1608Metric, symbol _SCHLIB_Qcopter:RES_470R_1/10W_1%_R0603
- added U1502: NX3L1T3157GMZ, footrpring, symbol _SCHLIB_Qcopter:IC_SWITCH_NX3L1T3157GMZ_SPDT_1C_900mR_6-XSON
Connections:
- net STM32WLE5_SWCLK is gone; now on net ATWILC_IRQN: J1501.2
- net STM32WLE5_SWDIO is gone; now on net ATWILC_WAKEUP: J1501.3
- net +PWR: now also U1502.5 (VCC); no longer U1501.25 (VDDPA), U1501.46 (VDDSMPS)
- net FE_CTRL1: now also U1502.6 (S)
- net GND: now also U1501.48 (VSSSMPS), C1509.2, C1510.2, C1511.2, LED1501.1, U1502.2 (GND)
- net STM32WLE5_+1.55V: now also C1509.1, L1501.2, U1502.1 (Y1)
- net STM32WLE5_VDDRF: now reaches U1501.28 (VDDRF)
- net STM32WLE5_VDDRF: now also U1501.46 (VDDSMPS), C1510.1, C1511.1, U1502.3 (Y0)
- net LED_INDC: now reaches U1501.38 (PC13)
- net LED_INDC: now also R1502.1
- net STM32WLE5_VLXSMPS: now reaches U1501.47 (VLXSMPS)
- net STM32WLE5_VLXSMPS: now also L1501.1
- new net: LED1501.2, R1502.2
- new net STM32WLE5_VDDPA: U1501.25 (VDDPA), U1502.4 (Z)
Other:
- note added: "INFO:"
- note removed: "MAKE SURE ABOUT THE CORRECT MCU AS IT HAS A BT AND LOAR THING!!!"
- moved on the sheet: C1501, C1502, C1503, C1504, C1505, C1506, J1501
