File: Hardware/_Sub_HW_Qcopter/v1_20240309/Design Folder/_Sub_HW_Qcopter/[0404] - Antenna Driver.kicad_sch (KiCad schematic)
At the start: 0 parts

Commit message: 97% drawing schematic is done
Parts:
- added C1701, C1705, C1709, C1712: 33pF_50V_C0G, Capacitor_SMD:C_0402_1005Metric, symbol _SCHLIB_Qcopter:CAP_CER_33pF_50V_C0G_C0402
- added C1702, C1715: 5p6F_50V_C0G, Capacitor_SMD:C_0402_1005Metric, symbol _SCHLIB_Qcopter:CAP_CER_5.6pF_50V_C0G_C0402
- added C1703, C1710, C1711: 3p3F_50V_C0G, Capacitor_SMD:C_0402_1005Metric, symbol _SCHLIB_Qcopter:CAP_CER_3.3pF_50V_C0G_C0402
- added C1704, C1707: 2p7F_50V_C0G, Capacitor_SMD:C_0402_1005Metric, symbol _SCHLIB_Qcopter:CAP_CER_2.7pF_50V_C0G_C0402
- added C1706: 1p3F_50V_C0G, Capacitor_SMD:C_0402_1005Metric, symbol _SCHLIB_Qcopter:CAP_CER_1.3pF_50V_C0G_C0402
- added C1708: 3p6F_50V_C0G, Capacitor_SMD:C_0402_1005Metric, symbol _SCHLIB_Qcopter:CAP_CER_3.6pF_50V_C0G_C0402
- added C1713, C1719: 68pF_50V_C0G, Capacitor_SMD:C_0402_1005Metric, symbol _SCHLIB_Qcopter:CAP_CER_68pF_50V_C0G_C0402
- added C1714, C1717, C1720: 1p2F_50V_C0G, Capacitor_SMD:C_0402_1005Metric, symbol _SCHLIB_Qcopter:CAP_CER_1.2pF_50V_C0G_C0402
- added C1716: 2p2F_50V_C0G, Capacitor_SMD:C_0402_1005Metric, symbol _SCHLIB_Qcopter:CAP_CER_2.2pF_50V_C0G_C0402
- added C1718: 47nF_25V_X7R, Capacitor_SMD:C_0402_1005Metric, symbol _SCHLIB_Qcopter:CAP_CER_47nF_25V_X7R_C0402
- added C1721, C1722, C1723: 1nF_50V_X7R, Capacitor_SMD:C_0603_1608Metric, symbol _SCHLIB_Qcopter:CAP_CER_1nF_50V_X7R_C0603
- added J1701: RECEPT_RF_50R, footrpring, symbol _SCHLIB_Qcopter:CONN_RECEPT_RF_50R_6GHz_UMCC
- added L1701: 47nH_210mA_1.08Ohm, Inductor_SMD:L_0402_1005Metric, symbol _SCHLIB_Qcopter:IND_47nH_210mA_1.08Ohm_L0402
- added L1702: 3n3H_2A_30mOhm, Inductor_SMD:L_0402_1005Metric, symbol _SCHLIB_Qcopter:IND_3.3nH_2A_30mR_14GHz_L0402
- added L1703: 3nH_750mA_70mOhm, Inductor_SMD:L_0402_1005Metric, symbol _SCHLIB_Qcopter:IND_3nH_750mA_70mOhm_15GHz_L0402
- added L1704, L1706, L1709: 8n7H_540mA_0.14R, Inductor_SMD:L_0402_1005Metric, symbol _SCHLIB_Qcopter:IND_8.7nH_540mA_0.14R_5.5GHz_L0402
- added L1705: 11nH_500mA_0.14R, Inductor_SMD:L_0402_1005Metric, symbol _SCHLIB_Qcopter:IND_11nH_500mA_0.14R_5.5GHz_L0402
- added L1707: 33nH_260mA_0.63Ohm, Inductor_SMD:L_0402_1005Metric, symbol _SCHLIB_Qcopter:IND_33nH_260mA_3.2GHz_0.63Ohm_L0402
- added L1708: 3n6H_900mA_40mOhm, Inductor_SMD:L_0402_1005Metric, symbol _SCHLIB_Qcopter:IND_3.6nH_900mA_40mOhm_9.5GHz_L0402
- added R1701: 0R_1/16W, Resistor_SMD:R_0402_1005Metric, symbol _SCHLIB_Qcopter:RES_0R_1/16W_R0402
- added R1702, R1703, R1704: 100R_1/10W_1%, Resistor_SMD:R_0603_1608Metric, symbol _SCHLIB_Qcopter:RES_100R_1/10W_1%_R0603
- added U1701: NX3L1T3157GMZ, footrpring, symbol _SCHLIB_Qcopter:IC_SWITCH_NX3L1T3157GMZ_SPDT_1C_900mR_6-XSON
- added U1702: BGS13SN8E6327XTSA1, footrpring, symbol _SCHLIB_Qcopter:IC_SWITCH_BGS13SN8E6327XTSA1_SP3T_1C_6GHz_PG-TSNP-8-1
Connections:
- new net: C1702.1, C1704.1, L1701.2, L1702.2, L1703.1
- new net: C1703.1, C1704.2, C1705.1, L1703.2
- new net: C1709.2, C1710.1, L1706.1
- new net: C1711.1, J1701.1 (SIG), L1706.2
- new net: C1722.1, R1703.2, U1702.2 (V2)
- new net: C1712.1, L1707.1, U1701.3 (Y0)
- new net: C1716.1, C1717.1, L1707.2, L1708.1, R1701.2
- new net: C1713.1, C1715.1, C1716.2, L1708.2
- new net: C1721.1, R1702.2, U1702.1 (VDD)
- new net: C1723.1, R1704.2, U1702.3 (V1)
- new net: C1706.1, L1704.2, U1702.4 (RF3)
- new net: C1708.2, U1702.5 (RF1)
- new net: C1709.1, U1702.6 (RFin)
- new net: C1714.1, L1709.2, U1702.7 (RF2)
- new net: C1705.2, L1704.1
- new net: C1713.2, L1709.1
- new net: C1701.1, L1701.1, U1701.1 (Y1)
- new net FE_CTRL1: R1704.1, U1701.6 (S)
- new net FE_CTRL2: R1703.1
- new net FE_CTRL3: R1702.1
- new net GND: C1701.2, C1702.2, C1703.2, C1706.2, C1707.2, C1710.2, C1711.2, C1712.2, C1714.2, C1715.2, C1717.2, C1718.2, C1719.2, C1720.2, C1721.2, C1722.2, C1723.2, J1701.2 (GND), U1701.2 (GND), U1702.8 (DGND)
- new net RFI_N: C1707.1, L1705.2
- new net RFI_P: C1708.1, L1705.1
- new net RFO_HP: R1701.1
- new net RFO_LP: L1702.1
- new net VR_PA: C1718.1, C1719.1, C1720.1, U1701.4 (Z)

Commit message: Schematic draft is done
Other:
- note added: "INFO:"
