File: Hardware/_Sub_HW_Qcopter/v1_20240309/Design Folder/_Sub_HW_Qcopter/[020303] - LDO +3V3.kicad_sch (KiCad schematic)
At the start: 6 parts, among them U3801 TLV74033PDBVR

Commit message: Update [020303] - LDO +3V3.kicad_sch
Parts:
- renumbered C3801 to C3401, C3602 to C3402, LED3801 to LED3401, R3801 to R3401, R3802 to R3402, U3801 to U3401
Other:
- company: (none) -> Mend0z0
- title: (none) -> Quadcopter
Changed lines of the file:
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@@
 	(paper "C")
 	(title_block
-		(comment 2 "DRAFT")
+		(title "Quadcopter")
+		(date "2024-03-17")
+		(rev "01")
+		(company "Mend0z0")
+		(comment 1 "01")
+		(comment 2 "PRELIMINARY")
+		(comment 3 "Siavash Taher Parvar")
+		(comment 8 "N/A")
+		(comment 9 "First Version")
 	)
 	(junction
@@
 		)
 	)
-	(hierarchical_label "GND"
-		(shape passive)
-		(at 165.1 226.06 180)
-		(fields_autoplaced yes)
-		(effects
-			(font
-				(size 1.27 1.27)
-			)
-			(justify right)
-		)
-	)
 	(symbol
 		(lib_id "_SCHLIB_Qcopter:CAP_CER_10uF_16V_X5R_C0603")
@@
 		(dnp no)
 		(fields_autoplaced yes)
-		(property "Reference" "C3602"
+		(property "Reference" "C3402"
 			(at 294.64 196.8499 90)
 			(effects
@@
 			(project "_Sub_HW_Qcopter"
 				(path "/b8703f06-b3da-4de2-b217-f104939b36e8/6184e84e-040e-4878-8152-76cf0b949e21/0ce565c6-f8fe-4174-9716-15fae563dcc2/f68d8295-72fb-4a7a-82e7-db0d0a2f4ced"
-					(reference "C3602")
-					(unit 1)
-				)
-				(path "/b8703f06-b3da-4de2-b217-f104939b36e8/6184e84e-040e-4878-8152-76cf0b949e21/0ce565c6-f8fe-4174-9716-15fae563dcc2/c687d90c-2ade-43f2-9366-cfff9c79456b"
-					(reference "C3603")
-					(unit 1)
-				)
-				(path "/b8703f06-b3da-4de2-b217-f104939b36e8/6184e84e-040e-4878-8152-76cf0b949e21/0ce565c6-f8fe-4174-9716-15fae563dcc2/89c85fef-530b-4b8e-8624-d86fb53e17b7"
-					(reference "C1302")
-					(unit 1)
-				)
-				(path "/b8703f06-b3da-4de2-b217-f104939b36e8/6184e84e-040e-4878-8152-76cf0b949e21/0ce565c6-f8fe-4174-9716-15fae563dcc2/ccf78d53-405f-4cbf-a00f-81329b3705d6"
-					(reference "C3803")
+					(reference "C3402")
 					(unit 1)
 				)
@@
 		(dnp no)
 		(fields_autoplaced yes)
-		(property "Reference" "R3801"
+		(property "Reference" "R3401"
 			(at 215.9 204.4699 90)
 			(effects
@@
 			(project "_Sub_HW_Qcopter"
 				(path "/b8703f06-b3da-4de2-b217-f104939b36e8/6184e84e-040e-4878-8152-76cf0b949e21/0ce565c6-f8fe-4174-9716-15fae563dcc2/f68d8295-72fb-4a7a-82e7-db0d0a2f4ced"
-					(reference "R3801")
-					(unit 1)
-				)
-				(path "/b8703f06-b3da-4de2-b217-f104939b36e8/6184e84e-040e-4878-8152-76cf0b949e21/0ce565c6-f8fe-4174-9716-15fae563dcc2/c687d90c-2ade-43f2-9366-cfff9c79456b"
-					(reference "R3601")
-					(unit 1)
-				)
-				(path "/b8703f06-b3da-4de2-b217-f104939b36e8/6184e84e-040e-4878-8152-76cf0b949e21/0ce565c6-f8fe-4174-9716-15fae563dcc2/89c85fef-530b-4b8e-8624-d86fb53e17b7"
-					(reference "R1301")
-					(unit 1)
-				)
-				(path "/b8703f06-b3da-4de2-b217-f104939b36e8/6184e84e-040e-4878-8152-76cf0b949e21/0ce565c6-f8fe-4174-9716-15fae563dcc2/ccf78d53-405f-4cbf-a00f-81329b3705d6"
-					(reference "R3803")
+					(reference "R3401")
 					(unit 1)
 				)
@@
 		(dnp no)
 		(fields_autoplaced yes)
-		(property "Reference" "C3801"
+		(property "Reference" "C3401"
 			(at 180.34 204.4699 90)
 			(effects
@@
 			(project "_Sub_HW_Qcopter"
 				(path "/b8703f06-b3da-4de2-b217-f104939b36e8/6184e84e-040e-4878-8152-76cf0b949e21/0ce565c6-f8fe-4174-9716-15fae563dcc2/f68d8295-72fb-4a7a-82e7-db0d0a2f4ced"
-					(reference "C3801")
-					(unit 1)
-				)
-				(path "/b8703f06-b3da-4de2-b217-f104939b36e8/6184e84e-040e-4878-8152-76cf0b949e21/0ce565c6-f8fe-4174-9716-15fae563dcc2/c687d90c-2ade-43f2-9366-cfff9c79456b"
-					(reference "C3601")
-					(unit 1)
-				)
-				(path "/b8703f06-b3da-4de2-b217-f104939b36e8/6184e84e-040e-4878-8152-76cf0b949e21/0ce565c6-f8fe-4174-9716-15fae563dcc2/89c85fef-530b-4b8e-8624-d86fb53e17b7"
-					(reference "C1301")
-					(unit 1)
-				)
-				(path "/b8703f06-b3da-4de2-b217-f104939b36e8/6184e84e-040e-4878-8152-76cf0b949e21/0ce565c6-f8fe-4174-9716-15fae563dcc2/ccf78d53-405f-4cbf-a00f-81329b3705d6"
-					(reference "C3802")
+					(reference "C3401")
 					(unit 1)
 				)
@@
 		(dnp no)
 		(fields_autoplaced yes)
-		(property "Reference" "LED3801"
+		(property "Reference" "LED3401"
 			(at 335.28 212.6614 90)
 			(effects
@@
 			(project "_Sub_HW_Qcopter"
 				(path "/b8703f06-b3da-4de2-b217-f104939b36e8/6184e84e-040e-4878-8152-76cf0b949e21/0ce565c6-f8fe-4174-9716-15fae563dcc2/f68d8295-72fb-4a7a-82e7-db0d0a2f4ced"
-					(reference "LED3801")
-					(unit 1)
-				)
-				(path "/b8703f06-b3da-4de2-b217-f104939b36e8/6184e84e-040e-4878-8152-76cf0b949e21/0ce565c6-f8fe-4174-9716-15fae563dcc2/c687d90c-2ade-43f2-9366-cfff9c79456b"
-					(reference "LED3601")
-					(unit 1)
-				)
-				(path "/b8703f06-b3da-4de2-b217-f104939b36e8/6184e84e-040e-4878-8152-76cf0b949e21/0ce565c6-f8fe-4174-9716-15fae563dcc2/89c85fef-530b-4b8e-8624-d86fb53e17b7"
-					(reference "LED1301")
-					(unit 1)
-				)
-				(path "/b8703f06-b3da-4de2-b217-f104939b36e8/6184e84e-040e-4878-8152-76cf0b949e21/0ce565c6-f8fe-4174-9716-15fae563dcc2/ccf78d53-405f-4cbf-a00f-81329b3705d6"
-					(reference "LED3802")
+					(reference "LED3401")
 					(unit 1)
 				)
@@
 		(dnp no)
 		(fields_autoplaced yes)
-		(property "Reference" "R3802"
+		(property "Reference" "R3402"
 			(at 332.74 196.8499 90)
 			(effects
@@
 			(project "_Sub_HW_Qcopter"
 				(path "/b8703f06-b3da-4de2-b217-f104939b36e8/6184e84e-040e-4878-8152-76cf0b949e21/0ce565c6-f8fe-4174-9716-15fae563dcc2/f68d8295-72fb-4a7a-82e7-db0d0a2f4ced"
-					(reference "R3802")
+					(reference "R3402")
 					(unit 1)
 				)
-				(path "/b8703f06-b3da-4de2-b217-f104939b36e8/6184e84e-040e-4878-8152-76cf0b949e21/0ce565c6-f8fe-4174-9716-15fae563dcc2/c687d90c-2ade-43f2-9366-cfff9c79456b"
-					(reference "R3602")
-					(unit 1)
-				)
-				(path "/b8703f06-b3da-4de2-b217-f104939b36e8/6184e84e-040e-4878-8152-76cf0b949e21/0ce565c6-f8fe-4174-9716-15fae563dcc2/89c85fef-530b-4b8e-8624-d86fb53e17b7"
-					(reference "R1302")
-					(unit 1)
-				)
-				(path "/b8703f06-b3da-4de2-b217-f104939b36e8/6184e84e-040e-4878-8152-76cf0b949e21/0ce565c6-f8fe-4174-9716-15fae563dcc2/ccf78d53-405f-4cbf-a00f-81329b3705d6"
-					(reference "R3804")
+			)
+		)
+	)
+	(symbol
+		(lib_id "power:GND")
+		(at 165.1 226.06 270)
+		(unit 1)
+		(exclude_from_sim no)
+		(in_bom yes)
+		(on_board yes)
+		(dnp no)
+		(fields_autoplaced yes)
+		(property "Reference" "#PWR03401"
+			(at 158.75 226.06 0)
+			(effects
+				(font
+					(size 1.27 1.27)
+				)
+				(hide yes)
+			)
+		)
+		(property "Value" "GND"
+			(at 161.29 226.0599 90)
+			(effects
+				(font
+					(size 1.27 1.27)
+				)
+				(justify right)
+			)
+		)
+		(property "Footprint" ""
+			(at 165.1 226.06 0)
+			(effects
+				(font
+					(size 1.27 1.27)
+				)
+				(hide yes)
+			)
+		)
+		(property "Datasheet" ""
+			(at 165.1 226.06 0)
+			(effects
+				(font
+					(size 1.27 1.27)
+				)
+				(hide yes)
+			)
+		)
+		(property "Description" "Power symbol creates a global label with name \"GND\" , ground"
+			(at 165.1 226.06 0)
+			(effects
+				(font
+					(size 1.27 1.27)
+				)
+				(hide yes)
+			)
+		)
+		(pin "1"
+		)
+		(instances
+			(project "_Sub_HW_Qcopter"
+				(path "/b8703f06-b3da-4de2-b217-f104939b36e8/6184e84e-040e-4878-8152-76cf0b949e21/0ce565c6-f8fe-4174-9716-15fae563dcc2/f68d8295-72fb-4a7a-82e7-db0d0a2f4ced"
+					(reference "#PWR03401")
 					(unit 1)
 				)
@@
 		(dnp no)
 		(fields_autoplaced yes)
-		(property "Reference" "U3801"
+		(property "Reference" "U3401"
 			(at 255.27 177.8 0)
 			(effects
@@
 			(project "_Sub_HW_Qcopter"
 				(path "/b8703f06-b3da-4de2-b217-f104939b36e8/6184e84e-040e-4878-8152-76cf0b949e21/0ce565c6-f8fe-4174-9716-15fae563dcc2/f68d8295-72fb-4a7a-82e7-db0d0a2f4ced"
-					(reference "U3801")
+					(reference "U3401")
 					(unit 1)
 				)
-				(path "/b8703f06-b3da-4de2-b217-f104939b36e8/6184e84e-040e-4878-8152-76cf0b949e21/0ce565c6-f8fe-4174-9716-15fae563dcc2/c687d90c-2ade-43f2-9366-cfff9c79456b"
-					(reference "U3601")
-					(unit 1)
-				)
-				(path "/b8703f06-b3da-4de2-b217-f104939b36e8/6184e84e-040e-4878-8152-76cf0b949e21/0ce565c6-f8fe-4174-9716-15fae563dcc2/89c85fef-530b-4b8e-8624-d86fb53e17b7"
-					(reference "U1301")
-					(unit 1)
-				)
-				(path "/b8703f06-b3da-4de2-b217-f104939b36e8/6184e84e-040e-4878-8152-76cf0b949e21/0ce565c6-f8fe-4174-9716-15fae563dcc2/ccf78d53-405f-4cbf-a00f-81329b3705d6"
-					(reference "U3802")
-					(unit 1)
-				)
