File: Hardware/_Sub_HW_Qcopter/v1_20240309/Design Folder/_Sub_HW_Qcopter/[03] - MECHANICAL PARTS.kicad_sch (KiCad schematic)
At the start: 0 parts

Commit message: 97% drawing schematic is done
Changed lines of the file:
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@@
 		(comment 2 "DRAFT")
 	)
-	(text_box "4xLED 5MM BLUE\n4xLED HOLDER BLACK 5MM\n\n1 m WIRE\n4xJST 1.27mm FEMALE HEADER\n\n1xBATTERY 3.7V\n\n\n1xFRAME\n4xCORELESS MOTORS 0716\n4xM3x3MM STAND OFF\n4xM3 PHILLIPS SCREW\n4xM3 NUTS\n\n1xPCB 50x50 MM2 4LAYERs IMPEDANCE CONTROLLED\n\n\n1x OV2640 CAMERA MODULE \n\n\n4x mounting holes"
+	(text_box "4xLED 5MM BLUE\n4xLED HOLDER BLACK 5MM\n\n1 m WIRE\n4xJST 1.27mm FEMALE HEADER\n\n1xBATTERY 3.7V\n\n\n1xFRAME\n4xCORELESS MOTORS 0716\n4xpropeller\n4xM3x3MM STAND OFF\n4xM3 PHILLIPS SCREW\n4xM3 NUTS\n\n1xPCB 50x50 MM2 4LAYERs IMPEDANCE CONTROLLED\n\n\n1x OV2640 CAMERA MODULE \n\n\n4x mounting holes"
 		(exclude_from_sim no)
 		(at 121.92 130.81 0)

Commit message: Update [03] - MECHANICAL PARTS.kicad_sch
Parts:
- added FD3801, FD3802, FD3803, FD3804: ~, Fiducial:Fiducial_0.5mm_Mask1mm, symbol _SCHLIB_Qcopter:MECH_FD
- added MH3801, MH3802, MH3803, MH3804: M3, MountingHole:MountingHole_3.2mm_M3_DIN965_Pad_TopBottom, symbol _SCHLIB_Qcopter:MECH_MH_M3
- added TXT3801: ~, _PCBLIB_Qcopter:LOGO_Mend0z0, symbol _SCHLIB_Qcopter:MECH_LOGO
Connections:
- new net GND: MH3801.1, MH3802.1, MH3803.1, MH3804.1
Other:
- company: (none) -> Mend0z0
- title: (none) -> Quadcopter
