File: Hardware/_Sub_HW_Qcopter/v1_20240309/Design Folder/_Sub_HW_Qcopter/[020104] - GPIO Expander.kicad_sch (KiCad schematic)
At the start: 0 parts

Commit message: Update [020104] - GPIO Expander.kicad_sch
Other:
- note added: "CHECKED"
Changed lines of the file:
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@@
 	(title_block
 		(title "Quadcopter")
-		(date "2024-03-17")
+		(date "2024-03-18")
 		(rev "01")
 		(company "Mend0z0")
 		(comment 1 "01")
-		(comment 2 "PRELIMINARY")
+		(comment 2 "CHECKED")
 		(comment 3 "Siavash Taher Parvar")
 		(comment 8 "N/A")
@@
 		)
 	)
+	(text "CHECKED"
+		(exclude_from_sim no)
+		(at 167.386 167.64 0)
+		(effects
+			(font
+				(size 1.905 1.905)
+				(thickness 0.381)
+				(bold yes)
+			)
+		)
+	)
 	(text "GROUP 3"
 		(exclude_from_sim no)
@@
 		)
 	)
+	(text "CHECKED"
+		(exclude_from_sim no)
+		(at 345.186 167.64 0)
+		(effects
+			(font
+				(size 1.905 1.905)
+				(thickness 0.381)
+				(bold yes)
+			)
+		)
+	)
 	(text "GROUP 2"
 		(exclude_from_sim no)
@@
 			)
 		)
+	)
+	(text "CHECKED"
+		(exclude_from_sim no)
+		(at 256.794 167.386 0)
+		(effects
+			(font
+				(size 1.905 1.905)
+				(thickness 0.381)
+				(bold yes)
+			)
+		)
