File: Hardware/_Sub_HW_Qcopter/v1_20240309/Design Folder/_Sub_HW_Qcopter/[020103] - Battery Voltage Sampler.kicad_sch (KiCad schematic)
At the start: 6 parts, among them U801 MCP6006T-E/OT

Commit message: Update [020103] - Battery Voltage Sampler.kicad_sch
Other:
- note added: "INFO:"
Changed lines of the file:
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@@
 	(title_block
 		(title "Quadcopter")
-		(date "2024-03-17")
+		(date "2024-03-18")
 		(rev "01")
 		(company "Mend0z0")
 		(comment 1 "01")
-		(comment 2 "PRELIMINARY")
+		(comment 2 "CHECKED")
 		(comment 3 "Siavash Taher Parvar")
 		(comment 8 "N/A")
@@
 		)
 	)
+	(polyline
+		(pts
+			(xy 199.39 176.53) (xy 203.2 181.61)
+		)
+		(stroke
+			(width 0)
+			(type default)
+		)
+	)
 	(wire
 		(pts
@@
 			(width 0)
 			(type default)
+		)
+	)
+	(rectangle
+		(start 201.93 182.88)
+		(end 204.47 185.42)
+		(stroke
+			(width 0)
+			(type default)
+		)
+		(fill
+			(type none)
+		)
+	)
+	(text_box "\n\nAny input value would be divided by two. As a result the 3.7v battery voltage would be 1.85v once it's fully charged"
+		(exclude_from_sim no)
+		(at 172.72 162.56 0)
+		(size 25.4 16.51)
+		(stroke
+			(width 0)
+			(type default)
+		)
+		(fill
+			(type none)
+		)
+		(effects
+			(font
+				(size 1.27 1.27)
+			)
+			(justify left top)
+		)
+	)
+	(text "INFO:"
+		(exclude_from_sim no)
+		(at 177.292 165.354 0)
+		(effects
+			(font
+				(size 1.905 1.905)
+				(thickness 0.381)
+				(bold yes)
+			)
 		)
 	)
@@
 	)
 	(hierarchical_label "PWR"
-		(shape passive)
+		(shape input)
 		(at 234.95 187.96 180)
 		(fields_autoplaced yes)

Commit message: Update [020103] - Battery Voltage Sampler.kicad_sch
Parts:
- C801, R801, R802, R803, R804, U801: SCH CHECK SCH (N/A) -> SCH (CHECKED)
Changed lines of the file:
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@@
 			)
 		)
-		(property "SCH CHECK" "SCH (N/A)"
+		(property "SCH CHECK" "SCH (CHECKED)"
 			(at 289.306 156.464 0)
 			(effects
@@
 			)
 		)
-		(property "SCH CHECK" "SCH (N/A)"
+		(property "SCH CHECK" "SCH (CHECKED)"
 			(at 320.04 193.0399 90)
 			(effects
@@
 			)
 		)
-		(property "SCH CHECK" "SCH (N/A)"
+		(property "SCH CHECK" "SCH (CHECKED)"
 			(at 205.74 199.3899 90)
 			(effects
@@
 			)
 		)
-		(property "SCH CHECK" "SCH (N/A)"
+		(property "SCH CHECK" "SCH (CHECKED)"
 			(at 243.84 199.3899 90)
 			(effects
@@
 			)
 		)
-		(property "SCH CHECK" "SCH (N/A)"
+		(property "SCH CHECK" "SCH (CHECKED)"
 			(at 195.58 185.674 0)
 			(effects
@@
 			)
 		)
-		(property "SCH CHECK" "SCH (N/A)"
+		(property "SCH CHECK" "SCH (CHECKED)"
 			(at 278.765 172.72 0)
 			(effects
