File: Hardware/_Sub_HW_Qcopter/v1_20240309/Design Folder/_Sub_HW_Qcopter/[020105] - ICM-20948 Driver.kicad_sch (KiCad schematic)
At the start: 7 parts, among them U1301 ICM-20948

Commit message: Update [020105] - ICM-20948 Driver.kicad_sch
Parts:
- C1301, C1302, C1303, R1301, R1302, R1303, U1301: SCH CHECK SCH (N/A) -> SCH (CHECKED)
Changed lines of the file:
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@@
 			)
 		)
-		(property "SCH CHECK" "SCH (N/A)"
+		(property "SCH CHECK" "SCH (CHECKED)"
 			(at 194.31 161.2899 90)
 			(effects
@@
 			)
 		)
-		(property "SCH CHECK" "SCH (N/A)"
+		(property "SCH CHECK" "SCH (CHECKED)"
 			(at 261.62 165.1 0)
 			(effects
@@
 			)
 		)
-		(property "SCH CHECK" "SCH (N/A)"
+		(property "SCH CHECK" "SCH (CHECKED)"
 			(at 226.314 186.69 0)
 			(effects
@@
 			)
 		)
-		(property "SCH CHECK" "SCH (N/A)"
+		(property "SCH CHECK" "SCH (CHECKED)"
 			(at 218.44 161.2899 90)
 			(effects
@@
 			)
 		)
-		(property "SCH CHECK" "SCH (N/A)"
+		(property "SCH CHECK" "SCH (CHECKED)"
 			(at 182.88 208.2799 90)
 			(effects
@@
 			)
 		)
-		(property "SCH CHECK" "SCH (N/A)"
+		(property "SCH CHECK" "SCH (CHECKED)"
 			(at 204.47 208.2799 90)
 			(effects
@@
 			)
 		)
-		(property "SCH CHECK" "SCH (N/A)"
+		(property "SCH CHECK" "SCH (CHECKED)"
 			(at 224.79 208.2799 90)
 			(effects
