File: Hardware/_Sub_HW_Qcopter/v1_20240309/Design Folder/_Sub_HW_Qcopter/[020107] - LEDs Driver.kicad_sch (KiCad schematic)
At the start: 4 parts

Commit message: Update [020107] - LEDs Driver.kicad_sch
Parts:
- LED1501, LED1502, R1501, R1502: SCH CHECK SCH (N/A) -> SCH (CHECKED)
Changed lines of the file:
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@@
 			)
 		)
-		(property "SCH CHECK" "SCH (N/A)"
+		(property "SCH CHECK" "SCH (CHECKED)"
 			(at 264.414 204.724 0)
 			(effects
@@
 			)
 		)
-		(property "SCH CHECK" "SCH (N/A)"
+		(property "SCH CHECK" "SCH (CHECKED)"
 			(at 264.414 242.824 0)
 			(effects
@@
 			)
 		)
-		(property "SCH CHECK" "SCH (N/A)"
+		(property "SCH CHECK" "SCH (CHECKED)"
 			(at 280.67 254.5714 90)
 			(effects
@@
 			)
 		)
-		(property "SCH CHECK" "SCH (N/A)"
+		(property "SCH CHECK" "SCH (CHECKED)"
 			(at 280.67 216.4714 90)
 			(effects
