File: Hardware/_Sub_HW_Qcopter/v1_20240309/Design Folder/_Sub_HW_Qcopter/[02011001] - DRV8837 Driver.kicad_sch (KiCad schematic)
At the start: 5 parts, among them U2301 SN74LVC1G18DCKR, U2302 DRV8837CDSGR

Commit message: Update [02011001] - DRV8837 Driver.kicad_sch
Parts:
- C2301, C2302, C2303, U2301, U2302: SCH CHECK SCH (N/A) -> SCH (CHECKED)
Connections:
- net GND: now also U2302.9 (GND)
Other:
- moved on the sheet: C2302
Changed lines of the file:
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@@
 	)
 	(junction
-		(at 266.7 199.39)
+		(at 266.7 196.85)
 		(diameter 0)
 		(color 0 0 0 0)
 	)
 	(junction
-		(at 266.7 223.52)
+		(at 287.02 201.93)
+		(diameter 0)
+		(color 0 0 0 0)
+	)
+	(junction
+		(at 266.7 215.9)
 		(diameter 0)
 		(color 0 0 0 0)
@@
 		)
 	)
-	(wire
-		(pts
-			(xy 290.83 199.39) (xy 266.7 199.39)
-		)
-		(stroke
-			(width 0)
-			(type default)
-		)
-	)
 	(polyline
 		(pts
@@
 	(wire
 		(pts
-			(xy 254 199.39) (xy 266.7 199.39)
+			(xy 254 196.85) (xy 266.7 196.85)
 		)
 		(stroke
@@
 	(wire
 		(pts
-			(xy 266.7 223.52) (xy 266.7 215.9)
+			(xy 290.83 199.39) (xy 287.02 199.39)
+		)
+		(stroke
+			(width 0)
+			(type default)
+		)
+	)
+	(wire
+		(pts
+			(xy 266.7 215.9) (xy 266.7 213.36)
+		)
+		(stroke
+			(width 0)
+			(type default)
+		)
+	)
+	(wire
+		(pts
+			(xy 287.02 199.39) (xy 287.02 201.93)
 		)
 		(stroke
@@
 		)
 	)
+	(wire
+		(pts
+			(xy 290.83 196.85) (xy 266.7 196.85)
+		)
+		(stroke
+			(width 0)
+			(type default)
+		)
+	)
 	(polyline
 		(pts
@@
 	(wire
 		(pts
-			(xy 255.27 223.52) (xy 266.7 223.52)
+			(xy 255.27 215.9) (xy 266.7 215.9)
 		)
 		(stroke
@@
 		)
 	)
-	(wire
-		(pts
-			(xy 266.7 199.39) (xy 266.7 203.2)
-		)
-		(stroke
-			(width 0)
-			(type default)
-		)
-	)
 	(polyline
 		(pts
@@
 	(wire
 		(pts
-			(xy 287.02 223.52) (xy 266.7 223.52)
+			(xy 287.02 215.9) (xy 266.7 215.9)
 		)
 		(stroke
@@
 		)
 	)
+	(wire
+		(pts
+			(xy 266.7 196.85) (xy 266.7 200.66)
+		)
+		(stroke
+			(width 0)
+			(type default)
+		)
+	)
 	(polyline
 		(pts
@@
 	(wire
 		(pts
-			(xy 287.02 201.93) (xy 287.02 223.52)
+			(xy 287.02 201.93) (xy 287.02 215.9)
 		)
 		(stroke
@@
 	)
 	(label "PWR"
-		(at 254 199.39 0)
+		(at 254 196.85 0)
 		(fields_autoplaced yes)
 		(effects
@@
 	(symbol
 		(lib_id "power:GND")
-		(at 255.27 223.52 270)
+		(at 255.27 215.9 270)
 		(unit 1)
 		(exclude_from_sim no)
@@
 		(fields_autoplaced yes)
 		(property "Reference" "#PWR02302"
-			(at 248.92 223.52 0)
+			(at 248.92 215.9 0)
 			(effects
 				(font
@@
 		)
 		(property "Value" "GND"
-			(at 251.46 223.5199 90)
+			(at 251.46 215.8999 90)
 			(effects
 				(font
@@
 		)
 		(property "Footprint" ""
-			(at 255.27 223.52 0)
+			(at 255.27 215.9 0)
 			(effects
 				(font
@@
 		)
 		(property "Datasheet" ""
-			(at 255.27 223.52 0)
+			(at 255.27 215.9 0)
 			(effects
 				(font
@@
 		)
 		(property "Description" "Power symbol creates a global label with name \"GND\" , ground"
-			(at 255.27 223.52 0)
+			(at 255.27 215.9 0)
 			(effects
 				(font
@@
 			)
 		)
-		(property "SCH CHECK" "SCH (N/A)"
+		(property "SCH CHECK" "SCH (CHECKED)"
 			(at 213.36 181.61 0)
 			(effects
@@
 			)
 		)
-		(property "SCH CHECK" "SCH (N/A)"
+		(property "SCH CHECK" "SCH (CHECKED)"
 			(at 345.44 176.5299 90)
 			(effects
@@
 			)
 		)
-		(property "SCH CHECK" "SCH (N/A)"
+		(property "SCH CHECK" "SCH (CHECKED)"
 			(at 180.34 212.0899 90)
 			(effects
@@
 	(symbol
 		(lib_id "_SCHLIB_Qcopter:CAP_CER_100nF_16V_X7R_C0603")
-		(at 266.7 203.2 270)
+		(at 266.7 200.66 270)
 		(unit 1)
 		(exclude_from_sim no)
@@
 		(fields_autoplaced yes)
 		(property "Reference" "C2302"
-			(at 269.24 204.4699 90)
+			(at 269.24 201.9299 90)
 			(effects
 				(font
@@
 		)
 		(property "Value" "100nF_16V_X7R"
-			(at 269.24 207.0099 90)
+			(at 269.24 204.4699 90)
 			(effects
 				(font
@@
 		)
 		(property "Footprint" "Capacitor_SMD:C_0603_1608Metric"
-			(at 284.988 206.756 0)
+			(at 284.988 204.216 0)
 			(effects
 				(font
@@
 		)
 		(property "Datasheet" "https://mm.digikey.com/Volume0/opasdata/d220001/medias/docus/609/CL10B104KO8NNNC_Spec.pdf"
-			(at 276.606 206.502 0)
+			(at 276.606 203.962 0)
 			(effects
 				(font
@@
 		)
 		(property "Description" "0.1 µF ±10% 16V Ceramic Capacitor X7R 0603 (1608 Metric)"
-			(at 282.194 206.756 0)
+			(at 282.194 204.216 0)
 			(effects
 				(font
@@
 		)
 		(property "Package" "C0603"
-			(at 269.24 209.5499 90)
+			(at 269.24 207.0099 90)
 			(effects
 				(font
@@
 		)
 		(property "Part Number (Manufacturer)" "CL10B104KO8NNNC"
-			(at 287.528 206.756 0)
+			(at 287.528 204.216 0)
 			(effects
 				(font
@@
 		)
 		(property "Manufacturer" "Samsung Electro-Mechanics"
-			(at 292.862 206.756 0)
+			(at 292.862 204.216 0)
 			(effects
 				(font
@@
 		)
 		(property "Part Number (Vendor)" "1276-1005-2-ND"
-			(at 290.068 206.756 0)
+			(at 290.068 204.216 0)
 			(effects
 				(font
@@
 		)
 		(property "Vendor" "Digikey"
-			(at 295.402 206.756 0)
+			(at 295.402 204.216 0)
 			(effects
 				(font
@@
 		)
 		(property "Purchase Link" "https://www.digikey.ca/en/products/detail/samsung-electro-mechanics/CL10B104KO8NNNC/3886663"
-			(at 279.4 206.502 0)
+			(at 279.4 203.962 0)
 			(effects
 				(font
@@
 			)
 		)
-		(property "SCH CHECK" "SCH (N/A)"
-			(at 269.24 212.0899 90)
+		(property "SCH CHECK" "SCH (CHECKED)"
+			(at 269.24 209.5499 90)
 			(effects
 				(font
@@
 		)
 		(property "PCB CHECK" "PCB (N/A)"
-			(at 269.24 214.6299 90)
+			(at 269.24 212.0899 90)
 			(effects
 				(font
@@
 			)
 		)
-		(property "SCH CHECK" "SCH (N/A)"
+		(property "SCH CHECK" "SCH (CHECKED)"
 			(at 304.8 179.07 0)
 			(effects
@@
 		(pin "6"
 		)
+		(pin "9"
+		)
 		(instances
