File: Hardware/_Sub_HW_Qcopter/v1_20240309/Design Folder/_Sub_HW_Qcopter/[020110] - Motor Driver.kicad_sch (KiCad schematic)
At the start: 7 parts, among them J2201 HDR_1X2_5A_THD-RA, J2202 HDR_1X2_VERT_1.25MM, J2203 HDR_1X2_VERT_1.25MM, J2204 HDR_1X2_VERT_1.25MM, J2205 HDR_1X2_VERT_1.25MM

Commit message: Update [020110] - Motor Driver.kicad_sch
Other:
- note added: "CHECKED"
Changed lines of the file:
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@@
 	(title_block
 		(title "Quadcopter")
-		(date "2024-03-17")
+		(date "2024-03-18")
 		(rev "01")
 		(company "Mend0z0")
 		(comment 1 "01")
-		(comment 2 "PRELIMINARY")
+		(comment 2 "CHECKED")
 		(comment 3 "Siavash Taher Parvar")
 		(comment 8 "N/A")
@@
 		)
 	)
+	(text "CHECKED"
+		(exclude_from_sim no)
+		(at 253.492 206.502 0)
+		(effects
+			(font
+				(size 1.905 1.905)
+				(thickness 0.381)
+				(bold yes)
+			)
+		)
+	)
 	(text "DESIGN NOTE:"
 		(exclude_from_sim no)
@@
 		)
 	)
+	(text "CHECKED"
+		(exclude_from_sim no)
+		(at 254 130.556 0)
+		(effects
+			(font
+				(size 1.905 1.905)
+				(thickness 0.381)
+				(bold yes)
+			)
+		)
+	)
+	(text "CHECKED"
+		(exclude_from_sim no)
+		(at 254.762 181.102 0)
+		(effects
+			(font
+				(size 1.905 1.905)
+				(thickness 0.381)
+				(bold yes)
+			)
+		)
+	)
+	(text "CHECKED"
+		(exclude_from_sim no)
+		(at 254.254 155.956 0)
+		(effects
+			(font
+				(size 1.905 1.905)
+				(thickness 0.381)
+				(bold yes)
+			)
+		)
+	)

Commit message: Update [020110] - Motor Driver.kicad_sch
Parts:
- F2201, J2201, J2202, J2203, J2204, J2205, JP2201: SCH CHECK SCH (N/A) -> SCH (CHECKED)
Changed lines of the file:
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@@
 			)
 		)
-		(property "SCH CHECK" "SCH (N/A)"
+		(property "SCH CHECK" "SCH (CHECKED)"
 			(at 137.16 115.824 0)
 			(effects
@@
 			)
 		)
-		(property "SCH CHECK" "SCH (N/A)"
+		(property "SCH CHECK" "SCH (CHECKED)"
 			(at 306.07 137.1599 0)
 			(effects
@@
 			)
 		)
-		(property "SCH CHECK" "SCH (N/A)"
+		(property "SCH CHECK" "SCH (CHECKED)"
 			(at 140.716 154.178 0)
 			(effects
@@
 			)
 		)
-		(property "SCH CHECK" "SCH (N/A)"
+		(property "SCH CHECK" "SCH (CHECKED)"
 			(at 183.896 130.81 0)
 			(effects
@@
 			)
 		)
-		(property "SCH CHECK" "SCH (N/A)"
+		(property "SCH CHECK" "SCH (CHECKED)"
 			(at 306.07 162.5599 0)
 			(effects
@@
 			)
 		)
-		(property "SCH CHECK" "SCH (N/A)"
+		(property "SCH CHECK" "SCH (CHECKED)"
 			(at 306.07 187.9599 0)
 			(effects
@@
 			)
 		)
-		(property "SCH CHECK" "SCH (N/A)"
+		(property "SCH CHECK" "SCH (CHECKED)"
 			(at 306.07 213.3599 0)
 			(effects
