File: Hardware/_Sub_HW_Qcopter/v1_20240309/Design Folder/_Sub_HW_Qcopter/[020203] - Antenna Driver.kicad_sch (KiCad schematic)
At the start: 39 parts, among them J2901 RECEPT_RF_50R, U2901 NX3L1T3157GMZ, U2902 BGS13SN8E6327XTSA1

Commit message: Update [020203] - Antenna Driver.kicad_sch
Parts:
- C2901, C2902, C2903, C2904, C2905, C2906, C2907, C2908, C2909, C2910, C2911, C2912, C2913, C2914, C2915, C2916, C2917, C2918, C2919, C2920, C2921, C2922, C2923, J2901, L2901, L2902, L2903, L2904, L2905, L2906, L2907, L2908, L2909, R2901, R2902, R2903, R2904, U2901, U2902: SCH CHECK SCH (N/A) -> SCH (CHECKED)
Changed lines of the file:
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@@
 			)
 		)
-		(property "SCH CHECK" "SCH (N/A)"
+		(property "SCH CHECK" "SCH (CHECKED)"
 			(at 525.78 175.26 0)
 			(effects
@@
 			)
 		)
-		(property "SCH CHECK" "SCH (N/A)"
+		(property "SCH CHECK" "SCH (CHECKED)"
 			(at 66.04 195.5799 90)
 			(effects
@@
 			)
 		)
-		(property "SCH CHECK" "SCH (N/A)"
+		(property "SCH CHECK" "SCH (CHECKED)"
 			(at 216.916 174.244 0)
 			(effects
@@
 			)
 		)
-		(property "SCH CHECK" "SCH (N/A)"
+		(property "SCH CHECK" "SCH (CHECKED)"
 			(at 497.586 184.404 0)
 			(effects
@@
 			)
 		)
-		(property "SCH CHECK" "SCH (N/A)"
+		(property "SCH CHECK" "SCH (CHECKED)"
 			(at 325.374 293.624 0)
 			(effects
@@
 			)
 		)
-		(property "SCH CHECK" "SCH (N/A)"
+		(property "SCH CHECK" "SCH (CHECKED)"
 			(at 163.83 125.984 0)
 			(effects
@@
 			)
 		)
-		(property "SCH CHECK" "SCH (N/A)"
+		(property "SCH CHECK" "SCH (CHECKED)"
 			(at 27.94 195.5799 90)
 			(effects
@@
 			)
 		)
-		(property "SCH CHECK" "SCH (N/A)"
+		(property "SCH CHECK" "SCH (CHECKED)"
 			(at 341.63 306.0699 90)
 			(effects
@@
 			)
 		)
-		(property "SCH CHECK" "SCH (N/A)"
+		(property "SCH CHECK" "SCH (CHECKED)"
 			(at 220.726 115.57 0)
 			(effects
@@
 			)
 		)
-		(property "SCH CHECK" "SCH (N/A)"
+		(property "SCH CHECK" "SCH (CHECKED)"
 			(at 393.7 172.72 0)
 			(effects
@@
 			)
 		)
-		(property "SCH CHECK" "SCH (N/A)"
+		(property "SCH CHECK" "SCH (CHECKED)"
 			(at 331.216 187.198 0)
 			(effects
@@
 			)
 		)
-		(property "SCH CHECK" "SCH (N/A)"
+		(property "SCH CHECK" "SCH (CHECKED)"
 			(at 341.63 128.2699 90)
 			(effects
@@
 			)
 		)
-		(property "SCH CHECK" "SCH (N/A)"
+		(property "SCH CHECK" "SCH (CHECKED)"
 			(at 341.63 331.4699 90)
 			(effects
@@
 			)
 		)
-		(property "SCH CHECK" "SCH (N/A)"
+		(property "SCH CHECK" "SCH (CHECKED)"
 			(at 341.63 207.0099 90)
 			(effects
@@
 			)
 		)
-		(property "SCH CHECK" "SCH (N/A)"
+		(property "SCH CHECK" "SCH (CHECKED)"
 			(at 508 204.4699 90)
 			(effects
@@
 			)
 		)
-		(property "SCH CHECK" "SCH (N/A)"
+		(property "SCH CHECK" "SCH (CHECKED)"
 			(at 231.14 128.2699 90)
 			(effects
@@
 			)
 		)
-		(property "SCH CHECK" "SCH (N/A)"
+		(property "SCH CHECK" "SCH (CHECKED)"
 			(at 325.374 268.224 0)
 			(effects
@@
 			)
 		)
-		(property "SCH CHECK" "SCH (N/A)"
+		(property "SCH CHECK" "SCH (CHECKED)"
 			(at 123.19 140.9699 90)
 			(effects
@@
 			)
 		)
-		(property "SCH CHECK" "SCH (N/A)"
+		(property "SCH CHECK" "SCH (CHECKED)"
 			(at 341.63 280.6699 90)
 			(effects
@@
 			)
 		)
-		(property "SCH CHECK" "SCH (N/A)"
+		(property "SCH CHECK" "SCH (CHECKED)"
 			(at 240.03 207.0099 90)
 			(effects
@@
 			)
 		)
-		(property "SCH CHECK" "SCH (N/A)"
+		(property "SCH CHECK" "SCH (CHECKED)"
 			(at 125.73 293.3699 90)
 			(effects
@@
 			)
 		)
-		(property "SCH CHECK" "SCH (N/A)"
+		(property "SCH CHECK" "SCH (CHECKED)"
 			(at 179.07 255.778 0)
 			(effects
@@
 			)
 		)
-		(property "SCH CHECK" "SCH (N/A)"
+		(property "SCH CHECK" "SCH (CHECKED)"
 			(at 176.53 207.0099 90)
 			(effects
@@
 			)
 		)
-		(property "SCH CHECK" "SCH (N/A)"
+		(property "SCH CHECK" "SCH (CHECKED)"
 			(at 217.17 186.944 0)
 			(effects
@@
 			)
 		)
-		(property "SCH CHECK" "SCH (N/A)"
+		(property "SCH CHECK" "SCH (CHECKED)"
 			(at 322.326 116.078 0)
 			(effects
@@
 			)
 		)
-		(property "SCH CHECK" "SCH (N/A)"
+		(property "SCH CHECK" "SCH (CHECKED)"
 			(at 447.04 184.404 0)
 			(effects
@@
 			)
 		)
-		(property "SCH CHECK" "SCH (N/A)"
+		(property "SCH CHECK" "SCH (CHECKED)"
 			(at 325.374 319.024 0)
 			(effects
@@
 			)
 		)
-		(property "SCH CHECK" "SCH (N/A)"
+		(property "SCH CHECK" "SCH (CHECKED)"
 			(at 457.2 204.4699 90)
 			(effects
@@
 			)
 		)
-		(property "SCH CHECK" "SCH (N/A)"
+		(property "SCH CHECK" "SCH (CHECKED)"
 			(at 157.48 217.424 0)
 			(effects
@@
 			)
 		)
-		(property "SCH CHECK" "SCH (N/A)"
+		(property "SCH CHECK" "SCH (CHECKED)"
 			(at 280.416 186.944 0)
 			(effects
@@
 			)
 		)
-		(property "SCH CHECK" "SCH (N/A)"
+		(property "SCH CHECK" "SCH (CHECKED)"
 			(at 157.48 186.69 0)
 			(effects
@@
 			)
 		)
-		(property "SCH CHECK" "SCH (N/A)"
+		(property "SCH CHECK" "SCH (CHECKED)"
 			(at 180.34 128.2699 90)
 			(effects
@@
 			)
 		)
-		(property "SCH CHECK" "SCH (N/A)"
+		(property "SCH CHECK" "SCH (CHECKED)"
 			(at 46.99 195.5799 90)
 			(effects
@@
 			)
 		)
-		(property "SCH CHECK" "SCH (N/A)"
+		(property "SCH CHECK" "SCH (CHECKED)"
 			(at 163.83 116.078 0)
 			(effects
@@
 			)
 		)
-		(property "SCH CHECK" "SCH (N/A)"
+		(property "SCH CHECK" "SCH (CHECKED)"
 			(at 220.726 102.87 0)
 			(effects
@@
 			)
 		)
-		(property "SCH CHECK" "SCH (N/A)"
+		(property "SCH CHECK" "SCH (CHECKED)"
 			(at 87.63 170.18 0)
 			(effects
@@
 			)
 		)
-		(property "SCH CHECK" "SCH (N/A)"
+		(property "SCH CHECK" "SCH (CHECKED)"
 			(at 271.526 115.824 0)
 			(effects
@@
 			)
 		)
-		(property "SCH CHECK" "SCH (N/A)"
+		(property "SCH CHECK" "SCH (CHECKED)"
 			(at 124.46 267.9699 90)
 			(effects
@@
 			)
 		)
-		(property "SCH CHECK" "SCH (N/A)"
+		(property "SCH CHECK" "SCH (CHECKED)"
 			(at 116.84 199.3899 90)
 			(effects
