File: Hardware/_Sub_HW_Qcopter/v1_20240309/Design Folder/_Sub_HW_Qcopter/[020301] - BATTERY CHARGER.kicad_sch (KiCad schematic)
At the start: 11 parts, among them J3901 HDR_1X2_VERT_1.25MM, J3902 USB_MICRO B_RA, U3901 MCP73811T-420I/OT

Commit message: Update [020301] - BATTERY CHARGER.kicad_sch
Parts:
- J3201: renamed from J3902; footprint _PCBLIB_HotPlate:USB_Micro-B_Amphenol_10118194_Horizontal -> _PCBLIB_Qcopter:USB_Micro-B_Amphenol_10118194_Horizontal
- renumbered C3903 to C3201, C3901 to C3202, C3902 to C3203, D3901 to D3201, D3902 to D3202, D3903 to D3203, D3904 to D3204, J3901 to J3202, RV3901 to RV3201, U3901 to U3201
Other:
- company: (none) -> Mend0z0
- title: (none) -> Quadcopter
Changed lines of the file:
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@@
 	(paper "C")
 	(title_block
-		(comment 2 "DRAFT")
+		(title "Quadcopter")
+		(date "2024-03-17")
+		(rev "01")
+		(company "Mend0z0")
+		(comment 1 "01")
+		(comment 2 "PRELIMINARY")
+		(comment 3 "Siavash Taher Parvar")
+		(comment 8 "N/A")
+		(comment 9 "First Version")
 	)
 	(junction
@@
 	(wire
 		(pts
+			(xy 97.79 208.28) (xy 97.79 203.2)
+		)
+		(stroke
+			(width 0)
+			(type default)
+		)
+	)
+	(wire
+		(pts
 			(xy 279.4 185.42) (xy 269.24 185.42)
 		)
@@
 		(pts
 			(xy 109.22 190.5) (xy 109.22 203.2)
-		)
-		(stroke
-			(width 0)
-			(type default)
-		)
-	)
-	(wire
-		(pts
-			(xy 92.71 203.2) (xy 97.79 203.2)
 		)
 		(stroke
@@
 		)
 	)
-	(label "MCP_GND"
-		(at 270.51 203.2 0)
-		(fields_autoplaced yes)
-		(effects
-			(font
-				(size 1.27 1.27)
-			)
-			(justify left bottom)
-		)
-	)
 	(label "DP"
 		(at 110.49 185.42 0)
@@
 			)
 			(justify left)
-		)
-	)
-	(hierarchical_label "GND"
-		(shape passive)
-		(at 92.71 203.2 180)
-		(fields_autoplaced yes)
-		(effects
-			(font
-				(size 1.27 1.27)
-			)
-			(justify right)
 		)
 	)
@@
 		(dnp no)
 		(fields_autoplaced yes)
-		(property "Reference" "C3902"
+		(property "Reference" "C3203"
 			(at 326.39 186.6899 90)
 			(effects
@@
 			(project "_Sub_HW_Qcopter"
 				(path "/b8703f06-b3da-4de2-b217-f104939b36e8/6184e84e-040e-4878-8152-76cf0b949e21/0ce565c6-f8fe-4174-9716-15fae563dcc2/82e4bdd4-fd10-4d98-b6d8-ce5d864ae438"
-					(reference "C3902")
+					(reference "C3203")
 					(unit 1)
 				)
@@
 		(dnp no)
 		(fields_autoplaced yes)
-		(property "Reference" "D3904"
+		(property "Reference" "D3204"
 			(at 210.82 190.4999 90)
 			(effects
@@
 			(project "_Sub_HW_Qcopter"
 				(path "/b8703f06-b3da-4de2-b217-f104939b36e8/6184e84e-040e-4878-8152-76cf0b949e21/0ce565c6-f8fe-4174-9716-15fae563dcc2/82e4bdd4-fd10-4d98-b6d8-ce5d864ae438"
-					(reference "D3904")
+					(reference "D3204")
 					(unit 1)
 				)
@@
 		(dnp no)
 		(fields_autoplaced yes)
-		(property "Reference" "D3903"
+		(property "Reference" "D3203"
 			(at 173.99 190.4999 90)
 			(effects
@@
 			(project "_Sub_HW_Qcopter"
 				(path "/b8703f06-b3da-4de2-b217-f104939b36e8/6184e84e-040e-4878-8152-76cf0b949e21/0ce565c6-f8fe-4174-9716-15fae563dcc2/82e4bdd4-fd10-4d98-b6d8-ce5d864ae438"
-					(reference "D3903")
+					(reference "D3203")
 					(unit 1)
 				)
@@
 		(dnp no)
 		(fields_autoplaced yes)
-		(property "Reference" "U3901"
+		(property "Reference" "U3201"
 			(at 292.1 165.1 0)
 			(effects
@@
 			(project "_Sub_HW_Qcopter"
 				(path "/b8703f06-b3da-4de2-b217-f104939b36e8/6184e84e-040e-4878-8152-76cf0b949e21/0ce565c6-f8fe-4174-9716-15fae563dcc2/82e4bdd4-fd10-4d98-b6d8-ce5d864ae438"
-					(reference "U3901")
+					(reference "U3201")
 					(unit 1)
 				)
@@
 		(dnp no)
 		(fields_autoplaced yes)
-		(property "Reference" "D3902"
+		(property "Reference" "D3202"
 			(at 148.59 190.4999 90)
 			(effects
@@
 			(project "_Sub_HW_Qcopter"
 				(path "/b8703f06-b3da-4de2-b217-f104939b36e8/6184e84e-040e-4878-8152-76cf0b949e21/0ce565c6-f8fe-4174-9716-15fae563dcc2/82e4bdd4-fd10-4d98-b6d8-ce5d864ae438"
-					(reference "D3902")
+					(reference "D3202")
 					(unit 1)
 				)
@@
 		(dnp no)
 		(fields_autoplaced yes)
-		(property "Reference" "J3902"
+		(property "Reference" "J3201"
 			(at 97.79 165.1 0)
 			(effects
@@
 			)
 		)
-		(property "Footprint" "_PCBLIB_HotPlate:USB_Micro-B_Amphenol_10118194_Horizontal"
+		(property "Footprint" "_PCBLIB_Qcopter:USB_Micro-B_Amphenol_10118194_Horizontal"
 			(at 96.52 162.56 0)
 			(effects
@@
 			(project "_Sub_HW_Qcopter"
 				(path "/b8703f06-b3da-4de2-b217-f104939b36e8/6184e84e-040e-4878-8152-76cf0b949e21/0ce565c6-f8fe-4174-9716-15fae563dcc2/82e4bdd4-fd10-4d98-b6d8-ce5d864ae438"
-					(reference "J3902")
+					(reference "J3201")
 					(unit 1)
 				)
@@
 		(dnp no)
 		(fields_autoplaced yes)
-		(property "Reference" "D3901"
+		(property "Reference" "D3201"
 			(at 123.19 190.4999 90)
 			(effects
@@
 			(project "_Sub_HW_Qcopter"
 				(path "/b8703f06-b3da-4de2-b217-f104939b36e8/6184e84e-040e-4878-8152-76cf0b949e21/0ce565c6-f8fe-4174-9716-15fae563dcc2/82e4bdd4-fd10-4d98-b6d8-ce5d864ae438"
-					(reference "D3901")
+					(reference "D3201")
 					(unit 1)
 				)
@@
 		(dnp no)
 		(fields_autoplaced yes)
-		(property "Reference" "C3903"
+		(property "Reference" "C3201"
 			(at 233.68 190.4999 90)
 			(effects
@@
 			(project "_Sub_HW_Qcopter"
 				(path "/b8703f06-b3da-4de2-b217-f104939b36e8/6184e84e-040e-4878-8152-76cf0b949e21/0ce565c6-f8fe-4174-9716-15fae563dcc2/82e4bdd4-fd10-4d98-b6d8-ce5d864ae438"
-					(reference "C3903")
+					(reference "C3201")
 					(unit 1)
 				)
@@
 		(on_board yes)
 		(dnp no)
-		(property "Reference" "RV3901"
+		(property "Reference" "RV3201"
 			(at 154.686 175.514 0)
 			(effects
@@
 			(project "_Sub_HW_Qcopter"
 				(path "/b8703f06-b3da-4de2-b217-f104939b36e8/6184e84e-040e-4878-8152-76cf0b949e21/0ce565c6-f8fe-4174-9716-15fae563dcc2/82e4bdd4-fd10-4d98-b6d8-ce5d864ae438"
-					(reference "RV3901")
+					(reference "RV3201")
 					(unit 1)
 				)
@@
 		(dnp no)
 		(fields_autoplaced yes)
-		(property "Reference" "C3901"
+		(property "Reference" "C3202"
 			(at 254 190.4999 90)
 			(effects
@@
 			(project "_Sub_HW_Qcopter"
 				(path "/b8703f06-b3da-4de2-b217-f104939b36e8/6184e84e-040e-4878-8152-76cf0b949e21/0ce565c6-f8fe-4174-9716-15fae563dcc2/82e4bdd4-fd10-4d98-b6d8-ce5d864ae438"
-					(reference "C3901")
+					(reference "C3202")
 					(unit 1)
 				)
@@
 		(on_board yes)
 		(dnp no)
-		(property "Reference" "J3901"
+		(property "Reference" "J3202"
 			(at 360.68 196.8501 0)
 			(effects
@@
 			(project "_Sub_HW_Qcopter"
 				(path "/b8703f06-b3da-4de2-b217-f104939b36e8/6184e84e-040e-4878-8152-76cf0b949e21/0ce565c6-f8fe-4174-9716-15fae563dcc2/82e4bdd4-fd10-4d98-b6d8-ce5d864ae438"
-					(reference "J3901")
+					(reference "J3202")
 					(unit 1)
 				)
+			)
+		)
+	)
+	(symbol
+		(lib_id "power:GND")
+		(at 97.79 208.28 0)
+		(unit 1)
+		(exclude_from_sim no)
+		(in_bom yes)
+		(on_board yes)
+		(dnp no)
+		(property "Reference" "#PWR03201"
+			(at 97.79 214.63 0)
+			(effects
+				(font
+					(size 1.27 1.27)
+				)
+				(hide yes)
+			)
+		)
+		(property "Value" "GND"
+			(at 95.758 212.598 0)
+			(effects
+				(font
+					(size 1.27 1.27)
+				)
+				(justify left)
+			)
+		)
+		(property "Footprint" ""
+			(at 97.79 208.28 0)
+			(effects
+				(font
+					(size 1.27 1.27)
+				)
+				(hide yes)
+			)
+		)
+		(property "Datasheet" ""
+			(at 97.79 208.28 0)
+			(effects
+				(font
+					(size 1.27 1.27)
+				)
+				(hide yes)
+			)
+		)
+		(property "Description" "Power symbol creates a global label with name \"GND\" , ground"
+			(at 97.79 208.28 0)
+			(effects
+				(font
+					(size 1.27 1.27)
+				)
+				(hide yes)
+			)
+		)
+		(pin "1"
+		)
+		(instances
+			(project "_Sub_HW_Qcopter"
+				(path "/b8703f06-b3da-4de2-b217-f104939b36e8/6184e84e-040e-4878-8152-76cf0b949e21/0ce565c6-f8fe-4174-9716-15fae563dcc2/82e4bdd4-fd10-4d98-b6d8-ce5d864ae438"
+					(reference "#PWR03201")
+					(unit 1)
+				)

Commit message: Update [020301] - BATTERY CHARGER.kicad_sch
Other:
- note added: "LAYOUT NOTE:"

Commit message: Update [020301] - BATTERY CHARGER.kicad_sch
Parts:
- C3201, C3202, C3203, D3201, D3202, D3203, D3204, J3201, J3202, RV3201, U3201: SCH CHECK SCH (N/A) -> SCH (CHECKED)
Changed lines of the file:
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@@
 			)
 		)
-		(property "SCH CHECK" "SCH (N/A)"
+		(property "SCH CHECK" "SCH (CHECKED)"
 			(at 326.39 194.3099 90)
 			(effects
@@
 			)
 		)
-		(property "SCH CHECK" "SCH (N/A)"
+		(property "SCH CHECK" "SCH (CHECKED)"
 			(at 210.82 198.1199 90)
 			(effects
@@
 			)
 		)
-		(property "SCH CHECK" "SCH (N/A)"
+		(property "SCH CHECK" "SCH (CHECKED)"
 			(at 173.99 198.1199 90)
 			(effects
@@
 			)
 		)
-		(property "SCH CHECK" "SCH (N/A)"
+		(property "SCH CHECK" "SCH (CHECKED)"
 			(at 292.1 172.72 0)
 			(effects
@@
 		(pin "5"
 		)
+		(pin "2"
+		)
+		(pin "1"
+		)
+		(pin "4"
+		)
 		(pin "3"
-		)
-		(pin "4"
-		)
-		(pin "2"
-		)
-		(pin "1"
 		)
 		(instances
@@
 			)
 		)
-		(property "SCH CHECK" "SCH (N/A)"
+		(property "SCH CHECK" "SCH (CHECKED)"
 			(at 148.59 198.1199 90)
 			(effects
@@
 			)
 		)
-		(property "SCH CHECK" "SCH (N/A)"
+		(property "SCH CHECK" "SCH (CHECKED)"
 			(at 97.79 172.72 0)
 			(effects
@@
 			)
 		)
-		(property "SCH CHECK" "SCH (N/A)"
+		(property "SCH CHECK" "SCH (CHECKED)"
 			(at 123.19 198.1199 90)
 			(effects
@@
 			)
 		)
-		(property "SCH CHECK" "SCH (N/A)"
+		(property "SCH CHECK" "SCH (CHECKED)"
 			(at 233.68 198.1199 90)
 			(effects
@@
 			)
 		)
-		(property "SCH CHECK" "SCH (N/A)"
+		(property "SCH CHECK" "SCH (CHECKED)"
 			(at 156.21 178.054 0)
 			(effects
@@
 			)
 		)
-		(property "SCH CHECK" "SCH (N/A)"
+		(property "SCH CHECK" "SCH (CHECKED)"
 			(at 254 198.1199 90)
 			(effects
@@
 			)
 		)
-		(property "SCH CHECK" "SCH (N/A)"
+		(property "SCH CHECK" "SCH (CHECKED)"
 			(at 360.68 189.2301 0)
 			(effects
