File: Hardware/_Sub_HW_Qcopter/v1_20240309/Design Folder/_Sub_HW_Qcopter/[0201] - FBD_FlightController.kicad_sch (KiCad schematic)
At the start: 0 parts

Commit message: Update [0201] - FBD_FlightController.kicad_sch
Other:
- sheet STM32U575 Driver ports: added ADC1_IN1; removed ADC_A0
- note added: "CHECKED"
