File: Hardware/_Sub_HW_Qcopter/v1_20240309/Design Folder/_Sub_HW_Qcopter/[020201] - STM32WLE5 Driver.kicad_sch (KiCad schematic)
At the start: 24 parts, among them J2701 HDR_1X4_VERT, U2701 SN74LVC1G17DCKR, U2702 NX3L1T3157GMZ, U2703 STM32WLE5CCU7, X2701 32MHz_10pF_10ppm

Commit message: Update [020201] - STM32WLE5 Driver.kicad_sch
Parts:
- C2701, C2702, C2703, C2704, C2705, C2706, C2707, C2708, C2709, C2710, C2711, C2712, J2701, JP2701, L2701, LED2701, R2701, R2702, R2703, R2704, U2701, U2702, U2703, X2701: SCH CHECK SCH (N/A) -> SCH (CHECKED)
Changed lines of the file:
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@@
 			)
 		)
-		(property "SCH CHECK" "SCH (N/A)"
+		(property "SCH CHECK" "SCH (CHECKED)"
 			(at 40.64 210.8199 90)
 			(effects
@@
 			)
 		)
-		(property "SCH CHECK" "SCH (N/A)"
+		(property "SCH CHECK" "SCH (CHECKED)"
 			(at 421.64 255.2699 90)
 			(effects
@@
 			)
 		)
-		(property "SCH CHECK" "SCH (N/A)"
+		(property "SCH CHECK" "SCH (CHECKED)"
 			(at 296.926 158.75 0)
 			(effects
@@
 			)
 		)
-		(property "SCH CHECK" "SCH (N/A)"
+		(property "SCH CHECK" "SCH (CHECKED)"
 			(at 167.64 210.8199 90)
 			(effects
@@
 			)
 		)
-		(property "SCH CHECK" "SCH (N/A)"
+		(property "SCH CHECK" "SCH (CHECKED)"
 			(at 243.84 228.5999 90)
 			(effects
@@
 			)
 		)
-		(property "SCH CHECK" "SCH (N/A)"
+		(property "SCH CHECK" "SCH (CHECKED)"
 			(at 218.44 224.7899 90)
 			(effects
@@
 			)
 		)
-		(property "SCH CHECK" "SCH (N/A)"
+		(property "SCH CHECK" "SCH (CHECKED)"
 			(at 193.04 224.7899 90)
 			(effects
@@
 			)
 		)
-		(property "SCH CHECK" "SCH (N/A)"
+		(property "SCH CHECK" "SCH (CHECKED)"
 			(at 91.44 210.8199 90)
 			(effects
@@
 			)
 		)
-		(property "SCH CHECK" "SCH (N/A)"
+		(property "SCH CHECK" "SCH (CHECKED)"
 			(at 276.86 184.404 0)
 			(effects
@@
 			)
 		)
-		(property "SCH CHECK" "SCH (N/A)"
+		(property "SCH CHECK" "SCH (CHECKED)"
 			(at 386.08 283.2099 0)
 			(effects
@@
 			)
 		)
-		(property "SCH CHECK" "SCH (N/A)"
+		(property "SCH CHECK" "SCH (CHECKED)"
 			(at 245.11 253.9999 90)
 			(effects
@@
 			)
 		)
-		(property "SCH CHECK" "SCH (N/A)"
+		(property "SCH CHECK" "SCH (CHECKED)"
 			(at 116.84 212.0899 90)
 			(effects
@@
 			)
 		)
-		(property "SCH CHECK" "SCH (N/A)"
+		(property "SCH CHECK" "SCH (CHECKED)"
 			(at 314.96 223.52 0)
 			(effects
@@
 			)
 		)
-		(property "SCH CHECK" "SCH (N/A)"
+		(property "SCH CHECK" "SCH (CHECKED)"
 			(at 142.24 210.8199 90)
 			(effects
@@
 			)
 		)
-		(property "SCH CHECK" "SCH (N/A)"
+		(property "SCH CHECK" "SCH (CHECKED)"
 			(at 276.86 169.164 0)
 			(effects
@@
 			)
 		)
-		(property "SCH CHECK" "SCH (N/A)"
+		(property "SCH CHECK" "SCH (CHECKED)"
 			(at 307.34 148.5899 90)
 			(effects
@@
 			)
 		)
-		(property "SCH CHECK" "SCH (N/A)"
+		(property "SCH CHECK" "SCH (CHECKED)"
 			(at 288.29 91.44 0)
 			(effects
@@
 			)
 		)
-		(property "SCH CHECK" "SCH (N/A)"
+		(property "SCH CHECK" "SCH (CHECKED)"
 			(at 381 147.32 0)
 			(effects
@@
 			)
 		)
-		(property "SCH CHECK" "SCH (N/A)"
+		(property "SCH CHECK" "SCH (CHECKED)"
 			(at 66.04 210.8199 90)
 			(effects
@@
 			)
 		)
-		(property "SCH CHECK" "SCH (N/A)"
+		(property "SCH CHECK" "SCH (CHECKED)"
 			(at 307.34 111.7599 90)
 			(effects
@@
 			)
 		)
-		(property "SCH CHECK" "SCH (N/A)"
+		(property "SCH CHECK" "SCH (CHECKED)"
 			(at 248.92 111.7599 90)
 			(effects
@@
 			)
 		)
-		(property "SCH CHECK" "SCH (N/A)"
+		(property "SCH CHECK" "SCH (CHECKED)"
 			(at 424.18 271.0814 90)
 			(effects
@@
 			)
 		)
-		(property "SCH CHECK" "SCH (N/A)"
+		(property "SCH CHECK" "SCH (CHECKED)"
 			(at 248.92 96.5199 90)
 			(effects
@@
 			)
 		)
-		(property "SCH CHECK" "SCH (N/A)"
+		(property "SCH CHECK" "SCH (CHECKED)"
 			(at 307.34 177.7999 90)
 			(effects

Commit message: Update [020201] - STM32WLE5 Driver.kicad_sch
Connections:
- net STM32WLE5_BOOT0: now reaches JP2701.2, R2702.1, U2703.19 (PH3-BOOT0)
- net STM32WLE5_VRPA renamed STM32WLE5_VR_PA
Changed lines of the file:
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@@
 	(title_block
 		(title "Quadcopter")
-		(date "2024-03-17")
+		(date "2024-03-20")
 		(rev "01")
 		(company "Mend0z0")
 		(comment 1 "01")
-		(comment 2 "PRELIMINARY")
+		(comment 2 "CHECKED")
 		(comment 3 "Siavash Taher Parvar")
 		(comment 8 "N/A")
@@
 		)
 	)
+	(label "STM32WLE5_BOOT0"
+		(at 336.55 157.48 0)
+		(fields_autoplaced yes)
+		(effects
+			(font
+				(size 1.27 1.27)
+			)
+			(justify left bottom)
+		)
+	)
 	(label "STM32WLE5_VDD"
 		(at 337.82 193.04 0)
@@
 	)
 	(hierarchical_label "STM32WLE5_RFIP"
-		(shape bidirectional)
+		(shape input)
 		(at 431.8 162.56 0)
 		(fields_autoplaced yes)
@@
 	)
 	(hierarchical_label "STM32WLE5_RFOHP"
-		(shape bidirectional)
+		(shape output)
 		(at 431.8 157.48 0)
 		(fields_autoplaced yes)
@@
 	)
 	(hierarchical_label "STM32WLE5_RFOLP"
-		(shape bidirectional)
+		(shape output)
 		(at 431.8 160.02 0)
 		(fields_autoplaced yes)
@@
 		)
 	)
-	(hierarchical_label "STM32WLE5_VRPA"
-		(shape bidirectional)
+	(hierarchical_label "STM32WLE5_VR_PA"
+		(shape output)
 		(at 431.8 154.94 0)
 		(fields_autoplaced yes)
@@
 	)
 	(hierarchical_label "STM32WLE5_RFIN"
-		(shape bidirectional)
+		(shape input)
 		(at 431.8 165.1 0)
 		(fields_autoplaced yes)
