File: Hardware/_Sub_HW_Qcopter/v1_20240309/Design Folder/_Sub_HW_Qcopter/[0202] - FBD_RadioController.kicad_sch (KiCad schematic)
At the start: 0 parts

Commit message: Update [0202] - FBD_RadioController.kicad_sch
Other:
- sheet STM32WLE5 Driver ports: added STM32WLE5_VR_PA; removed STM32WLE5_VRPA
- note added: "CHECKED"
Changed lines of the file:
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@@
 	(title_block
 		(title "Quadcopter")
-		(date "2024-03-17")
+		(date "2024-03-20")
 		(rev "01")
 		(company "Mend0z0")
 		(comment 1 "01")
-		(comment 2 "PRELIMINARY")
+		(comment 2 "CHECKED")
 		(comment 3 "Siavash Taher Parvar")
 		(comment 8 "N/A")
@@
 	(wire
 		(pts
-			(xy 201.93 168.91) (xy 228.6 168.91)
+			(xy 203.2 168.91) (xy 228.6 168.91)
 		)
 		(stroke
@@
 	(wire
 		(pts
-			(xy 201.93 173.99) (xy 228.6 173.99)
+			(xy 203.2 173.99) (xy 228.6 173.99)
 		)
 		(stroke
@@
 	(wire
 		(pts
-			(xy 321.31 137.16) (xy 330.2 137.16)
+			(xy 317.5 137.16) (xy 330.2 137.16)
 		)
 		(stroke
@@
 	(wire
 		(pts
-			(xy 201.93 166.37) (xy 228.6 166.37)
+			(xy 203.2 166.37) (xy 228.6 166.37)
 		)
 		(stroke
@@
 	(wire
 		(pts
-			(xy 201.93 177.8) (xy 228.6 177.8)
+			(xy 203.2 177.8) (xy 228.6 177.8)
 		)
 		(stroke
@@
 	(wire
 		(pts
-			(xy 201.93 171.45) (xy 228.6 171.45)
+			(xy 203.2 171.45) (xy 228.6 171.45)
 		)
 		(stroke
@@
 	(wire
 		(pts
-			(xy 201.93 180.34) (xy 228.6 180.34)
+			(xy 203.2 180.34) (xy 228.6 180.34)
 		)
 		(stroke
@@
 	(text_box "4"
 		(exclude_from_sim no)
-		(at 342.9 189.23 0)
-		(size 11.43 12.7)
+		(at 344.17 187.96 0)
+		(size 10.16 11.43)
 		(stroke
 			(width 0)
@@
 	(text_box "3"
 		(exclude_from_sim no)
-		(at 342.9 148.59 0)
+		(at 342.9 140.97 0)
 		(size 11.43 12.7)
 		(stroke
@@
 		)
 	)
+	(text "CHECKED"
+		(exclude_from_sim no)
+		(at 348.742 155.956 0)
+		(effects
+			(font
+				(size 1.905 1.905)
+				(thickness 0.381)
+				(bold yes)
+			)
+		)
+	)
+	(text "CHECKED"
+		(exclude_from_sim no)
+		(at 254 215.9 0)
+		(effects
+			(font
+				(size 1.905 1.905)
+				(thickness 0.381)
+				(bold yes)
+			)
+		)
+	)
+	(text "CHECKED"
+		(exclude_from_sim no)
+		(at 348.742 201.676 0)
+		(effects
+			(font
+				(size 1.905 1.905)
+				(thickness 0.381)
+				(bold yes)
+			)
+		)
+	)
+	(text "CHECKED"
+		(exclude_from_sim no)
+		(at 348.742 254.762 0)
+		(effects
+			(font
+				(size 1.905 1.905)
+				(thickness 0.381)
+				(bold yes)
+			)
+		)
+	)
+	(text "CHECKED"
+		(exclude_from_sim no)
+		(at 186.436 237.744 0)
+		(effects
+			(font
+				(size 1.905 1.905)
+				(thickness 0.381)
+				(bold yes)
+			)
+		)
+	)
 	(label "+3V3_2"
-		(at 321.31 137.16 0)
+		(at 317.5 137.16 0)
 		(fields_autoplaced yes)
 		(effects
@@
 	(hierarchical_label "FLIGHT_CTR_SPI_CLK"
 		(shape input)
-		(at 201.93 168.91 180)
+		(at 203.2 168.91 180)
 		(fields_autoplaced yes)
 		(effects
@@
 	(hierarchical_label "FLIGHT_CTR_SPI_MISO"
 		(shape output)
-		(at 201.93 171.45 180)
+		(at 203.2 171.45 180)
 		(fields_autoplaced yes)
 		(effects
@@
 	(hierarchical_label "FLIGHT_CTR_SPI_NSS"
 		(shape input)
-		(at 201.93 166.37 180)
+		(at 203.2 166.37 180)
 		(fields_autoplaced yes)
 		(effects
@@
 	(hierarchical_label "FLIGHT_CTR_UART_RX"
 		(shape output)
-		(at 201.93 180.34 180)
+		(at 203.2 180.34 180)
 		(fields_autoplaced yes)
 		(effects
@@
 	(hierarchical_label "FLIGHT_CTR_UART_TX"
 		(shape input)
-		(at 201.93 177.8 180)
+		(at 203.2 177.8 180)
 		(fields_autoplaced yes)
 		(effects
@@
 	(hierarchical_label "FLIGHT_CTR_SPI_MOSI"
 		(shape input)
-		(at 201.93 173.99 180)
+		(at 203.2 173.99 180)
 		(fields_autoplaced yes)
 		(effects
@@
 			)
 		)
-		(pin "RFO_LP" bidirectional
-			(at 330.2 144.78 180)
-			(effects
-				(font
-					(size 1.27 1.27)
-				)
-				(justify left)
-			)
-		)
 		(pin "VR_PA" input
 			(at 330.2 139.7 180)
@@
 			)
 		)
-		(pin "RFI_P" bidirectional
-			(at 330.2 147.32 180)
-			(effects
-				(font
-					(size 1.27 1.27)
-				)
-				(justify left)
-			)
-		)
-		(pin "RFI_N" bidirectional
-			(at 330.2 149.86 180)
-			(effects
-				(font
-					(size 1.27 1.27)
-				)
-				(justify left)
-			)
-		)
 		(pin "FE_CTRL2" input
 			(at 330.2 157.48 180)
@@
 			)
 		)
-		(pin "RFO_HP" bidirectional
-			(at 330.2 142.24 180)
-			(effects
-				(font
-					(size 1.27 1.27)
-				)
-				(justify left)
-			)
-		)
 		(pin "+PWR" input
 			(at 330.2 137.16 180)
+			(effects
+				(font
+					(size 1.27 1.27)
+				)
+				(justify left)
+			)
+		)
+		(pin "RFO_HP" input
+			(at 330.2 142.24 180)
+			(effects
+				(font
+					(size 1.27 1.27)
+				)
+				(justify left)
+			)
+		)
+		(pin "RFI_P" output
+			(at 330.2 147.32 180)
+			(effects
+				(font
+					(size 1.27 1.27)
+				)
+				(justify left)
+			)
+		)
+		(pin "RFO_LP" input
+			(at 330.2 144.78 180)
+			(effects
+				(font
+					(size 1.27 1.27)
+				)
+				(justify left)
+			)
+		)
+		(pin "RFI_N" output
+			(at 330.2 149.86 180)
 			(effects
 				(font
@@
 			)
 		)
-		(pin "STM32WLE5_RFIN" bidirectional
-			(at 279.4 149.86 0)
-			(effects
-				(font
-					(size 1.27 1.27)
-				)
-				(justify right)
-			)
-		)
-		(pin "STM32WLE5_RFIP" bidirectional
-			(at 279.4 147.32 0)
-			(effects
-				(font
-					(size 1.27 1.27)
-				)
-				(justify right)
-			)
-		)
-		(pin "STM32WLE5_RFOHP" bidirectional
-			(at 279.4 142.24 0)
-			(effects
-				(font
-					(size 1.27 1.27)
-				)
-				(justify right)
-			)
-		)
-		(pin "STM32WLE5_RFOLP" bidirectional
-			(at 279.4 144.78 0)
-			(effects
-				(font
-					(size 1.27 1.27)
-				)
-				(justify right)
-			)
-		)
-		(pin "STM32WLE5_VRPA" bidirectional
-			(at 279.4 139.7 0)
-			(effects
-				(font
-					(size 1.27 1.27)
-				)
-				(justify right)
-			)
-		)
 		(pin "FE_CTRL1" output
 			(at 279.4 154.94 0)
@@
 			)
 		)
+		(pin "STM32WLE5_VR_PA" output
+			(at 279.4 139.7 0)
+			(effects
+				(font
+					(size 1.27 1.27)
+				)
+				(justify right)
+			)
+		)
+		(pin "STM32WLE5_RFOHP" output
+			(at 279.4 142.24 0)
+			(effects
+				(font
+					(size 1.27 1.27)
+				)
+				(justify right)
+			)
+		)
+		(pin "STM32WLE5_RFOLP" output
+			(at 279.4 144.78 0)
+			(effects
+				(font
+					(size 1.27 1.27)
+				)
+				(justify right)
+			)
+		)
+		(pin "STM32WLE5_RFIP" input
+			(at 279.4 147.32 0)
+			(effects
+				(font
+					(size 1.27 1.27)
+				)
+				(justify right)
+			)
+		)
+		(pin "STM32WLE5_RFIN" input
+			(at 279.4 149.86 0)
+			(effects
+				(font
+					(size 1.27 1.27)
+				)
+				(justify right)
+			)
+		)
