File: Hardware/_Sub_HW_Qcopter/v1_20240309/Design Folder/_Sub_HW_Qcopter/_Sub_HW_Qcopter.kicad_pcb (KiCad board)
At the start: 4 copper layers, 0 parts

Commit message: Update _Sub_HW_Qcopter.kicad_pcb
Parts:
- added ANT3101: 2.4GHz_2W_0.5dBi, RF_Antenna:Johanson_2450AT18x100, B.Cu at (177.8, 252.7)
- added C1001: 100nF_16V_X7R, Capacitor_SMD:C_0603_1608Metric, B.Cu at (167.2, 223.1)
- added C1101: 100nF_16V_X7R, Capacitor_SMD:C_0603_1608Metric, B.Cu at (166.2, 235.5)
- added C1201: 100nF_16V_X7R, Capacitor_SMD:C_0603_1608Metric, B.Cu at (195.1, 240.1)
- added C1301: 100nF_16V_X7R, Capacitor_SMD:C_0603_1608Metric, B.Cu at (177.5, 223.8)
- added C1302: 100nF_16V_X7R, Capacitor_SMD:C_0603_1608Metric, B.Cu at (176.3, 233.9)
- added C1303: 100nF_16V_X7R, Capacitor_SMD:C_0603_1608Metric, B.Cu at (174.8, 233.9)
- added C1401: 100nF_16V_X7R, Capacitor_SMD:C_0603_1608Metric, B.Cu at (184.2, 247.1)
- added C1402: 100nF_16V_X7R, Capacitor_SMD:C_0603_1608Metric, B.Cu at (184.2, 245.4)
- added C2001: 1uF_10V_X7R, Capacitor_SMD:C_0603_1608Metric, F.Cu at (184.9, 241.6)
- added C2101: 4u7F_16V_X7R, Capacitor_SMD:C_0603_1608Metric, B.Cu at (199.9, 231.4)
- added C2102: 4u7F_16V_X7R, Capacitor_SMD:C_0603_1608Metric, B.Cu at (199.9, 233.2)
- added C2103: 4u7F_16V_X7R, Capacitor_SMD:C_0603_1608Metric, B.Cu at (199.9, 234.9)
- added C2301: 100nF_16V_X7R, Capacitor_SMD:C_0603_1608Metric, B.Cu at (160.3, 244.3)
- added C2302: 100nF_16V_X7R, Capacitor_SMD:C_0603_1608Metric, F.Cu at (160.3, 244.3)
- added C2303: 1uF_10V_X7R, Capacitor_SMD:C_0603_1608Metric, F.Cu at (156.2, 246.6)
- added C2401: 100nF_16V_X7R, Capacitor_SMD:C_0603_1608Metric, B.Cu at (191.5, 245.1)
- added C2402: 100nF_16V_X7R, Capacitor_SMD:C_0603_1608Metric, F.Cu at (191.5, 245.1)
- added C2403: 1uF_10V_X7R, Capacitor_SMD:C_0603_1608Metric, F.Cu at (191.9, 247.7)
- added C2501: 100nF_16V_X7R, Capacitor_SMD:C_0603_1608Metric, F.Cu at (184.9, 205.7)
- added C2502: 100nF_16V_X7R, Capacitor_SMD:C_0603_1608Metric, B.Cu at (184.9, 205.7)
- added C2503: 1uF_10V_X7R, Capacitor_SMD:C_0603_1608Metric, F.Cu at (184.9, 207.5)
- added C2601: 100nF_16V_X7R, Capacitor_SMD:C_0603_1608Metric, B.Cu at (167.5, 211.6)
- added C2602: 100nF_16V_X7R, Capacitor_SMD:C_0603_1608Metric, F.Cu at (167.5, 211.6)
- added C2603: 1uF_10V_X7R, Capacitor_SMD:C_0603_1608Metric, F.Cu at (167.5, 209.8)
- added C2701: 1uF_10V_X7R, Capacitor_SMD:C_0603_1608Metric, F.Cu at (195.7, 217.3)
- added C2702: 100nF_16V_X7R, Capacitor_SMD:C_0603_1608Metric, F.Cu at (195.7, 215.8)
- added C2703: 1uF_10V_X7R, Capacitor_SMD:C_0603_1608Metric, F.Cu at (193.4, 220.9)
- added C2704: 100nF_16V_X7R, Capacitor_SMD:C_0603_1608Metric, F.Cu at (191.8, 220.9)
- added C2705: 1uF_10V_X7R, Capacitor_SMD:C_0603_1608Metric, F.Cu at (195.7, 220.3)
- added C2706: 100nF_16V_X7R, Capacitor_SMD:C_0603_1608Metric, F.Cu at (195.7, 218.8)
- added C2707: 4u7F_16V_X7R, Capacitor_SMD:C_0603_1608Metric, F.Cu at (191.9, 215.5)
- added C2708: 100nF_16V_X7R, Capacitor_SMD:C_0603_1608Metric, F.Cu at (190.4, 215.5)
- added C2709: 470nF_16V_X7R, Capacitor_SMD:C_0603_1608Metric, F.Cu at (193.4, 215.5)
- added C2710: 100nF_16V_X7R, Capacitor_SMD:C_0603_1608Metric, B.Cu at (199.9, 229.6)
- added C2711: 10pF_50V_C0G, Capacitor_SMD:C_0603_1608Metric, B.Cu at (193.3, 210.3)
- added C2712: 10pF_50V_C0G, Capacitor_SMD:C_0603_1608Metric, B.Cu at (188.7, 210.3)
- added C2901: 68pF_50V_C0G, Capacitor_SMD:C_0402_1005Metric, F.Cu at (189.7, 217.7)
- added C2902: 47nF_25V_X7R, Capacitor_SMD:C_0402_1005Metric, F.Cu at (189.7, 218.8)
- added C2903: 1p2F_50V_C0G, Capacitor_SMD:C_0402_1005Metric, F.Cu at (189.7, 220.1)
- added C2904: 33pF_50V_C0G, Capacitor_SMD:C_0402_1005Metric, B.Cu at (181.9, 215.1)
- added C2905: 33pF_50V_C0G, Capacitor_SMD:C_0402_1005Metric, B.Cu at (181.9, 213.6)
- added C2906: 2p7F_50V_C0G, Capacitor_SMD:C_0402_1005Metric, B.Cu at (184.9, 216.4)
- added C2907: 3p6F_50V_C0G, Capacitor_SMD:C_0402_1005Metric, B.Cu at (184.9, 217.4)
- added C2908: 5p6F_50V_C0G, Capacitor_SMD:C_0402_1005Metric, F.Cu at (184.1, 209.6)
- added C2909: 1p2F_50V_C0G, Capacitor_SMD:C_0402_1005Metric, B.Cu at (184.2, 209.6)
- added C2910: 2p7F_50V_C0G, Capacitor_SMD:C_0402_1005Metric, F.Cu at (182.4, 210.6)
- added C2911: 2p2F_50V_C0G, Capacitor_SMD:C_0402_1005Metric, B.Cu at (182.4, 210.6)
- added C2912: 5p6F_50V_C0G, Capacitor_SMD:C_0402_1005Metric, B.Cu at (180.6, 210.6)
- added C2913: 3p3F_50V_C0G, Capacitor_SMD:C_0402_1005Metric, F.Cu at (180.6, 210.6)
- added C2914: 68pF_50V_C0G, Capacitor_SMD:C_0402_1005Metric, B.Cu at (180.6, 209.6)
- added C2915: 33pF_50V_C0G, Capacitor_SMD:C_0402_1005Metric, F.Cu at (180.6, 209.6)
- added C2916: 1p2F_50V_C0G, Capacitor_SMD:C_0402_1005Metric, B.Cu at (177.3, 210.1)
- added C2917: 1p3F_50V_C0G, Capacitor_SMD:C_0402_1005Metric, F.Cu at (177.3, 210.1)
- added C2918: 1nF_50V_X7R, Capacitor_SMD:C_0603_1608Metric, F.Cu at (165.9, 206.8)
- added C2919: 1nF_50V_X7R, Capacitor_SMD:C_0603_1608Metric, F.Cu at (168.9, 206.8)
- added C2920: 1nF_50V_X7R, Capacitor_SMD:C_0603_1608Metric, F.Cu at (172.0, 206.8)
- added C2921: 33pF_50V_C0G, Capacitor_SMD:C_0402_1005Metric, F.Cu at (177.8, 208.3)
- added C2922: 3p3F_50V_C0G, Capacitor_SMD:C_0402_1005Metric, F.Cu at (179.3, 207.8)
- added C2923: 3p3F_50V_C0G, Capacitor_SMD:C_0402_1005Metric, F.Cu at (180.6, 205.7)
- added C3101: 4u7F_16V_X7R, Capacitor_SMD:C_0603_1608Metric, B.Cu at (165.4, 244.7)
- added C3102: 4u7F_16V_X7R, Capacitor_SMD:C_0603_1608Metric, B.Cu at (165.4, 246.2)
- added C3103: 4u7F_16V_X7R, Capacitor_SMD:C_0603_1608Metric, F.Cu at (170.2, 244.3)
- added C3104: 4u7F_16V_X7R, Capacitor_SMD:C_0603_1608Metric, B.Cu at (167.6, 240.0)
- added C3105: 4u7F_16V_X7R, Capacitor_SMD:C_0603_1608Metric, B.Cu at (178.3, 245.4)
- added C3106: 4u7F_16V_X7R, Capacitor_SMD:C_0603_1608Metric, B.Cu at (178.3, 243.8)
- added C3107: 4u7F_16V_X7R, Capacitor_SMD:C_0603_1608Metric, F.Cu at (173.2, 248.2)
- added C3108: 4u7F_16V_X7R, Capacitor_SMD:C_0603_1608Metric, F.Cu at (165.4, 244.7)
- added C3109: 1uF_10V_X7R, Capacitor_SMD:C_0603_1608Metric, F.Cu at (171.7, 244.3)
- added C3110: 4u7F_16V_X7R, Capacitor_SMD:C_0603_1608Metric, F.Cu at (170.2, 248.2)
- added C3111: 4u7F_16V_X7R, Capacitor_SMD:C_0603_1608Metric, F.Cu at (178.3, 245.4)
- added C3112: 4u7F_16V_X7R, Capacitor_SMD:C_0603_1608Metric, F.Cu at (178.3, 243.8)
- added C3113: 12pF_50V_C0G, Capacitor_SMD:C_0603_1608Metric, B.Cu at (174.0, 240.0)
- added C3114: 12pF_50V_C0G, Capacitor_SMD:C_0603_1608Metric, B.Cu at (169.4, 240.0)
- added C3115: 1pF_50V_C0G, Capacitor_SMD:C_0201_0603Metric, B.Cu at (181.1, 248.4)
- added C3116: 1uF_10V_X7R, Capacitor_SMD:C_0603_1608Metric, F.Cu at (171.7, 248.2)
- added C3117: 1pF_50V_C0G, Capacitor_SMD:C_0201_0603Metric, B.Cu at (179.1, 248.4)
- added C3118: 1uF_10V_X7R, Capacitor_SMD:C_0603_1608Metric, F.Cu at (165.4, 246.2)
- added C3119: 1pF_50V_C0G, Capacitor_SMD:C_0201_0603Metric, B.Cu at (179.1, 246.9)
- added C3120: 1uF_10V_X7R, Capacitor_SMD:C_0603_1608Metric, F.Cu at (173.2, 244.3)
- added C3121: 1p8F_50V_C0G, Capacitor_SMD:C_0201_0603Metric, B.Cu at (177.9, 247.9)
- added C3122: 1p8F_50V_C0G, Capacitor_SMD:C_0201_0603Metric, B.Cu at (177.9, 246.9)
- added C3201: 4u7F_16V_X7R, Capacitor_SMD:C_0603_1608Metric, B.Cu at (159.0, 216.9)
- added C3202: 1uF_10V_X7R, Capacitor_SMD:C_0603_1608Metric, B.Cu at (159.0, 214.9)
- added C3203: 1uF_10V_X7R, Capacitor_SMD:C_0603_1608Metric, B.Cu at (159.0, 219.2)
- added C3301: 4u7F_16V_X7R, Capacitor_SMD:C_0603_1608Metric, F.Cu at (157.2, 220.8)
- added C3302: 4u7F_16V_X7R, Capacitor_SMD:C_0603_1608Metric, F.Cu at (157.2, 222.6)
- added C3303: 680pF_100V_X7R, Capacitor_SMD:C_0603_1608Metric, F.Cu at (158.3, 211.3)
- added C3304: 4u7F_16V_X7R, Capacitor_SMD:C_0603_1608Metric, F.Cu at (161.3, 217.7)
- added C3305: 4u7F_16V_X7R, Capacitor_SMD:C_0603_1608Metric, F.Cu at (161.3, 219.5)
- added C3306: 4u7F_16V_X7R, Capacitor_SMD:C_0603_1608Metric, F.Cu at (161.3, 221.0)
- added C3401: 10uF_16V_X5R, Capacitor_SMD:C_0603_1608Metric, F.Cu at (157.7, 233.9)
- added C3402: 10uF_16V_X5R, Capacitor_SMD:C_0603_1608Metric, F.Cu at (160.0, 237.0)
- added C3501: 10uF_16V_X5R, Capacitor_SMD:C_0603_1608Metric, F.Cu at (163.3, 227.1)
- added C3502: 10uF_16V_X5R, Capacitor_SMD:C_0603_1608Metric, F.Cu at (160.3, 230.6)
- added C3601: 10uF_16V_X5R, Capacitor_SMD:C_0603_1608Metric, F.Cu at (187.2, 209.6)
- added C3602: 10uF_16V_X5R, Capacitor_SMD:C_0603_1608Metric, F.Cu at (194.9, 211.6)
- added C3701: 10uF_16V_X5R, Capacitor_SMD:C_0603_1608Metric, F.Cu at (165.4, 237.7)
- added C3702: 10uF_16V_X5R, Capacitor_SMD:C_0603_1608Metric, F.Cu at (162.3, 241.6)
- added C501: 10uF_16V_X5R, Capacitor_SMD:C_0603_1608Metric, B.Cu at (192.5, 234.7)
- added C502: 10uF_16V_X5R, Capacitor_SMD:C_0603_1608Metric, B.Cu at (195.4, 230.4)
- added C503: 10uF_16V_X5R, Capacitor_SMD:C_0603_1608Metric, B.Cu at (195.3, 238.3)
- added C504: 10uF_16V_X5R, Capacitor_SMD:C_0603_1608Metric, B.Cu at (195.4, 224.3)
- added C601: 4u7F_16V_X7R, Capacitor_SMD:C_0603_1608Metric, B.Cu at (179.3, 221.5)
- added C602: 4u7F_16V_X7R, Capacitor_SMD:C_0603_1608Metric, B.Cu at (181.1, 221.5)
- added C603: 100nF_16V_X7R, Capacitor_SMD:C_0603_1608Metric, B.Cu at (190.0, 225.9)
- added C604: 1uF_10V_X7R, Capacitor_SMD:C_0603_1608Metric, B.Cu at (179.8, 235.4)
- added C605: 12pF_50V_C0G, Capacitor_SMD:C_0603_1608Metric, F.Cu at (190.4, 226.3)
- added C606: 12pF_50V_C0G, Capacitor_SMD:C_0603_1608Metric, F.Cu at (190.4, 230.4)
- added C607: 1uF_10V_X7R, Capacitor_SMD:C_0603_1608Metric, B.Cu at (178.3, 235.4)
- added C608: 1uF_10V_X7R, Capacitor_SMD:C_0603_1608Metric, B.Cu at (172.0, 229.4)
- added C609: 1uF_10V_X7R, Capacitor_SMD:C_0603_1608Metric, B.Cu at (172.0, 225.8)
- added C610: 1uF_10V_X7R, Capacitor_SMD:C_0603_1608Metric, B.Cu at (183.6, 231.1)
- added C611: 1uF_10V_X7R, Capacitor_SMD:C_0603_1608Metric, B.Cu at (172.0, 232.9)
- added C612: 1uF_10V_X7R, Capacitor_SMD:C_0603_1608Metric, B.Cu at (181.4, 235.4)
- added C613: 1uF_10V_X7R, Capacitor_SMD:C_0603_1608Metric, B.Cu at (183.6, 222.2)
- added C614: 1uF_10V_X7R, Capacitor_SMD:C_0603_1608Metric, B.Cu at (183.6, 225.8)
- added C615: 1uF_10V_X7R, Capacitor_SMD:C_0603_1608Metric, B.Cu at (172.0, 222.2)
- added C616: 100nF_16V_X7R, Capacitor_SMD:C_0603_1608Metric, B.Cu at (172.0, 231.1)
- added C617: 100nF_16V_X7R, Capacitor_SMD:C_0603_1608Metric, B.Cu at (171.9, 227.6)
- added C618: 100nF_16V_X7R, Capacitor_SMD:C_0603_1608Metric, B.Cu at (183.6, 229.4)
- added C619: 100nF_16V_X7R, Capacitor_SMD:C_0603_1608Metric, B.Cu at (172.0, 234.7)
- added C620: 100nF_16V_X7R, Capacitor_SMD:C_0603_1608Metric, B.Cu at (182.9, 235.4)
- added C621: 100nF_16V_X7R, Capacitor_SMD:C_0603_1608Metric, B.Cu at (183.6, 220.5)
- added C622: 100nF_16V_X7R, Capacitor_SMD:C_0603_1608Metric, B.Cu at (183.6, 224.0)
- added C623: 1uF_10V_X7R, Capacitor_SMD:C_0603_1608Metric, B.Cu at (172.0, 224.0)
- added C624: 10nF_100V_X7R, Capacitor_SMD:C_0603_1608Metric, B.Cu at (183.6, 227.6)
- added C801: 100nF_16V_X7R, Capacitor_SMD:C_0603_1608Metric, B.Cu at (162.3, 214.9)
- added D3201: GG040205100N2P, Diode_SMD:D_0402_1005Metric, B.Cu at (153.9, 227.3)
- added D3202: GG040205100N2P, Diode_SMD:D_0402_1005Metric, B.Cu at (153.9, 228.3)
- added D3203: GG040205100N2P, Diode_SMD:D_0402_1005Metric, B.Cu at (153.9, 229.4)
- added D3204: GG040205100N2P, Diode_SMD:D_0402_1005Metric, B.Cu at (159.3, 221.0)
- added D3301: SK510A-LTP, Diode_SMD:D_SMA, F.Cu at (156.7, 214.1)
- added D3302: GG040205100N2P, Diode_SMD:D_0402_1005Metric, F.Cu at (161.0, 222.2)
- added D501: GEN_75V_100mA, Diode_SMD:D_0603_1608Metric, F.Cu at (154.4, 233.9)
- added F2201: 4A_8V_2mR, Fuse:Fuse_0805_2012Metric, F.Cu at (153.9, 244.1)
- added FB3101: FB_550mA_0.19R, Inductor_SMD:L_0402_1005Metric, B.Cu at (166.1, 240.3)
- added FB3102: FB_550mA_0.19R, Inductor_SMD:L_0402_1005Metric, B.Cu at (178.1, 242.6)
- added FB3103: FB_550mA_0.19R, Inductor_SMD:L_0402_1005Metric, F.Cu at (170.2, 251.0)
- added FB3104: FB_550mA_0.19R, Inductor_SMD:L_0402_1005Metric, F.Cu at (178.1, 246.6)
- added FD3801: ~, Fiducial:Fiducial_0.5mm_Mask1mm, F.Cu at (222.5, 223.0)
- added FD3802: ~, Fiducial:Fiducial_0.5mm_Mask1mm, F.Cu at (222.5, 225.5)
- added FD3803: ~, Fiducial:Fiducial_0.5mm_Mask1mm, F.Cu at (222.5, 228.1)
- added FD3804: ~, Fiducial:Fiducial_0.5mm_Mask1mm, F.Cu at (222.5, 230.6)
- added J1601: HDR_1X2_VERT, Connector_PinHeader_1.27mm:PinHeader_1x02_P1.27mm_Vertical, F.Cu at (199.8, 245.9)
- added J1701: HDR_1X2_VERT, Connector_PinHeader_1.27mm:PinHeader_1x02_P1.27mm_Vertical, F.Cu at (199.8, 243.3)
- added J1801: HDR_1X2_VERT, Connector_PinHeader_1.27mm:PinHeader_1x02_P1.27mm_Vertical, F.Cu at (199.8, 240.8)
- added J1901: HDR_1X2_VERT, Connector_PinHeader_1.27mm:PinHeader_1x02_P1.27mm_Vertical, F.Cu at (199.8, 238.3)
- added J2101: FPC_24_R/A-BOTT, _PCBLIB_Qcopter:CVILUX_CF35242D0RD-NH, F.Cu at (200.8, 228.3)
- added J2201: HDR_1X2_5A_THD-RA, Connector_PinHeader_2.54mm:PinHeader_1x02_P2.54mm_Horizontal, B.Cu at (156.5, 240.5)
- added J2202: HDR_1X2_VERT_1.25MM, Connector_Hirose:Hirose_DF13-02P-1.25DSA_1x02_P1.25mm_Vertical, B.Cu at (160.7, 251.3)
- added J2203: HDR_1X2_VERT_1.25MM, Connector_Hirose:Hirose_DF13-02P-1.25DSA_1x02_P1.25mm_Vertical, B.Cu at (193.0, 251.3)
- added J2204: HDR_1X2_VERT_1.25MM, Connector_Hirose:Hirose_DF13-02P-1.25DSA_1x02_P1.25mm_Vertical, B.Cu at (194.2, 206.8)
- added J2205: HDR_1X2_VERT_1.25MM, Connector_Hirose:Hirose_DF13-02P-1.25DSA_1x02_P1.25mm_Vertical, B.Cu at (163.2, 206.9)
- added J2701: HDR_1X4_VERT, Connector_PinHeader_1.27mm:PinHeader_1x04_P1.27mm_Vertical, B.Cu at (201.0, 211.6)
- added J2801: HDR_1X3_THD-1.27MM, Connector_PinHeader_1.27mm:PinHeader_1x03_P1.27mm_Vertical, F.Cu at (201.2, 214.6)
- added J2901: RECEPT_RF_50R, _PCBLIB_Qcopter:MURATA_MM8030-2610RJ3, F.Cu at (177.3, 205.7)
- added J3201: USB_MICRO B_RA, _PCBLIB_Qcopter:USB_Micro-B_Amphenol_10118194_Horizontal, F.Cu at (155.1, 228.3)
- added J3202: HDR_1X2_VERT_1.25MM, Connector_Hirose:Hirose_DF13-02P-1.25DSA_1x02_P1.25mm_Vertical, B.Cu at (154.2, 221.9)
- added J501: HDR_1X2_VERT, Connector_PinHeader_1.27mm:PinHeader_1x02_P1.27mm_Vertical, F.Cu at (153.9, 236.3)
- added J601: HDR_1X4_VERT, Connector_PinHeader_1.27mm:PinHeader_1x04_P1.27mm_Vertical, F.Cu at (186.2, 252.7)
- added J701: HDR_1X3_THD-1.27MM, Connector_PinHeader_1.27mm:PinHeader_1x03_P1.27mm_Vertical, F.Cu at (189.2, 252.7)
- added JP2201: JP_2POS, Jumper:SolderJumper-2_P1.3mm_Open_TrianglePad1.0x1.5mm, B.Cu at (156.7, 237.5)
- added JP2701: JP_2POS, Jumper:SolderJumper-2_P1.3mm_Open_TrianglePad1.0x1.5mm, B.Cu at (199.9, 221.0)
- added JP601: JP_2POS, Jumper:SolderJumper-2_P1.3mm_Open_TrianglePad1.0x1.5mm, F.Cu at (183.4, 247.7)
- added L2701: 15uH_250mA_0.95Ohm, Inductor_SMD:L_0805_2012Metric, B.Cu at (195.1, 210.6)
- added L2901: 11nH_500mA_0.14R, Inductor_SMD:L_0402_1005Metric, B.Cu at (186.4, 216.9)
- added L2902: 47nH_210mA_1.08Ohm, Inductor_SMD:L_0402_1005Metric, B.Cu at (183.9, 215.1)
- added L2903: 3n3H_2A_30mOhm, Inductor_SMD:L_0402_1005Metric, B.Cu at (185.9, 215.1)
- added L2904: 33nH_260mA_0.63Ohm, Inductor_SMD:L_0402_1005Metric, B.Cu at (183.9, 213.6)
- added L2905: 3nH_750mA_70mOhm, Inductor_SMD:L_0402_1005Metric, F.Cu at (182.4, 209.6)
- added L2906: 3n6H_900mA_40mOhm, Inductor_SMD:L_0402_1005Metric, B.Cu at (182.4, 209.6)
- added L2907: 8n7H_540mA_0.14R, Inductor_SMD:L_0402_1005Metric, B.Cu at (178.8, 209.6)
- added L2908: 8n7H_540mA_0.14R, Inductor_SMD:L_0402_1005Metric, F.Cu at (178.8, 209.6)
- added L2909: 8n7H_540mA_0.14R, Inductor_SMD:L_0402_1005Metric, F.Cu at (180.6, 207.8)
- added L3101: 3n9H_300mA_0.22R, Inductor_SMD:L_0402_1005Metric, B.Cu at (181.1, 252.2)
- added L3102: 2n7H_300mA_0.17R, Inductor_SMD:L_0402_1005Metric, B.Cu at (181.6, 250.2)
- added L3103: 2u2H_350mA_0.55R, Inductor_SMD:L_0402_1005Metric, B.Cu at (165.6, 247.7)
- added L3104: 3n3H_400mA_0.3R, Inductor_SMD:L_0201_0603Metric, B.Cu at (180.1, 248.4)
- added L3105: 15nH_560mA_0.172R, Inductor_SMD:L_0402_1005Metric, B.Cu at (165.6, 248.8)
- added L3106: 3n3H_400mA_0.3R, Inductor_SMD:L_0201_0603Metric, B.Cu at (180.1, 246.9)
- added L3301: 2u2H_2A_0.14R, Inductor_SMD:L_0805_2012Metric, F.Cu at (153.9, 218.0)
- added L601: 2u2H_1.3A_156mOhm, Inductor_SMD:L_0805_2012Metric, F.Cu at (172.2, 215.6)
- added LED1501: ORANGE_2V_20mA, LED_SMD:LED_0603_1608Metric, F.Cu at (191.0, 238.0)
- added LED1502: YELLOW_2V_20mA, LED_SMD:LED_0603_1608Metric, F.Cu at (191.0, 236.2)
- added LED2701: WHITE_3V2_420mcd, LED_SMD:LED_0603_1608Metric, F.Cu at (200.4, 218.7)
- added LED3001: RED_2V_20mA, LED_SMD:LED_0603_1608Metric, F.Cu at (191.0, 243.3)
- added LED3002: GREEN_3.3V_20mA, LED_SMD:LED_0603_1608Metric, F.Cu at (191.0, 241.6)
- added LED3003: BLUE_3.3V_20mA, LED_SMD:LED_0603_1608Metric, F.Cu at (191.0, 239.8)
- added LED3401: GREEN_3.3V_20mA, LED_SMD:LED_0603_1608Metric, F.Cu at (158.5, 241.6)
- added LED3501: GREEN_3.3V_20mA, LED_SMD:LED_0603_1608Metric, F.Cu at (160.3, 232.4)
- added LED3601: GREEN_3.3V_20mA, LED_SMD:LED_0603_1608Metric, F.Cu at (194.8, 208.5)
- added LED3701: GREEN_3.3V_20mA, LED_SMD:LED_0603_1608Metric, F.Cu at (163.0, 246.9)
- added LED601: WHITE_3V2_420mcd, LED_SMD:LED_0603_1608Metric, F.Cu at (180.6, 240.8)
- added MH3801: M3, MountingHole:MountingHole_3.2mm_M3_DIN965_Pad_TopBottom, F.Cu at (155.4, 251.0)
- added MH3802: M3, MountingHole:MountingHole_3.2mm_M3_DIN965_Pad_TopBottom, F.Cu at (199.5, 251.0)
- added MH3803: M3, MountingHole:MountingHole_3.2mm_M3_DIN965_Pad_TopBottom, F.Cu at (199.5, 207.0)
- added MH3804: M3, MountingHole:MountingHole_3.2mm_M3_DIN965_Pad_TopBottom, F.Cu at (155.4, 207.0)
- added R1301: 10kR_1/10W_1%, Resistor_SMD:R_0603_1608Metric, B.Cu at (176.0, 223.8)
- added R1302: 10kR_1/10W_1%, Resistor_SMD:R_0603_1608Metric, B.Cu at (183.6, 232.9)
- added R1303: 10kR_1/10W_1%, Resistor_SMD:R_0603_1608Metric, B.Cu at (174.5, 223.8)
- added R1401: 10kR_1/10W_1%, Resistor_SMD:R_0603_1608Metric, B.Cu at (191.4, 246.6)
- added R1501: 470R_1/10W_1%, Resistor_SMD:R_0603_1608Metric, F.Cu at (188.0, 238.0)
- added R1502: 470R_1/10W_1%, Resistor_SMD:R_0603_1608Metric, F.Cu at (188.0, 236.2)
- added R1601: 100R_1/10W_1%, Resistor_SMD:R_0603_1608Metric, B.Cu at (198.1, 246.4)
- added R1701: 100R_1/10W_1%, Resistor_SMD:R_0603_1608Metric, B.Cu at (198.1, 243.3)
- added R1801: 100R_1/10W_1%, Resistor_SMD:R_0603_1608Metric, B.Cu at (198.1, 240.3)
- added R1901: 100R_1/10W_1%, Resistor_SMD:R_0603_1608Metric, B.Cu at (198.1, 237.2)
- added R2001: 10kR_1/10W_1%, Resistor_SMD:R_0603_1608Metric, B.Cu at (190.8, 237.2)
- added R2701: 10kR_1/10W_1%, Resistor_SMD:R_0603_1608Metric, B.Cu at (199.9, 224.5)
- added R2702: 10kR_1/10W_1%, Resistor_SMD:R_0603_1608Metric, B.Cu at (199.9, 223.0)
- added R2703: 100kR_1/10W_1%, Resistor_SMD:R_0603_1608Metric, B.Cu at (197.9, 227.1)
- added R2704: 470R_1/10W_1%, Resistor_SMD:R_0603_1608Metric, F.Cu at (200.4, 217.2)
- added R2801: 100R_1/10W_1%, Resistor_SMD:R_0603_1608Metric, B.Cu at (201.2, 217.9)
- added R2802: 100R_1/10W_1%, Resistor_SMD:R_0603_1608Metric, B.Cu at (199.6, 217.9)
- added R2901: 0R_1/16W, Resistor_SMD:R_0402_1005Metric, B.Cu at (185.9, 213.6)
- added R2902: 100R_1/10W_1%, Resistor_SMD:R_0603_1608Metric, F.Cu at (167.4, 206.8)
- added R2903: 100R_1/10W_1%, Resistor_SMD:R_0603_1608Metric, F.Cu at (170.5, 206.8)
- added R2904: 100R_1/10W_1%, Resistor_SMD:R_0603_1608Metric, F.Cu at (173.5, 206.8)
- added R3001: 470R_1/10W_1%, Resistor_SMD:R_0603_1608Metric, F.Cu at (188.0, 243.3)
- added R3002: 100R_1/10W_1%, Resistor_SMD:R_0603_1608Metric, F.Cu at (188.0, 241.6)
- added R3003: 100R_1/10W_1%, Resistor_SMD:R_0603_1608Metric, F.Cu at (188.0, 239.8)
- added R3101: 100kR_1/10W_1%, Resistor_SMD:R_0603_1608Metric, F.Cu at (178.3, 247.9)
- added R3102: 100kR_1/10W_1%, Resistor_SMD:R_0603_1608Metric, F.Cu at (165.4, 247.9)
- added R3103: 100kR_1/10W_1%, Resistor_SMD:R_0603_1608Metric, B.Cu at (169.4, 252.0)
- added R3104: 100kR_1/10W_1%, Resistor_SMD:R_0603_1608Metric, F.Cu at (167.9, 252.0)
- added R3105: 1kR_1/10W_1%, Resistor_SMD:R_0603_1608Metric, F.Cu at (164.6, 252.0)
- added R3106: 1kR_1/10W_1%, Resistor_SMD:R_0603_1608Metric, F.Cu at (165.4, 241.6)
- added R3107: 1kR_1/10W_1%, Resistor_SMD:R_0603_1608Metric, F.Cu at (165.4, 243.1)
- added R3108: 100kR_1/10W_1%, Resistor_SMD:R_0603_1608Metric, F.Cu at (169.4, 240.0)
- added R3109: 100kR_1/10W_1%, Resistor_SMD:R_0603_1608Metric, B.Cu at (167.9, 252.0)
- added R3110: 1kR_1/10W_1%, Resistor_SMD:R_0603_1608Metric, F.Cu at (166.4, 252.0)
- added R3301: 4R7_1/4W_1%, Resistor_SMD:R_0805_2012Metric, F.Cu at (155.0, 211.4)
- added R3401: 100kR_1/10W_1%, Resistor_SMD:R_0603_1608Metric, F.Cu at (153.9, 240.3)
- added R3402: 470R_1/10W_1%, Resistor_SMD:R_0603_1608Metric, F.Cu at (160.0, 241.6)
- added R3501: 100kR_1/10W_1%, Resistor_SMD:R_0603_1608Metric, F.Cu at (160.5, 224.5)
- added R3502: 470R_1/10W_1%, Resistor_SMD:R_0603_1608Metric, F.Cu at (162.8, 231.4)
- added R3601: 100kR_1/10W_1%, Resistor_SMD:R_0603_1608Metric, F.Cu at (187.2, 211.6)
- added R3602: 470R_1/10W_1%, Resistor_SMD:R_0603_1608Metric, F.Cu at (194.9, 210.1)
- added R3701: 100kR_1/10W_1%, Resistor_SMD:R_0603_1608Metric, F.Cu at (162.6, 235.2)
- added R3702: 470R_1/10W_1%, Resistor_SMD:R_0603_1608Metric, F.Cu at (163.1, 243.8)
- added R501: 100kR_1/10W_1%, Resistor_SMD:R_0603_1608Metric, B.Cu at (195.6, 232.2)
- added R502: 100kR_1/10W_1%, Resistor_SMD:R_0603_1608Metric, B.Cu at (192.5, 227.6)
- added R601: 10kR_1/10W_1%, Resistor_SMD:R_0603_1608Metric, B.Cu at (190.0, 231.5)
- added R602: 100kR_1/10W_1%, Resistor_SMD:R_0603_1608Metric, B.Cu at (192.5, 230.8)
- added R603: 10kR_1/10W_1%, Resistor_SMD:R_0603_1608Metric, F.Cu at (186.2, 246.9)
- added R604: 1kR_1/10W_1%, Resistor_SMD:R_0603_1608Metric, F.Cu at (182.4, 240.8)
- added R605: 10kR_1/10W_1%, Resistor_SMD:R_0603_1608Metric, F.Cu at (176.8, 240.8)
- added R606: 10kR_1/10W_1%, Resistor_SMD:R_0603_1608Metric, F.Cu at (178.8, 240.8)
- added R607: 10kR_1/10W_1%, Resistor_SMD:R_0603_1608Metric, F.Cu at (175.6, 215.9)
- added R608: 10kR_1/10W_1%, Resistor_SMD:R_0603_1608Metric, F.Cu at (174.0, 215.9)
- added R701: 100R_1/10W_1%, Resistor_SMD:R_0603_1608Metric, F.Cu at (188.5, 247.3)
- added R702: 100R_1/10W_1%, Resistor_SMD:R_0603_1608Metric, F.Cu at (190.0, 247.3)
- added R801: 100kR_1/10W_1%, Resistor_SMD:R_0603_1608Metric, B.Cu at (154.9, 211.3)
- added R802: 100kR_1/10W_1%, Resistor_SMD:R_0603_1608Metric, B.Cu at (154.9, 213.1)
- added R803: 10kR_1/10W_1%, Resistor_SMD:R_0603_1608Metric, B.Cu at (159.5, 209.6)
- added R804: 100kR_1/10W_1%, Resistor_SMD:R_0603_1608Metric, F.Cu at (159.5, 209.6)
- added RV3201: 0.5A_6V_0.15R, Fuse:Fuse_0805_2012Metric, B.Cu at (159.5, 223.8)
- added TXT3801: ~, _PCBLIB_Qcopter:LOGO_Mend0z0, F.Cu at (177.8, 251.2)
- added U1001: PI4IOE5V9554ZHEX, _PCBLIB_Qcopter:QFN-16-1EP_3x3mm_P0.5mm_EP1.75x1.75mm_ThermalVias, B.Cu at (166.6, 219.3)
- added U1101: PI4IOE5V9554ZHEX, _PCBLIB_Qcopter:QFN-16-1EP_3x3mm_P0.5mm_EP1.75x1.75mm_ThermalVias, B.Cu at (165.6, 231.6)
- added U1201: PI4IOE5V9554ZHEX, _PCBLIB_Qcopter:QFN-16-1EP_3x3mm_P0.5mm_EP1.75x1.75mm_ThermalVias, B.Cu at (195.1, 243.2)
- added U1301: ICM-20948, Package_DFN_QFN:QFN-24-1EP_3x3mm_P0.4mm_EP1.75x1.6mm, B.Cu at (177.8, 228.3)
- added U1401: BME280, _PCBLIB_Qcopter:PSON65P250X250X100-8N, B.Cu at (188.0, 246.4)
- added U2001: W25Q64JVSSIQ, Package_SO:SOIC-8_5.23x5.23mm_P1.27mm, B.Cu at (188.0, 241.3)
- added U2301: SN74LVC1G18DCKR, Package_TO_SOT_SMD:SOT-363_SC-70-6, B.Cu at (160.3, 247.5)
- added U2302: DRV8837CDSGR, Package_SON:WSON-8-1EP_2x2mm_P0.5mm_EP0.9x1.6mm_ThermalVias, F.Cu at (160.3, 247.5)
- added U2401: SN74LVC1G18DCKR, Package_TO_SOT_SMD:SOT-363_SC-70-6, B.Cu at (194.8, 247.6)
- added U2402: DRV8837CDSGR, Package_SON:WSON-8-1EP_2x2mm_P0.5mm_EP0.9x1.6mm_ThermalVias, F.Cu at (194.8, 247.7)
- added U2501: SN74LVC1G18DCKR, Package_TO_SOT_SMD:SOT-363_SC-70-6, B.Cu at (189.0, 206.2)
- added U2502: DRV8837CDSGR, Package_SON:WSON-8-1EP_2x2mm_P0.5mm_EP0.9x1.6mm_ThermalVias, F.Cu at (189.0, 206.2)
- added U2601: SN74LVC1G18DCKR, Package_TO_SOT_SMD:SOT-363_SC-70-6, B.Cu at (163.8, 210.6)
- added U2602: DRV8837CDSGR, Package_SON:WSON-8-1EP_2x2mm_P0.5mm_EP0.9x1.6mm_ThermalVias, F.Cu at (163.8, 210.6)
- added U2701: SN74LVC1G17DCKR, Package_TO_SOT_SMD:SOT-353_SC-70-5, B.Cu at (199.9, 227.1)
- added U2702: NX3L1T3157GMZ, _PCBLIB_Qcopter:6-XSON, B.Cu at (186.7, 210.8)
- added U2703: STM32WLE5CCU7, Package_DFN_QFN:QFN-48-1EP_7x7mm_P0.5mm_EP5.6x5.6mm_ThermalVias, B.Cu at (192.7, 218.1)
- added U2901: NX3L1T3157GMZ, _PCBLIB_Qcopter:6-XSON, B.Cu at (179.8, 214.4)
- added U2902: BGS13SN8E6327XTSA1, _PCBLIB_Qcopter:TSNP-8-1_INF, F.Cu at (175.5, 208.9)
- added U3101: ATWILC1000B-MU-Y, _PCBLIB_Qcopter:QFN-40-1EP_5x5mm_P0.4mm_EP3.8x3.8mm_ThermalVias, B.Cu at (171.8, 246.2)
- added U3201: MCP73811T-420I/OT, Package_TO_SOT_SMD:SOT-23-5, B.Cu at (155.2, 216.2)
- added U3301: TPS613222ADBVR, Package_TO_SOT_SMD:SOT-23-5, F.Cu at (157.2, 217.7)
- added U3401: TLV74033PDBVR, Package_TO_SOT_SMD:SOT-23-5, F.Cu at (157.5, 237.0)
- added U3501: TLV74033PDBVR, Package_TO_SOT_SMD:SOT-23-5, F.Cu at (160.5, 227.6)
- added U3601: TLV74033PDBVR, Package_TO_SOT_SMD:SOT-23-5, F.Cu at (191.0, 210.6)
- added U3701: TLV74033PDBVR, Package_TO_SOT_SMD:SOT-23-5, F.Cu at (162.6, 238.3)
- added U501: TLV70313DBVR, Package_TO_SOT_SMD:SOT-23-5, B.Cu at (195.3, 235.2)
- added U502: TLV70328DBVR, Package_TO_SOT_SMD:SOT-23-5, B.Cu at (195.3, 227.3)
- added U601: SN74LVC1G17DCKR, Package_TO_SOT_SMD:SOT-353_SC-70-5, B.Cu at (190.0, 228.7)
- added U602: STM32U575VIT6Q, Package_QFP:LQFP-100_14x14mm_P0.5mm, F.Cu at (177.8, 228.3)
- added U801: MCP6006T-E/OT, Package_TO_SOT_SMD:SOT-23-5, B.Cu at (159.0, 212.2)
- added X2701: 32MHz_10pF_10ppm, _PCBLIB_Qcopter:NX2016SA_NDK, B.Cu at (191.0, 210.3)
- added X3101: 26MHz_10ppm_12pF, Crystal:Crystal_SMD_2016-4Pin_2.0x1.6mm, B.Cu at (171.7, 240.0)
- added X601: 16MHz_12pF_10ppm, Crystal:Crystal_SMD_2016-4Pin_2.0x1.6mm, F.Cu at (190.4, 228.3)
Other:
- board outline added: 49.9 x 49.9 mm
- board text added: "APPROVED"
- board text added: "CHECKED"
- board text added: "D"
- board text added: "DATE"
- board text added: "DESCRIPTION"
- board text added: "DRAWN"
- board text added: "DWG NO"
- board text added: "ENG APPR"
- board text added: "MGR APPR"
- board text added: "NAME"
- board text added: "REV"
- board text added: "REVISION HISTORY"
- board text added: "SCALE:"
- board text added: "SIZE"
- board text added: "Solid Edge"
- board text added: "TITLE"
- board text added: "WEIGHT:"
- board text added: "|p34;\C7;\H0.12;\W1.;2 PL ±X.XX 3 PL ±X.XXX}"

Commit message: Update _Sub_HW_Qcopter.kicad_pcb
Parts:
- C1201, C2102, C2103, C2301, C2401, C2601, C2904, C3101, C3102, C3104, C3105, C3106, C501, C502, C503, C504, C603, C801, D3201, D3202, D3203, FB3101, FB3102, J2701, JP2201, JP2701, L2902, L2903, R1601, R1701, R1801, R1901, R2001, R2702, R2801, R2802, R501, R502, R601, R801, R802, R803, U1201, U2301, U2401, U2501, U2601, U501, U502, U601, U801: moved to F.Cu
- C2708, C2709, C2921, C2922, C2923, C3108, C3501, C3502, C3701, C3702, J2901, J3201, J501, L2909, R3101, R3102, R3104, R3105, R3106, R3107, R3501, R3502, R3701, R605, R606, U2902, U3501, U3701: moved to B.Cu
- C3112: value 4u7F_16V_X7R -> 1pF_50V_C0G; footprint Capacitor_SMD:C_0603_1608Metric -> Capacitor_SMD:C_0201_0603Metric; moved to B.Cu
- C3113: value 12pF_50V_C0G -> 4u7F_16V_X7R; moved to F.Cu
- C3115: value 1pF_50V_C0G -> 12pF_50V_C0G; footprint Capacitor_SMD:C_0201_0603Metric -> Capacitor_SMD:C_0603_1608Metric
- J2202, J2203, J2204, J2205, J3202: footprint Connector_Hirose:Hirose_DF13-02P-1.25DSA_1x02_P1.25mm_Vertical -> _PCBLIB_Qcopter:Hirose_DF13-02P-1.25DSA_1x02_P1.25mm_Vertical
- L3105: value 15nH_560mA_0.172R -> 3n3H_400mA_0.3R; footprint Inductor_SMD:L_0402_1005Metric -> Inductor_SMD:L_0201_0603Metric
- L3106: value 3n3H_400mA_0.3R -> 15nH_560mA_0.172R; footprint Inductor_SMD:L_0201_0603Metric -> Inductor_SMD:L_0402_1005Metric
- R602: value 100kR_1/10W_1% -> 10kR_1/10W_1%; moved to F.Cu
- R603: value 10kR_1/10W_1% -> 100kR_1/10W_1%
- U2001: footprint Package_SO:SOIC-8_5.23x5.23mm_P1.27mm -> _PCBLIB_Qcopter:SOIC-8_5.23x5.23mm_P1.27mm; moved to F.Cu
- U2703: footprint Package_DFN_QFN:QFN-48-1EP_7x7mm_P0.5mm_EP5.6x5.6mm_ThermalVias -> _PCBLIB_Qcopter:QFN-48-1EP_7x7mm_P0.5mm_EP5.6x5.6mm_ThermalVias
- X3101, X601: footprint Crystal:Crystal_SMD_2016-4Pin_2.0x1.6mm -> _PCBLIB_Qcopter:Crystal_SMD_2016-4Pin_2.0x1.6mm
- moved FD3801 51.5 mm to (261.3, 189.1)
- moved FD3803 51.5 mm to (261.3, 194.2)
- moved FD3802 51.5 mm to (261.3, 191.6)
- moved FD3804 51.5 mm to (261.3, 196.7)
- moved J601 41.5 mm to (201.2, 214.0), turned to -90 degrees
- moved J701 36.3 mm to (201.2, 218.4), turned to -90 degrees
- moved C3502 34.8 mm to (194.9, 227.8)
- moved LED3501 34.7 mm to (194.9, 231.0)
- moved U3501 34.6 mm to (194.8, 232.4), turned to 90 degrees
- moved LED3002 33.1 mm to (185.3, 209.0), turned to 90 degrees
- moved R3501 32.8 mm to (192.2, 233.0), turned to 90 degrees
- moved C3501 32.7 mm to (195.0, 235.3), turned to 180 degrees
- moved R3002 32.5 mm to (186.8, 209.0), turned to 90 degrees
- moved R3502 32.2 mm to (194.9, 229.4), turned to 180 degrees
- moved LED3003 32.0 mm to (182.2, 209.0), turned to 90 degrees
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Connections:
- C3112 pad 1: Net-(U3101-VDD_BATT_PA_3V3) -> Net-(C3112-Pad1)
- C3112 pad 2: GND -> Net-(C3112-Pad2)
- C3113 pad 1: /FBD_Quadcopter/FBD_RadioController/ATWIL1000C Driver/ATWILC_XOP -> Net-(U3101-VDD_BATT_PA_3V3)
- C3114 pad 1: /FBD_Quadcopter/FBD_RadioController/ATWIL1000C Driver/ATWILC_XON -> /FBD_Quadcopter/FBD_RadioController/ATWIL1000C Driver/ATWILC_XOP
- C3115 pad 1: Net-(C3115-Pad1) -> /FBD_Quadcopter/FBD_RadioController/ATWIL1000C Driver/ATWILC_XON
- C3115 pad 2: Net-(C3115-Pad2) -> GND
- C3119 pad 2: Net-(C3115-Pad1) -> Net-(C3112-Pad1)
- J1601 pad 1: Net-(J1601-Pad1) -> GND
- J1601 pad 2: GND -> Net-(J1601-Pad2)
- J1701 pad 1: Net-(J1701-Pad1) -> GND
- J1701 pad 2: GND -> Net-(J1701-Pad2)
- J1801 pad 1: Net-(J1801-Pad1) -> GND
- J1801 pad 2: GND -> Net-(J1801-Pad2)
- J1901 pad 1: Net-(J1901-Pad1) -> GND
- J1901 pad 2: GND -> Net-(J1901-Pad2)
- L3101 pad 2: Net-(C3115-Pad2) -> Net-(C3112-Pad2)
- L3102 pad 1: Net-(C3115-Pad2) -> Net-(C3112-Pad2)
- L3104 pad 1: Net-(C3115-Pad1) -> Net-(C3112-Pad1)
- L3105 pad 1: Net-(L3103-Pad2) -> Net-(C3119-Pad1)
- L3105 pad 2: /FBD_Quadcopter/FBD_RadioController/ATWIL1000C Driver/ATWILC_SW -> GND
- L3106 pad 1: Net-(C3119-Pad1) -> Net-(L3103-Pad2)
- L3106 pad 2: GND -> /FBD_Quadcopter/FBD_RadioController/ATWIL1000C Driver/ATWILC_SW
- R1601 pad 2: Net-(J1601-Pad1) -> Net-(J1601-Pad2)
- R1701 pad 2: Net-(J1701-Pad1) -> Net-(J1701-Pad2)
- R1801 pad 2: Net-(J1801-Pad1) -> Net-(J1801-Pad2)
- R1901 pad 2: Net-(J1901-Pad1) -> Net-(J1901-Pad2)
- R602 pad 1: /FBD_Quadcopter/FBD_FlightController/STM32U575 Driver/STM32U5_NRST -> /FBD_Quadcopter/FBD_FlightController/STM32U575 Driver/STM32U5_BOOT0
- R603 pad 1: /FBD_Quadcopter/FBD_FlightController/STM32U575 Driver/STM32U5_BOOT0 -> /FBD_Quadcopter/FBD_FlightController/STM32U575 Driver/STM32U5_NRST

Commit message: Update _Sub_HW_Qcopter.kicad_pcb
Parts:
- moved U2502 0.25 mm to (190.6, 205.7)
- moved C2502 0.25 mm to (189.2, 206.0)
- moved U2901 0.25 mm to (189.2, 208.9)
- moved C3701 0.23 mm to (189.7, 252.2)
- moved C3702 0.23 mm to (189.7, 249.2)
- moved U2501 0.17 mm to (190.6, 208.7)
- moved LED3701 0.13 mm to (184.7, 252.2)
- moved R3701 0.13 mm to (184.7, 252.2)
- moved R3702 0.13 mm to (184.7, 249.2)
- moved C2101 0.10 mm to (200.4, 228.9)
- moved C2403 0.10 mm to (191.4, 252.2)
- moved C2904 0.05 mm to (187.4, 206.8)
- moved C2905 0.05 mm to (187.4, 206.8)
- moved C2908 0.05 mm to (184.9, 205.3)
- moved C2909 0.05 mm to (184.9, 205.3)
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Other:
- copper layers 4 -> 6

Commit message: Update _Sub_HW_Qcopter.kicad_pcb
Parts:
- FD3801, FD3802: moved to B.Cu
- moved FD3801 56.5 mm to (209.7, 212.0), turned to 180 degrees
- moved FD3802 56.5 mm to (209.7, 214.5), turned to 180 degrees
- moved FD3803 56.5 mm to (209.7, 217.1)
- moved FD3804 56.5 mm to (209.7, 219.6)
- moved C2402 8.46 mm to (188.6, 253.0)
- moved C2502 6.41 mm to (194.7, 209.3), turned to 0 degrees
- moved C2401 3.79 mm to (191.4, 249.2), turned to -90 degrees
- moved C1201 2.47 mm to (193.4, 245.7), turned to 0 degrees
- moved L3102 1.04 mm to (173.5, 252.2)
- moved R3104 0.99 mm to (161.0, 245.5), turned to 0 degrees
- moved L3101 0.94 mm to (174.9, 252.7)
- moved U2901 0.46 mm to (189.5, 208.6), turned to 180 degrees
- moved ANT3101 0.40 mm to (178.3, 252.7)
- moved C2711 0.18 mm to (194.7, 210.9)
- moved C2912 0.15 mm to (182.3, 205.3)
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Connections:
- U1001 pad 1: /FBD_Quadcopter/FBD_FlightController/GPIO Expander/GPIOExpander_GND -> GND
- U1001 pad 15: /FBD_Quadcopter/FBD_FlightController/GPIO Expander/GPIOExpander_GND -> GND
- U1001 pad 16: /FBD_Quadcopter/FBD_FlightController/GPIO Expander/GPIOExpander_GND -> GND
- U1101 pad 1: /FBD_Quadcopter/FBD_FlightController/GPIO Expander/GPIOExpander_GND -> GND
- U1101 pad 16: /FBD_Quadcopter/FBD_FlightController/GPIO Expander/GPIOExpander_GND -> GND
- U1201 pad 1: /FBD_Quadcopter/FBD_FlightController/GPIO Expander/GPIOExpander_GND -> GND
- U1201 pad 15: /FBD_Quadcopter/FBD_FlightController/GPIO Expander/GPIOExpander_GND -> GND
Routing:
- net /FBD_Quadcopter/FBD_RadioController/ATWIL1000C Driver/I2C_SDA: track 0.00 -> 104.8 mm, vias 0 -> 2
- net /FBD_Quadcopter/FBD_RadioController/ATWIL1000C Driver/I2C_SCL: track 0.00 -> 93.7 mm, vias 0 -> 2
- net /FBD_Quadcopter/FBD_RadioController/ATWIL1000C Driver/SPI_MOSI: track 0.00 -> 72.6 mm, vias 0 -> 2
- net /FBD_Quadcopter/FBD_RadioController/ATWIL1000C Driver/SPI_CS: track 0.00 -> 68.1 mm, vias 0 -> 2
- net /FBD_Quadcopter/FBD_RadioController/ATWIL1000C Driver/SPI_MISO: track 0.00 -> 62.3 mm, vias 0 -> 2
- net /FBD_Quadcopter/FBD_FlightController/W25Q64 Driver/W25Q64_~{CS}: track 0.00 -> 58.7 mm, vias 0 -> 2
- net /FBD_Quadcopter/FBD_FlightController/W25Q64 Driver/W25Q64_CLK: track 0.00 -> 52.7 mm, vias 0 -> 2
- net /FBD_Quadcopter/FBD_RadioController/ATWIL1000C Driver/SPI_SCK: track 0.00 -> 52.1 mm, vias 0 -> 2
- net /FBD_Quadcopter/FBD_FlightController/RADIO_CTR_SPI_CLK: track 0.00 -> 51.2 mm, vias 0 -> 2
- net /FBD_Quadcopter/FBD_RadioController/ATWIL1000C Driver/ATWILC_RESETN: track 0.00 -> 51.1 mm, vias 0 -> 2
- net /FBD_Quadcopter/FBD_FlightController/OV2640 Driver/OV2460_SIOD: track 0.00 -> 49.8 mm, vias 0 -> 2
- net /FBD_Quadcopter/FBD_FlightController/OV2640 Driver/OV2460_SIOC: track 0.00 -> 47.4 mm, vias 0 -> 2
- net /FBD_Quadcopter/FBD_RadioController/ATWIL1000C Driver/ATWILC_CHIPN: track 0.00 -> 42.9 mm, vias 0 -> 2
- net /FBD_Quadcopter/FBD_FlightController/OV2640 Driver/OV2460_DATA5: track 0.00 -> 41.9 mm, vias 0 -> 2
- net /FBD_Quadcopter/FBD_FlightController/OV2640 Driver/OV2460_STROBE: track 0.00 -> 39.7 mm, vias 0 -> 2
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- added copper zone on In1.Cu, net GND
- added copper zone on In4.Cu, net GND

Commit message: Update _Sub_HW_Qcopter.kicad_pcb
Parts:
- C3110, FB3103: moved to B.Cu
- moved C3110 15.1 mm to (161.1, 242.1), turned to 180 degrees
- moved FB3103 12.9 mm to (161.6, 243.8), turned to 180 degrees
- moved C1302 8.46 mm to (174.1, 228.4), turned to -90 degrees
- moved L3103 1.14 mm to (165.4, 240.3)
- moved L3106 1.14 mm to (164.2, 240.3)
- moved U2902 0.36 mm to (175.0, 205.8)
- moved C2921 0.27 mm to (172.9, 205.8)
- moved C2922 0.17 mm to (171.5, 205.3)
- moved L2909 0.09 mm to (170.1, 205.8)
Routing:
- net GND: track 35.7 -> 83.8 mm, vias 3 -> 16
- net /FBD_Quadcopter/FBD_RadioController/ATWIL1000C Driver/ATWILC_+3.3V: track 0.00 -> 24.6 mm, vias 0 -> 4
- net /FBD_Quadcopter/FBD_FlightController/+3V3_1: track 27.4 -> 47.4 mm, vias 1 -> 4
- net /FBD_Quadcopter/FBD_RadioController/ATWIL1000C Driver/ATWILC_+1.3V: track 2.55 -> 17.4 mm, vias 0 -> 5
- net Net-(U3101-VDD_RF_RX_1V3): track 2.80 -> 15.7 mm, vias 0 -> 3
- net /FBD_Quadcopter/FBD_FlightController/I2C_SDA: track 1.73 -> 12.4 mm, vias 1 -> 4
- net /FBD_Quadcopter/FBD_FlightController/I2C_SCL: track 0.79 -> 11.2 mm, vias 1 -> 4
- net /FBD_Quadcopter/FBD_FlightController/STM32U575 Driver/STM32U5_OSC_I: track 0.00 -> 10.4 mm
- net Net-(U3101-VDD_AMS_1V3): track 3.05 -> 11.5 mm, vias 0 -> 2
- net Net-(U3101-VBATT_BUCK_3V3): track 1.57 -> 10.0 mm, vias 0 -> 2
- net /FBD_Quadcopter/FBD_FlightController/STM32U575 Driver/STM32U5_NRST: track 0.00 -> 7.53 mm
- net /FBD_Quadcopter/FBD_FlightController/STM32U575 Driver/STM32U5_OSC_O: track 0.00 -> 6.03 mm
- net /FBD_Quadcopter/FBD_FlightController/ICM-20948 Driver/ICM_REGOUT: track 0.00 -> 5.59 mm
- net /FBD_Quadcopter/FBD_FlightController/Battery Voltage Sampler/MCP_VOUUT: track 0.00 -> 5.52 mm, vias 0 -> 1
- net /FBD_Quadcopter/FBD_FlightController/STM32U575 Driver/SWRST: track 0.00 -> 5.10 mm
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
Commit message: Update _Sub_HW_Qcopter.kicad_pcb
Parts:
- moved U2702 7.76 mm to (191.5, 209.7), turned to 180 degrees
- moved C1101 2.47 mm to (193.4, 245.7), turned to 0 degrees
- moved R3602 1.71 mm to (175.7, 210.7)
- moved R3502 1.65 mm to (194.9, 227.7)
- moved C3502 1.52 mm to (194.9, 229.4)
- moved C3602 1.46 mm to (174.0, 210.7)
- moved C2906 1.40 mm to (187.5, 208.0)
- moved U2901 0.19 mm to (189.6, 208.7), turned to -90 degrees
Connections:
- U1101 pad 2: /FBD_Quadcopter/Power Supply/LDO +3V3_1/TLV_EN -> /FBD_Quadcopter/Power Supply/LDO +3V3_3/TLV_EN
- U1101 pad 4: /FBD_Quadcopter/Power Supply/LDO +3V3_3/TLV_EN -> /FBD_Quadcopter/Power Supply/TLV13_EN
- U1101 pad 5: /FBD_Quadcopter/Power Supply/TLV13_EN -> /FBD_Quadcopter/Power Supply/LDO +3V3_1/TLV_EN
- U1101 pad 7: /FBD_Quadcopter/FBD_FlightController/OV2640 Driver/OV2460_PWDN -> /FBD_Quadcopter/Power Supply/TLV28_EN
- U1101 pad 8: /FBD_Quadcopter/Power Supply/TLV28_EN -> /FBD_Quadcopter/FBD_FlightController/OV2640 Driver/OV2460_PWDN
Routing:
- net /FBD_Quadcopter/FBD_RadioController/STM32WLE5 Driver/SWRST: track 0.00 -> 41.2 mm
- net /FBD_Quadcopter/Power Supply/TLV13_EN: track 1.60 -> 22.4 mm, vias 0 -> 1
- net /FBD_Quadcopter/Power Supply/LDO +3V3_3/TLV_EN: track 0.00 -> 16.9 mm
- net /FBD_Quadcopter/FBD_RadioController/STM32WLE5 Driver/STM32WLE5_BOOT0: track 0.00 -> 14.3 mm, vias 0 -> 1
- net /FBD_Quadcopter/FBD_FlightController/OV2640 Driver/OV2460_PWDN: track 0.98 -> 14.5 mm
- net /FBD_Quadcopter/FBD_FlightController/OV2640 Driver/OV2460_RESETB: track 0.96 -> 14.5 mm
- net /FBD_Quadcopter/FBD_RadioController/STM32WLE5 Driver/STM32WLE5_NRST: track 0.00 -> 13.2 mm
- net /FBD_Quadcopter/Power Supply/LDO +3V3_1/TLV_EN: track 0.00 -> 9.35 mm
- net GND: track 83.8 -> 91.4 mm
- net /FBD_Quadcopter/FBD_FlightController/STM32U575 Driver/STM32U5_VDDSMPS: track 0.00 -> 6.91 mm
- net /FBD_Quadcopter/FBD_FlightController/BME280 Driver/BME280_A0: track 5.09 -> 11.2 mm
- net /FBD_Quadcopter/FBD_RadioController/STM32WLE5 Driver/STM32WLE5_VDDRF: track 0.00 -> 6.01 mm
- net /FBD_Quadcopter/FBD_RadioController/Activity LEDs Driver/LED_SIG_BLUE: track 0.00 -> 4.84 mm, vias 0 -> 1
- net /FBD_Quadcopter/FBD_RadioController/STM32WLE5 Driver/STM32WLE5_+1.55V: track 0.00 -> 4.52 mm
- net /FBD_Quadcopter/FBD_FlightController/STM32U575 Driver/STM32U5_VDD11: track 0.00 -> 3.88 mm
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