File: Hardware/_Sub_HW_Qcopter/v1_20240309/Design Folder/_Sub_HW_Qcopter/_Sub_HW_Qcopter.kicad_pcb (KiCad board)
At the start: 6 copper layers, 49.9 x 49.9 mm, 293 parts, among them J1601 HDR_1X2_VERT, J1701 HDR_1X2_VERT, J1801 HDR_1X2_VERT, J1901 HDR_1X2_VERT, J2101 FPC_24_R/A-BOTT, J2201 HDR_1X2_5A_THD-RA, J2202 HDR_1X2_VERT_1.25MM, J2203 HDR_1X2_VERT_1.25MM, J2204 HDR_1X2_VERT_1.25MM, J2205 HDR_1X2_VERT_1.25MM, J2701 HDR_1X4_VERT, J2801 HDR_1X3_THD-1.27MM, J2901 RECEPT_RF_50R, J3201 USB_MICRO B_RA, J3202 HDR_1X2_VERT_1.25MM, J501 HDR_1X2_VERT, J601 HDR_1X4_VERT, J701 HDR_1X3_THD-1.27MM, U1001 PI4IOE5V9554ZHEX, U1101 PI4IOE5V9554ZHEX, U1201 PI4IOE5V9554ZHEX, U1301 ICM-20948, U1401 BME280, U2001 W25Q64JVSSIQ, U2301 SN74LVC1G18DCKR, U2302 DRV8837CDSGR, U2401 SN74LVC1G18DCKR, U2402 DRV8837CDSGR, U2501 SN74LVC1G18DCKR, U2502 DRV8837CDSGR, U2601 SN74LVC1G18DCKR, U2602 DRV8837CDSGR, U2701 SN74LVC1G17DCKR, U2702 NX3L1T3157GMZ, U2703 STM32WLE5CCU7, U2901 NX3L1T3157GMZ, U2902 BGS13SN8E6327XTSA1, U3101 ATWILC1000B-MU-Y, U3201 MCP73811T-420I/OT, U3301 TPS613222ADBVR, U3401 TLV74033PDBVR, U3501 TLV74033PDBVR, U3601 TLV74033PDBVR, U3701 TLV74033PDBVR, U501 TLV70313DBVR, U502 TLV70328DBVR, U601 SN74LVC1G17DCKR, U602 STM32U575VIT6Q, U801 MCP6006T-E/OT, X2701 32MHz_10pF_10ppm, X3101 26MHz_10ppm_12pF, X601 16MHz_12pF_10ppm

Commit message: Update _Sub_HW_Qcopter.kicad_pcb
Parts:
- C2502: moved to F.Cu
- moved R604 10.0 mm to (170.1, 239.8)
- moved LED601 9.66 mm to (168.4, 239.8)
- moved C2501 5.63 mm to (190.3, 205.9), turned to 180 degrees
- moved U2502 4.31 mm to (193.6, 208.8), turned to -90 degrees
- moved R2001 3.79 mm to (186.4, 238.4), turned to 90 degrees
- moved JP601 2.25 mm to (177.9, 243.0)
- moved C2502 2.08 mm to (194.7, 211.4), turned to 180 degrees
- moved R602 1.58 mm to (177.9, 239.8), turned to 90 degrees
- moved C2001 1.21 mm to (188.0, 238.4), turned to 90 degrees
- moved R3108 1.10 mm to (175.2, 242.6), turned to 90 degrees
- moved C3104 1.08 mm to (175.1, 246.9), turned to 90 degrees
- moved C3103 1.08 mm to (173.6, 246.9), turned to 90 degrees
- moved R3110 1.08 mm to (173.6, 242.6), turned to -90 degrees
- moved C2503 0.98 mm to (195.7, 207.1), turned to 90 degrees
- moved FB3102 0.80 mm to (171.1, 249.2), turned to -90 degrees
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Routing:
- net GND: track 91.4 -> 156.7 mm, vias 16 -> 31
- net /FBD_Quadcopter/FBD_FlightController/STM32U575 Driver/STM32U5_LED_IND: track 9.14 -> 24.5 mm
- net /FBD_Quadcopter/FBD_RadioController/+3V3_2: track 0.00 -> 9.77 mm, vias 0 -> 1
- net /FBD_Quadcopter/FBD_RadioController/Antenna Driver/RFO_LP: track 0.91 -> 7.85 mm
- net /FBD_Quadcopter/FBD_FlightController/+3V3_1: track 47.4 -> 54.2 mm, vias 4 -> 5
- net /FBD_Quadcopter/FBD_RadioController/Activity LEDs Driver/LED_SIG_RED: track 0.00 -> 6.02 mm, vias 0 -> 1
- net /FBD_Quadcopter/FBD_FlightController/Motor Driver/DRV8837 Driver2/DRV8837_IN_1: track 0.00 -> 5.68 mm
- net /FBD_Quadcopter/FBD_RadioController/STM32WLE5 Driver/LED_INDC: track 0.00 -> 5.57 mm, vias 0 -> 1
- net /FBD_Quadcopter/Power Supply/+5VDC: track 1.92 -> 6.85 mm
- net /FBD_Quadcopter/FBD_FlightController/Battery Voltage Sampler/MCP_VOUUT: track 5.52 -> 10.2 mm
- net /FBD_Quadcopter/FBD_FlightController/Battery Voltage Sampler/MCP_VIN-: track 0.00 -> 4.59 mm
- net Net-(F2201-Pad1): track 0.00 -> 4.56 mm
- net /FBD_Quadcopter/FBD_RadioController/STM32WLE5 Driver/STM32WLE5_+1.55V: track 4.52 -> 8.70 mm, vias 0 -> 2
- net /FBD_Quadcopter/FBD_RadioController/Antenna Driver/VR_PA: track 2.64 -> 6.35 mm, vias 0 -> 1
- net /FBD_Quadcopter/FBD_RadioController/STM32WLE5 Driver/STM32WLE5_VDDRF: track 6.01 -> 9.64 mm, vias 0 -> 2
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- added copper zone on F.Cu, net /FBD_Quadcopter/FBD_FlightController/+3V3DC
- added copper zone on F.Cu, net /FBD_Quadcopter/Power Supply/+5VDC
- added copper zone on F.Cu, net /FBD_Quadcopter/Power Supply/BATTERY CHARGER/MCP_VBAT
- added copper zone on F.Cu, net /FBD_Quadcopter/Power Supply/SMPS DCDC-BOOST +5V/TPS_SW
- added copper zone on F.Cu, net GND

Commit message: Update _Sub_HW_Qcopter.kicad_pcb
Parts:
- moved C2402 1.05 mm to (187.5, 253.0), turned to 180 degrees
- moved U2401 0.72 mm to (187.2, 250.4), turned to -90 degrees
- moved R3502 0.71 mm to (195.0, 227.0)
- moved C3502 0.51 mm to (195.0, 228.9)
- moved C3601 0.48 mm to (167.7, 210.7)
- moved C3501 0.44 mm to (195.0, 235.8)
- moved C3118 0.33 mm to (168.1, 243.6)
- moved C3109 0.30 mm to (169.7, 245.8)
- moved C3120 0.25 mm to (169.7, 247.4)
- moved C3602 0.23 mm to (174.3, 210.7)
- moved C3101 0.20 mm to (165.8, 243.1)
- moved C3102 0.20 mm to (165.8, 244.6)
- moved C3107 0.20 mm to (165.8, 247.7)
- moved C3116 0.20 mm to (165.8, 246.1)
- moved R3602 0.18 mm to (175.8, 210.7)
Connections:
- U2301 pad 1: /FBD_Quadcopter/FBD_FlightController/GPIO Expander/PI4IOE5V9554 Driver/P14IOE5_O5 -> /FBD_Quadcopter/FBD_FlightController/GPIO Expander/PI4IOE5V9554 Driver/P14IOE5_O6
- U2302 pad 7: /FBD_Quadcopter/FBD_FlightController/GPIO Expander/PI4IOE5V9554 Driver/P14IOE5_O1 -> /FBD_Quadcopter/FBD_FlightController/GPIO Expander/PI4IOE5V9554 Driver/P14IOE5_O5
- U2401 pad 1: /FBD_Quadcopter/FBD_FlightController/GPIO Expander/PI4IOE5V9554 Driver/P14IOE5_O6 -> /FBD_Quadcopter/FBD_FlightController/GPIO Expander/PI4IOE5V9554 Driver/P14IOE5_O4
- U2402 pad 7: /FBD_Quadcopter/FBD_FlightController/GPIO Expander/PI4IOE5V9554 Driver/P14IOE5_O2 -> /FBD_Quadcopter/FBD_FlightController/GPIO Expander/PI4IOE5V9554 Driver/P14IOE5_O3
- U2501 pad 1: /FBD_Quadcopter/FBD_FlightController/GPIO Expander/PI4IOE5V9554 Driver/P14IOE5_O7 -> /FBD_Quadcopter/FBD_FlightController/GPIO Expander/PI4IOE5V9554 Driver/P14IOE5_O2
- U2502 pad 7: /FBD_Quadcopter/FBD_FlightController/GPIO Expander/PI4IOE5V9554 Driver/P14IOE5_O3 -> /FBD_Quadcopter/FBD_FlightController/GPIO Expander/PI4IOE5V9554 Driver/P14IOE5_O1
- U2602 pad 7: /FBD_Quadcopter/FBD_FlightController/GPIO Expander/PI4IOE5V9554 Driver/P14IOE5_O4 -> /FBD_Quadcopter/FBD_FlightController/GPIO Expander/PI4IOE5V9554 Driver/P14IOE5_O7
Routing:
- net GND: track 156.7 -> 251.9 mm, vias 31 -> 103
- net /FBD_Quadcopter/FBD_FlightController/+3V3DC: track 10.2 -> 79.5 mm, vias 0 -> 24
- net /FBD_Quadcopter/FBD_FlightController/Motor Driver/DRV8837 Driver/SN74LVC1G18_A: track 1.64 -> 35.3 mm, vias 1 -> 2
- net /FBD_Quadcopter/FBD_FlightController/OV2640 Driver/OV2460_SIOD: track 49.8 -> 24.4 mm
- net /FBD_Quadcopter/FBD_FlightController/OV2640 Driver/OV2460_SIOC: track 47.4 -> 22.6 mm
- net /FBD_Quadcopter/FBD_FlightController/OV2640 Driver/OV2460_STROBE: track 39.9 -> 23.3 mm
- net /FBD_Quadcopter/FBD_FlightController/OV2640 Driver/OV2460_HREF: track 30.4 -> 14.4 mm
- net /FBD_Quadcopter/FBD_FlightController/+3V3_1: track 54.2 -> 69.2 mm, vias 5 -> 14
- net /FBD_Quadcopter/Power Supply/BATTERY CHARGER/DM: track 3.86 -> 18.3 mm
- net /FBD_Quadcopter/Power Supply/BATTERY CHARGER/DP: track 3.74 -> 18.0 mm
- net /FBD_Quadcopter/FBD_FlightController/GPIO Expander/PI4IOE5V9554 Driver/P14IOE5_O7: track 1.27 -> 15.5 mm
- net /FBD_Quadcopter/Power Supply/BATTERY CHARGER/ID: track 3.88 -> 17.5 mm
- net /FBD_Quadcopter/FBD_FlightController/GPIO Expander/PI4IOE5V9554 Driver/P14IOE5_O8: track 0.00 -> 10.4 mm, vias 0 -> 1
- net /FBD_Quadcopter/FBD_FlightController/STM32U575 Driver/STM32U5_VDD11: track 3.88 -> 14.3 mm, vias 0 -> 2
- net /FBD_Quadcopter/FBD_RadioController/+3V3_2: track 9.77 -> 19.1 mm, vias 1 -> 11
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- added copper zone on B.Cu, net /FBD_Quadcopter/FBD_FlightController/+3V3_1
- added copper zone on F.Cu, net /FBD_Quadcopter/FBD_RadioController/+3V3_2
- added copper zone on B.Cu, net /FBD_Quadcopter/FBD_RadioController/ATWIL1000C Driver/ATWILC_+3.3V
- added copper zone on B.Cu, net /FBD_Quadcopter/Power Supply/+5VDC
- added copper zone on B.Cu, net /FBD_Quadcopter/Power Supply/BATTERY CHARGER/MCP_VBAT
- added copper zone on B.Cu, net /FBD_Quadcopter/Power Supply/BATTERY CHARGER/MCP_VDD
- added copper zone on B.Cu, net GND

Commit message: Update _Sub_HW_Qcopter.kicad_pcb
Parts:
- removed D501: GEN_75V_100mA, Diode_SMD:D_0603_1608Metric
- added C501: 1uF_10V_X7R, Capacitor_SMD:C_0603_1608Metric, B.Cu at (154.6, 223.1)
- added R501: 100kR_1/10W_1%, Resistor_SMD:R_0603_1608Metric, B.Cu at (157.0, 222.2)
- added R502: 100kR_1/10W_1%, Resistor_SMD:R_0603_1608Metric, B.Cu at (154.6, 221.5)
- added R503: 100kR_1/10W_1%, Resistor_SMD:R_0603_1608Metric, B.Cu at (154.5, 216.3)
- added U501: SN74LVC1G86DCKR, Package_TO_SOT_SMD:SOT-353_SC-70-5, F.Cu at (154.6, 216.1)
- renumbered C501 to C502, C502 to C503, C503 to C504, C504 to C505, R501 to R504, R502 to R505, U501 to U502, U502 to U503
Connections:
- J501 pad 1: /FBD_Quadcopter/Power Supply/LDO +3V3/TLV_EN -> Net-(J501-Pad1)
Routing:
- net GND: track 251.9 -> 335.2 mm, vias 103 -> 126
- net /FBD_Quadcopter/FBD_FlightController/Motor Driver/MOTOR_VM: track 14.8 -> 20.5 mm, vias 0 -> 8
- net Net-(U501-A): track 0.00 -> 5.21 mm, vias 0 -> 2
- net Net-(J501-Pad1): track 0.00 -> 3.66 mm
- net /FBD_Quadcopter/FBD_FlightController/LDO_EN: track 2.29 -> 5.48 mm
- net /FBD_Quadcopter/Power Supply/LDO +3V3/TLV_EN: track 7.75 -> 5.51 mm
- net /FBD_Quadcopter/FBD_FlightController/GPIO Expander/PI4IOE5V9554 Driver/P14IOE5_O6: track 4.63 -> 2.46 mm
- net /FBD_Quadcopter/FBD_RadioController/Antenna Driver/FE_CTRL1: track 2.46 -> 3.49 mm, vias 1 -> 2
- net /FBD_Quadcopter/Power Supply/+5VDC: track 9.41 -> 10.4 mm, vias 40 -> 41
- net /FBD_Quadcopter/FBD_RadioController/Antenna Driver/FE_CTRL2: track 1.09 -> 2.08 mm, vias 1 -> 2
- net /FBD_Quadcopter/FBD_RadioController/Antenna Driver/FE_CTRL3: track 1.22 -> 2.10 mm, vias 1 -> 2
- net /FBD_Quadcopter/FBD_FlightController/W25Q64 Driver/W25Q64_IO0: track 31.3 -> 32.1 mm
- added copper zone on F.Cu, net /FBD_Quadcopter/FBD_FlightController/Motor Driver/MOTOR_VM

Commit message: Update _Sub_HW_Qcopter.kicad_pcb
Routing:
- net /FBD_Quadcopter/FBD_FlightController/+3V3_1: track 69.1 -> 346.6 mm
- net /FBD_Quadcopter/FBD_FlightController/+3V3DC: track 79.5 -> 327.6 mm
- net /FBD_Quadcopter/FBD_FlightController/Motor Driver/MOTOR_VM: track 20.5 -> 144.1 mm
- net /FBD_Quadcopter/FBD_FlightController/I2C_SCL: track 12.5 -> 103.4 mm, vias 5 -> 6
- net /FBD_Quadcopter/FBD_FlightController/I2C_SDA: track 13.4 -> 95.7 mm, vias 5 -> 4
- net /FBD_Quadcopter/FBD_RadioController/+3V3_2: track 19.1 -> 93.6 mm
- net /FBD_Quadcopter/FBD_FlightController/OV2640 Driver/OV2460_SIOD: track 24.4 -> 80.3 mm
- net /FBD_Quadcopter/FBD_FlightController/OV2640 Driver/OV2460_SIOC: track 22.6 -> 78.4 mm
- net /FBD_Quadcopter/FBD_RadioController/ATWIL1000C Driver/ATWILC_+3.3V: track 27.4 -> 77.6 mm
- net /FBD_Quadcopter/FBD_RadioController/DEBUG UART/UART_TX: track 2.42 -> 20.0 mm, vias 1 -> 2
- net /FBD_Quadcopter/FBD_FlightController/OV2640 Driver/OV2460_HREF: track 14.4 -> 30.9 mm
- net /FBD_Quadcopter/FBD_RadioController/DEBUG UART/UART_RX: track 1.77 -> 18.2 mm, vias 1 -> 2
- net /FBD_Quadcopter/FBD_FlightController/OV2640 Driver/OV2460_STROBE: track 23.3 -> 39.6 mm
- net /FBD_Quadcopter/FBD_RadioController/ATWIL1000C Driver/ATWILC_+1.3V: track 17.9 -> 31.9 mm
- net /FBD_Quadcopter/FBD_RadioController/ATWIL1000C Driver/SPI_MISO: track 63.2 -> 51.2 mm
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- added copper zone on In3.Cu, net /FBD_Quadcopter/FBD_FlightController/+3V3DC
- added copper zone on In3.Cu, net /FBD_Quadcopter/FBD_RadioController/+3V3_2
- added copper zone on In3.Cu, net /FBD_Quadcopter/FBD_RadioController/ATWIL1000C Driver/ATWILC_+3.3V
