File: Hardware/_Sub_HW_Qcopter/v1_20240309/Design Folder/_Sub_HW_Qcopter/_Sub_HW_Qcopter.kicad_pcb (KiCad board)
At the start: 6 copper layers, 49.9 x 49.9 mm, 297 parts, among them J1601 HDR_1X2_VERT, J1701 HDR_1X2_VERT, J1801 HDR_1X2_VERT, J1901 HDR_1X2_VERT, J2101 FPC_24_R/A-BOTT, J2201 HDR_1X2_5A_THD-RA, J2202 HDR_1X2_VERT_1.25MM, J2203 HDR_1X2_VERT_1.25MM, J2204 HDR_1X2_VERT_1.25MM, J2205 HDR_1X2_VERT_1.25MM, J2701 HDR_1X4_VERT, J2801 HDR_1X3_THD-1.27MM, J2901 RECEPT_RF_50R, J3201 USB_MICRO B_RA, J3202 HDR_1X2_VERT_1.25MM, J501 HDR_1X2_VERT, J601 HDR_1X4_VERT, J701 HDR_1X3_THD-1.27MM, U1001 PI4IOE5V9554ZHEX, U1101 PI4IOE5V9554ZHEX, U1201 PI4IOE5V9554ZHEX, U1301 ICM-20948, U1401 BME280, U2001 W25Q64JVSSIQ, U2301 SN74LVC1G18DCKR, U2302 DRV8837CDSGR, U2401 SN74LVC1G18DCKR, U2402 DRV8837CDSGR, U2501 SN74LVC1G18DCKR, U2502 DRV8837CDSGR, U2601 SN74LVC1G18DCKR, U2602 DRV8837CDSGR, U2701 SN74LVC1G17DCKR, U2702 NX3L1T3157GMZ, U2703 STM32WLE5CCU7, U2901 NX3L1T3157GMZ, U2902 BGS13SN8E6327XTSA1, U3101 ATWILC1000B-MU-Y, U3201 MCP73811T-420I/OT, U3301 TPS613222ADBVR, U3401 TLV74033PDBVR, U3501 TLV74033PDBVR, U3601 TLV74033PDBVR, U3701 TLV74033PDBVR, U501 SN74LVC1G86DCKR, U502 TLV70313DBVR, U503 TLV70328DBVR, U601 SN74LVC1G17DCKR, U602 STM32U575VIT6Q, U801 MCP6006T-E/OT, X2701 32MHz_10pF_10ppm, X3101 26MHz_10ppm_12pF, X601 16MHz_12pF_10ppm

Commit message: Update _Sub_HW_Qcopter.kicad_pcb
Routing:
- net /FBD_Quadcopter/FBD_FlightController/+3V3_1: track 346.6 -> 69.1 mm
- net /FBD_Quadcopter/FBD_FlightController/+3V3DC: track 327.6 -> 92.8 mm
- net /FBD_Quadcopter/FBD_FlightController/Motor Driver/MOTOR_VM: track 144.1 -> 20.5 mm
- net /FBD_Quadcopter/FBD_FlightController/GPIO Expander/PI4IOE5V9554 Driver/P14IOE5_O3: track 3.47 -> 87.2 mm
- net /FBD_Quadcopter/FBD_RadioController/+3V3_2: track 93.6 -> 19.1 mm
- net /FBD_Quadcopter/FBD_FlightController/GPIO Expander/PI4IOE5V9554 Driver/P14IOE5_O4: track 2.90 -> 63.5 mm
- net /FBD_Quadcopter/FBD_RadioController/ATWIL1000C Driver/ATWILC_+3.3V: track 77.6 -> 27.7 mm
- net /FBD_Quadcopter/FBD_FlightController/GPIO Expander/PI4IOE5V9554 Driver/P14IOE5_O1: track 4.11 -> 42.7 mm
- net /FBD_Quadcopter/FBD_FlightController/GPIO Expander/PI4IOE5V9554 Driver/P14IOE5_O5: track 4.06 -> 41.3 mm
- net /FBD_Quadcopter/FBD_FlightController/GPIO Expander/PI4IOE5V9554 Driver/P14IOE5_O6: track 2.46 -> 39.0 mm
- net /FBD_Quadcopter/FBD_FlightController/GPIO Expander/PI4IOE5V9554 Driver/P14IOE5_O2: track 2.57 -> 36.7 mm
- net /FBD_Quadcopter/FBD_FlightController/STM32U575 Driver/STM32U5_VDD11: track 14.3 -> 35.6 mm
- net Net-(U501-A): track 5.21 -> 19.2 mm
- net /FBD_Quadcopter/FBD_RadioController/ATWIL1000C Driver/ATWILC_+1.3V: track 31.9 -> 17.9 mm
- net /FBD_Quadcopter/FBD_FlightController/GPIO Expander/PI4IOE5V9554 Driver2/P14IOE5_O5: track 1.88 -> 11.5 mm
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- added copper zone on In3.Cu, net /FBD_Quadcopter/FBD_FlightController/+3V3_1
- added copper zone on In4.Cu, net /FBD_Quadcopter/FBD_FlightController/Motor Driver/MOTOR_VM
- added copper zone on In3.Cu, net /FBD_Quadcopter/FBD_RadioController/ATWIL1000C Driver/ATWILC_+1.3V
- added copper zone on In4.Cu, net /FBD_Quadcopter/Power Supply/+5VDC

Commit message: Update _Sub_HW_Qcopter.kicad_pcb
Parts:
- moved C2708 5.27 mm to (192.2, 222.8), turned to 0 degrees
- moved C2709 3.81 mm to (192.2, 221.3), turned to 0 degrees
- moved J601 2.34 mm to (201.1, 211.7)
- moved C2904 2.23 mm to (186.5, 204.8), turned to 180 degrees
- moved C2905 2.20 mm to (186.5, 204.8), turned to 180 degrees
- moved J2701 2.03 mm to (201.2, 213.9)
- moved L2701 1.71 mm to (186.6, 221.2), turned to 0 degrees
- moved R604 1.65 mm to (168.4, 239.8)
- moved LED601 1.65 mm to (166.8, 239.8)
- moved L2902 1.35 mm to (186.5, 205.8)
- moved L2904 1.35 mm to (186.5, 205.8)
- moved R2901 1.33 mm to (185.6, 206.8)
- moved L2903 1.33 mm to (185.6, 206.8)
- moved U2501 0.41 mm to (190.6, 209.3)
- moved U2901 0.23 mm to (189.7, 208.5), turned to 180 degrees
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Connections:
- R2701 pad 1: /FBD_Quadcopter/FBD_RadioController/STM32WLE5 Driver/STM32U5_VCC -> /FBD_Quadcopter/FBD_RadioController/+3V3_2
- U2701 pad 5: /FBD_Quadcopter/FBD_RadioController/STM32WLE5 Driver/STM32U5_VCC -> /FBD_Quadcopter/FBD_RadioController/+3V3_2
Routing:
- net /FBD_Quadcopter/FBD_FlightController/Motor Driver/DRV8837 Driver1/SN74LVC1G18_A: track 3.07 -> 112.5 mm
- net /FBD_Quadcopter/FBD_FlightController/Debug USART/UART_TX: track 1.47 -> 87.8 mm, vias 1 -> 2
- net /FBD_Quadcopter/FBD_FlightController/Debug USART/UART_RX: track 3.02 -> 87.7 mm, vias 1 -> 2
- net /FBD_Quadcopter/FBD_FlightController/GPIO Expander/PI4IOE5V9554 Driver2/P14IOE5_O7: track 2.87 -> 85.4 mm, vias 2 -> 3
- net /FBD_Quadcopter/FBD_RadioController/STM32WLE5 Driver/SWRST: track 41.6 -> 107.4 mm, vias 0 -> 2
- net /FBD_Quadcopter/FBD_FlightController/STM32U575 Driver/STM32U5_SWCLK: track 0.86 -> 62.1 mm
- net /FBD_Quadcopter/Power Supply/LDO +3V3_2/TLV_EN: track 2.84 -> 61.1 mm, vias 0 -> 1
- net /FBD_Quadcopter/FBD_FlightController/LDO_EN: track 5.48 -> 61.5 mm, vias 2 -> 1
- net /FBD_Quadcopter/FBD_RadioController/Antenna Driver/FE_CTRL1: track 3.49 -> 57.7 mm, vias 2 -> 4
- net /FBD_Quadcopter/FBD_FlightController/STM32U575 Driver/STM32U5_SWDIO: track 2.37 -> 54.3 mm
- net /FBD_Quadcopter/FBD_RadioController/Antenna Driver/FE_CTRL2: track 1.98 -> 47.5 mm
- net /FBD_Quadcopter/FBD_FlightController/Motor Driver/DRV8837 Driver3/SN74LVC1G18_A: track 2.74 -> 42.3 mm
- net GND: track 339.7 -> 366.2 mm, vias 123 -> 122
- net /FBD_Quadcopter/FBD_RadioController/Antenna Driver/FE_CTRL3: track 2.10 -> 28.3 mm, vias 2 -> 1
- net /FBD_Quadcopter/FBD_FlightController/Motor Driver/DRV8837 Driver2/SN74LVC1G18_A: track 5.31 -> 28.7 mm
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
Commit message: Update _Sub_HW_Qcopter.kicad_pcb
Parts:
- moved FD3802 53.3 mm to (156.5, 211.5)
- moved FD3804 47.6 mm to (163.1, 210.1)
- moved FD3801 36.2 mm to (198.3, 246.3)
- moved FD3803 34.4 mm to (196.2, 248.8)
Routing:
- net /FBD_Quadcopter/FBD_RadioController/STM32WLE5 Driver/STM32WLE5_SWCLK: track 24.2 -> 123.1 mm, vias 1 -> 2
- net /FBD_Quadcopter/FBD_RadioController/STM32WLE5 Driver/STM32WLE5_SWDIO: track 14.8 -> 112.7 mm, vias 1 -> 2
- net Net-(U3101-VBATT_BUCK_3V3): track 17.7 -> 31.3 mm
- net Net-(U501-A): track 19.6 -> 12.3 mm
- net /FBD_Quadcopter/FBD_RadioController/ATWIL1000C Driver/SPI_MISO: track 58.3 -> 51.2 mm
- net /FBD_Quadcopter/FBD_RadioController/ATWIL1000C Driver/I2C_SDA: track 110.1 -> 105.2 mm
- net /FBD_Quadcopter/FBD_RadioController/STM32WLE5 Driver/SWRST: track 107.4 -> 102.9 mm
- net /FBD_Quadcopter/FBD_RadioController/ATWIL1000C Driver/I2C_SCL: track 98.3 -> 93.9 mm
- net /FBD_Quadcopter/FBD_RadioController/ATWIL1000C Driver/SPI_SCK: track 58.5 -> 54.2 mm
- net /FBD_Quadcopter/FBD_FlightController/I2C_SCL: track 103.2 -> 99.3 mm
- net /FBD_Quadcopter/FBD_RadioController/ATWIL1000C Driver/SPI_CS: track 76.3 -> 72.9 mm
- net GND: track 366.2 -> 363.3 mm, vias 122 -> 123
- net /FBD_Quadcopter/FBD_FlightController/Motor Driver/DRV8837 Driver1/SN74LVC1G18_A: track 112.5 -> 109.6 mm
- net /FBD_Quadcopter/FBD_RadioController/ATWIL1000C Driver/SPI_MOSI: track 78.9 -> 76.2 mm
- net /FBD_Quadcopter/FBD_RadioController/ATWIL1000C Driver/ATWILC_RESETN: track 57.2 -> 55.4 mm
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Other:
- board text added: "- +"
- board text added: "-+"
- board text added: "3.3V"
- board text added: "3.3V_1"
- board text added: "3.3V_2"
- board text added: "3.3V_3"
- board text added: "BATT"
- board text added: "F_INDC"
- board text added: "GND CLK DIO RST"
- board text added: "GND TXD RXD"
- board text added: "M3x4"
- board text added: "RST DIO CLK GND"
- board text added: "RX"
- board text added: "RXD TXD GND"
- board text added: "R_INDC"
- board text added: "SW"
- board text added: "TX"
- board text added: "VM"
- board text added: "_HW_QCopter v1.0 - 03/25/2024 DSN: SiavashTP"
