File: Hardware/_Sub_HW_DroneController/v1_20240618/Design Folder/_Sub_HW_DroneController/_Sub_HW_DroneController.kicad_sch (KiCad schematic)
At the start: 0 parts

Commit message: Hardware Updates...
Other:
- added sheet FBD_DRONE_CONTROLLER ([02] - FBD_DRONE_CONTROLLER.kicad_sch)
- note added: "${COMMENT2}"
- note added: "${ISSUE_DATE}"
- note added: "${REVISION}"
- note added: "${TITLE}"
- note added: "1"
- note added: "1- Go to View -> Pge Preview Setting 2- Set Parameters based on the following Info COMMENT 1: Project Version COMMENT 2: Document Status COMMENT 3: Doc. Approval Eng. COMMENT 4: BOM Ref. DOC. COMMENT 5: PCB Ref. DOC. COMMENT 6: GBR Ref. DOC. COMMENT 7: ASM Ref. DOC. COMMENT 8: Variant Name COMMENT 9: Revision Description"
- note added: "12"
- note added: "13"
- note added: "14"
- note added: "15-18"
- note added: "19"
- note added: "2"
- note added: "20"
- note added: "21"
- note added: "22-25"
- note added: "26"
- note added: "27"
- note added: "28"
- note added: "29"
- note added: "3"
- note added: "30"
- note added: "31"
- note added: "32"
- note added: "33-36"
- note added: "37"
- note added: "38"
- note added: "39"
- note added: "3D Preview BOTTOM"
- note added: "3D Preview TOP"
- note added: "4"
- note added: "5"
- note added: "6"
- note added: "7"
- note added: "8"
- note added: "9-11"
- note added: "Board Statistics Stackup Info"
- note added: "CAUTIONARY:"
- note added: "COVER PAGE"
- note added: "DESIGN CONSIDERATION"
- note added: "DESIGN NOTE:"
- note added: "DNF"
- note added: "DRAFT - Very Early Stage of Schematic PRELIMINARY - Close to Final Schematic CHECKED - There Should Not Be Any Mistakes RELEASED - A Board with This Schematic Has Been Produced"
- note added: "Example text for Informational design notes."
- note added: "Example text for cautionary design notes."
- note added: "Example text for critial layout guidlines."
- note added: "Example text for critical design notes."
- note added: "FBD_DRONE_CONTROLLER"
- note added: "INFO:"
- note added: "Index"
- note added: "LAYOUT NOTE:"
- note added: "MECHANICAL PARTS"
- note added: "Mark Not Fitted Components as --> Differential Signal Example Net Class Example"
- note added: "PWR SEQUENCE"
- note added: "Page"
- note added: "REVISION HISTORY"
- note added: "SCHEMATIC STATUS:"
- note added: "Set Project Parameters"
- note added: "Symbols and Lables"
- note added: "TEMPLATE NOTES"
- note added: "VARIANT: ${COMMENT8}"
